File: radar_00/radar_01.sch (KiCad schematic (older format))
At the start: 44 parts, among them J1 Screw_Terminal_1x02, J2 Screw_Terminal_1x02, U1 LM358, U2 HB-100-Radar, U3 LM2903, U4 LM78L05ACZ

Commit message: up
Parts:
- added C18: 100,0, Capacitors_SMD:CP_Elec_6.3x5.3, symbol CP
- J1: value Screw_Terminal_1x02 -> Power
- J2: value Screw_Terminal_1x02 -> Out
Connections:
- net GND: now also C18.2
- net at D4.2 (A), J2.1: now also C18.1
Other:
- moved on the sheet: J2
Changed lines of the file:
@@
 P 2900 4950
 F 0 "J1" H 2900 5200 50  0000 C TNN
-F 1 "Screw_Terminal_1x02" V 2750 4950 50  0000 C TNN
+F 1 "Power" V 2750 4950 50  0000 C TNN
 F 2 "Connectors:bornier2" H 2900 4725 50  0001 C CNN
 F 3 "" H 2875 4950 50  0001 C CNN
@@
 L Screw_Terminal_1x02 J2
 U 1 1 5866AF4B
-P 8600 3100
-F 0 "J2" H 8600 3350 50  0000 C TNN
-F 1 "Screw_Terminal_1x02" V 8450 3100 50  0000 C TNN
-F 2 "Connectors:bornier2" H 8600 2875 50  0001 C CNN
-F 3 "" H 8575 3100 50  0001 C CNN
-	1    8600 3100
+P 8850 3100
+F 0 "J2" H 8850 3350 50  0000 C TNN
+F 1 "Out" V 8700 3100 50  0000 C TNN
+F 2 "Connectors:bornier2" H 8850 2875 50  0001 C CNN
+F 3 "" H 8825 3100 50  0001 C CNN
+	1    8850 3100
 	-1   0    0    -1
 $EndComp
@@
 L GND #PWR011
 U 1 1 58670BC3
-P 8400 3200
-F 0 "#PWR011" H 8400 2950 50  0001 C CNN
-F 1 "GND" H 8400 3050 50  0000 C CNN
-F 2 "" H 8400 3200 50  0000 C CNN
-F 3 "" H 8400 3200 50  0000 C CNN
-	1    8400 3200
+P 8500 3300
+F 0 "#PWR011" H 8500 3050 50  0001 C CNN
+F 1 "GND" H 8500 3150 50  0000 C CNN
+F 2 "" H 8500 3300 50  0000 C CNN
+F 3 "" H 8500 3300 50  0000 C CNN
+	1    8500 3300
 	1    0    0    -1
 $EndComp
@@
 	2850 1600 2550 1600
 Connection ~ 2650 1600
+$Comp
+L CP C18
+U 1 1 59F6393C
+P 8500 3150
+F 0 "C18" H 8525 3250 50  0000 L CNN
+F 1 "100,0" H 8250 3050 50  0000 L CNN
+F 2 "Capacitors_SMD:CP_Elec_6.3x5.3" H 8538 3000 50  0001 C CNN
+F 3 "" H 8500 3150 50  0000 C CNN
+	1    8500 3150
+	1    0    0    -1
+$EndComp
+Wire Wire Line
+	8650 3200 8650 3300
+Wire Wire Line
+	8650 3300 8500 3300
+Wire Wire Line
+	8400 3000 8650 3000
+Connection ~ 8500 3000
+Connection ~ 8500 3300
 $EndSCHEMATC
