File: radar_00/radar_04.kicad_pcb (KiCad board)
At the start: 2 copper layers, 88.9 x 44.5 mm, 44 parts, among them J1 Screw_Terminal_1x02, J2 Screw_Terminal_1x02, U1 LM358, U2 HB-100-Radar, U3 LM2903, U4 LM78L05ACZ

Commit message: up
Parts:
- added C18: 100,0, Capacitors_SMD:CP_Elec_6.3x5.3, B.Cu at (156.2, 64.8)
- J1: value Screw_Terminal_1x02 -> Power
- J2: value Screw_Terminal_1x02 -> Out
- moved R6 14.2 mm to (168.9, 67.3)
Routing:
- net Net-(D2-Pad1): track 10.6 -> 22.1 mm
- net Net-(C15-Pad1): track 52.7 -> 43.1 mm, vias 2 -> 4
- net GND: track 195.8 -> 203.7 mm
- net Net-(C18-Pad1): track 85.3 -> 92.6 mm
