File: radar_01/radar_01.sch (KiCad schematic (older format))
At the start: 45 parts, among them J1 Power, J2 Out, U1 LM358, U2 HB-100-Radar, U3 LM2903, U4 LM78L05ACZ

Commit message: up
Parts:
- removed C13, C8: 10,0, Capacitors_SMD:CP_Elec_4x5.3, symbol CP
- removed U4: LM78L05ACZ, TO_SOT_Packages_THT:TO-92_Molded_Wide_Oval, symbol LM78L05ACZ
- added C13, C8: 10,0, Capacitors_SMD:C_0805_HandSoldering, symbol C
- added M1: dcdc5v, dz_lib:dcdc5v, symbol dcdc5v
- C18: footprint (none) -> Capacitors_SMD:CP_Elec_6.3x5.3
- D1, D3, D4: footprint Diodes_SMD:D_MELF_Handsoldering -> Diodes_SMD:D_1206
- U1: footprint Housings_DIP:DIP-8_W7.62mm_Socket -> SMD_Packages:SOIC-8-N
Connections:
- wire segments 55 -> 56
Other:
- moved on the sheet: C7, C9, D2, R6
