File: radar_01/radar_01.kicad_pcb (KiCad board)
At the start: 2 copper layers, 77.5 x 44.5 mm, 45 parts, among them J1 Power, J2 Out, M1 dcdc5v, U1 LM358, U2 HB-100-Radar, U3 LM2903

Commit message: ta7281
Parts:
- moved C3 5.08 mm to (161.3, 86.4)
- moved C7 5.08 mm to (161.3, 68.6)
- moved M1 5.08 mm to (161.3, 77.5)
- moved D2 4.44 mm to (163.2, 64.8)
- moved R6 4.44 mm to (156.8, 64.8)
- moved R12 2.54 mm to (228.6, 72.4)
- moved R13 2.54 mm to (228.6, 64.8)
Routing:
- net Net-(C2-Pad1): track 16.6 -> 22.8 mm
- net +5V: track 125.8 -> 131.0 mm
- net GND: track 257.9 -> 256.2 mm
- net Net-(C15-Pad1): track 42.6 -> 43.7 mm
- net Net-(C13-Pad1): track 23.0 -> 22.2 mm
- net Net-(D3-Pad1): track 60.8 -> 61.4 mm

Commit message: update
Changed lines of the file:
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@@
   (segment (start 202.565 85.725) (end 203.2 86.36) (width 0.5) (layer F.Cu) (net 1))
   (segment (start 203.2 89.44) (end 202.47 90.17) (width 0.5) (layer F.Cu) (net 1) (status 30))
-  (segment (start 209.55 93.98) (end 212.09 93.98) (width 0.25) (layer F.Cu) (net 2))
+  (segment (start 209.55 93.98) (end 212.09 93.98) (width 0.5) (layer F.Cu) (net 2))
   (segment (start 206.47 93.98) (end 209.55 93.98) (width 0.5) (layer B.Cu) (net 2) (status 30))
   (segment (start 196.85 94.51) (end 196.85 95.25) (width 0.5) (layer F.Cu) (net 2) (status 30))
@@
   (segment (start 200.025 84.455) (end 197.39 87.09) (width 0.5) (layer F.Cu) (net 6) (status 20))
   (segment (start 197.39 87.09) (end 196.85 87.09) (width 0.5) (layer F.Cu) (net 6) (status 30))
+  (segment (start 209.55 59.69) (end 212.09 59.69) (width 0.5) (layer F.Cu) (net 7))
   (segment (start 224.79 62.23) (end 228.06 62.23) (width 0.5) (layer F.Cu) (net 7))
   (segment (start 228.06 62.23) (end 228.6 62.77) (width 0.5) (layer F.Cu) (net 7))
@@
   (segment (start 216.44 79.47) (end 215.9 80.01) (width 0.5) (layer F.Cu) (net 7))
   (segment (start 215.9 80.01) (end 209.55 80.01) (width 0.5) (layer F.Cu) (net 7))
-  (segment (start 209.55 59.69) (end 212.09 59.69) (width 0.25) (layer F.Cu) (net 7))
   (segment (start 168.29 68.47) (end 165.79 68.47) (width 0.5) (layer B.Cu) (net 7))
   (segment (start 165.79 68.47) (end 165.68 68.58) (width 0.5) (layer B.Cu) (net 7))
@@
   (segment (start 210.185 85.725) (end 210.82 86.36) (width 0.5) (layer F.Cu) (net 9) (status 20))
   (segment (start 210.82 86.36) (end 210.82 87.09) (width 0.5) (layer F.Cu) (net 9) (status 30))
-  (segment (start 219.71 96.52) (end 222.25 96.52) (width 0.5) (layer F.Cu) (net 10) (status 30))
+  (segment (start 219.71 96.52) (end 222.25 96.52) (width 0.5) (layer B.Cu) (net 10))
   (segment (start 219.71 96.52) (end 219.71 91.44) (width 0.5) (layer F.Cu) (net 10) (status 10))
   (segment (start 219.71 91.44) (end 218.44 90.17) (width 0.5) (layer F.Cu) (net 10))

Commit message: template
Parts:
- moved D5 1.27 mm to (227.3, 88.9)
Routing:
- net Net-(C17-Pad1): track 10.9 -> 8.40 mm
- net Net-(D5-Pad2): track 19.8 -> 19.3 mm
