File: room_unit/ss_relay/ss_relay.sch (KiCad schematic (older format))
At the start: 26 parts, among them J1 DC Load, J2 AC220, P1 CONN_01X02, Q1 IRF730, U1 PC817

Commit message: up
Parts:
- removed D1: MB6S, Diodes_SMD:Diode_Bridge_TO-269AA, symbol D_Bridge_+-AA
- removed R2: 560, Resistors_SMD:R_1206_HandSoldering, symbol R
- added P?: DI_B, Pin_Headers:Pin_Header_Straight_1x02_Pitch2.54mm, symbol CONN_01X02
- P1: value CONN_01X02 -> DI_A
- R1: value 560 -> 1k
Connections:
- net at P1.1 (P1): now also C1.2, D8.2 (A), R3.2, U1.2, P?.1 (P1)
- net at P1.2 (P2): now also R1.2, P?.2 (P2)
Changed lines of the file:
@@
 P 950 1900
 F 0 "P1" H 950 2050 50  0000 C CNN
-F 1 "CONN_01X02" V 1050 1900 50  0000 C CNN
+F 1 "DI_A" V 1050 1900 50  0000 C CNN
 F 2 "Pin_Headers:Pin_Header_Straight_1x02_Pitch2.54mm" H 950 1900 50  0001 C CNN
 F 3 "" H 950 1900 50  0000 C CNN
@@
 P 1600 2150
 F 0 "R1" V 1500 2150 50  0000 C CNN
-F 1 "560" V 1600 2150 50  0000 C CNN
+F 1 "1k" V 1600 2150 50  0000 C CNN
 F 2 "Resistors_SMD:R_1206_HandSoldering" V 1530 2150 50  0001 C CNN
 F 3 "" H 1600 2150 50  0000 C CNN
 	1    1600 2150
 	0    1    1    0
-$EndComp
-$Comp
-L R R2
-U 1 1 59EF8BD8
-P 1600 2750
-F 0 "R2" V 1680 2750 50  0000 C CNN
-F 1 "560" V 1600 2750 50  0000 C CNN
-F 2 "Resistors_SMD:R_1206_HandSoldering" V 1530 2750 50  0001 C CNN
-F 3 "" H 1600 2750 50  0000 C CNN
-	1    1600 2750
-	0    -1   -1   0
 $EndComp
 $Comp
@@
 $EndComp
 Wire Wire Line
-	1750 2750 2900 2750
+	1150 2750 2900 2750
 Wire Wire Line
 	2500 2750 2500 2150
@@
 Connection ~ 2600 2150
 Connection ~ 2600 2750
-Wire Wire Line
-	1750 2450 1750 1850
-Wire Wire Line
-	1750 1850 1150 1850
-Wire Wire Line
-	1150 1950 1150 2450
 Wire Wire Line
 	3500 2550 3500 2450
@@
 	1    3950 1750
 	0    1    1    0
-$EndComp
-$Comp
-L D_Bridge_+-AA D1
-U 1 1 59EFB950
-P 1450 2450
-F 0 "D1" V 1250 2700 50  0000 L CNN
-F 1 "MB6S" V 1150 2700 50  0000 L CNN
-F 2 "Diodes_SMD:Diode_Bridge_TO-269AA" H 1450 2450 50  0001 C CNN
-F 3 "" H 1450 2450 50  0000 C CNN
-	1    1450 2450
-	0    -1   -1   0
 $EndComp
 $Comp
@@
 Connection ~ 6450 2000
 Connection ~ 6800 2400
+$Comp
+L CONN_01X02 P?
+U 1 1 59F22711
+P 950 2700
+F 0 "P?" H 950 2850 50  0000 C CNN
+F 1 "DI_B" V 1050 2700 50  0000 C CNN
+F 2 "Pin_Headers:Pin_Header_Straight_1x02_Pitch2.54mm" H 950 2700 50  0001 C CNN
+F 3 "" H 950 2700 50  0000 C CNN
+	1    950  2700
+	-1   0    0    1
+$EndComp
+Wire Wire Line
+	1150 1850 1450 1850
+Wire Wire Line
+	1450 1850 1450 2650
+Wire Wire Line
+	1450 2650 1150 2650
+Connection ~ 1450 2150
+Wire Wire Line
+	1150 1950 1350 1950
+Wire Wire Line
+	1350 1950 1350 2750
+Connection ~ 1350 2750
 $EndSCHEMATC

Commit message: template
Parts:
- added R1: 1k, Resistors_SMD:R_1206_HandSoldering, symbol R
- Q1: symbol IRF540N -> IRF540N-RESCUE-ss_relay
- gave numbers to parts that had none: 1
- renumbered C3 to C1, C4 to C2, C1 to C3, C2 to C4, D3 to D1, D5 to D2, D2 to D3, D7 to D4, D6 to D5, D8 to D6, D4 to D7, R3 to R2, R6 to R3, R7 to R4, R1 to R5, R4 to R6, R5 to R7
Connections:
- net at C1.2, D2.2 (A), R3.1: now also R1.1; no longer D1.1 (K)
- new net: D1.1 (K), R1.2
Changed lines of the file:
@@
 EESchema Schematic File Version 2
+LIBS:ss_relay-rescue
 LIBS:power
 LIBS:device
@@
 $EndComp
 $Comp
-L R R1
+L R R5
 U 1 1 59EF8BA5
 P 1600 2150
-F 0 "R1" V 1500 2150 50  0000 C CNN
+F 0 "R5" V 1500 2150 50  0000 C CNN
 F 1 "1k" V 1600 2150 50  0000 C CNN
 F 2 "Resistors_SMD:R_1206_HandSoldering" V 1530 2150 50  0001 C CNN
@@
 $EndComp
 $Comp
-L D_Zener D8
+L D_Zener D6
 U 1 1 59EF8CF6
 P 2300 2600
-F 0 "D8" H 2300 2700 50  0000 C CNN
+F 0 "D6" H 2300 2700 50  0000 C CNN
 F 1 "5v6" H 2300 2500 50  0000 C CNN
 F 2 "Diodes_SMD:D_1206" H 2300 2600 50  0001 C CNN
@@
 $EndComp
 $Comp
-L LED D2
+L LED D3
 U 1 1 59EF8D3B
 P 2300 2000
-F 0 "D2" H 2300 2100 50  0000 C CNN
+F 0 "D3" H 2300 2100 50  0000 C CNN
 F 1 "LED" H 2300 1900 50  0000 C CNN
 F 2 "LEDs:LED_D3.0mm" H 2300 2000 50  0001 C CNN
@@
 $EndComp
 $Comp
-L R R3
+L R R2
 U 1 1 59EF8DE2
 P 2500 2000
-F 0 "R3" H 2600 2000 50  0000 C CNN
+F 0 "R2" H 2600 2000 50  0000 C CNN
 F 1 "1k" H 2600 2100 50  0000 C CNN
 F 2 "Resistors_SMD:R_1206_HandSoldering" V 2430 2000 50  0001 C CNN
@@
 $EndComp
 $Comp
-L R R4
+L R R6
 U 1 1 59EF8E4F
 P 2750 2150
-F 0 "R4" V 2830 2150 50  0000 C CNN
+F 0 "R6" V 2830 2150 50  0000 C CNN
 F 1 "1k" V 2900 2150 50  0000 C CNN
 F 2 "Resistors_SMD:R_1206_HandSoldering" V 2680 2150 50  0001 C CNN
@@
 $EndComp
 $Comp
-L C C1
+L C C3
 U 1 1 59EF8FE1
 P 2600 2600
-F 0 "C1" H 2625 2700 50  0000 L CNN
+F 0 "C3" H 2625 2700 50  0000 L CNN
 F 1 "0,1" H 2625 2500 50  0000 L CNN
 F 2 "Capacitors_SMD:C_1206_HandSoldering" H 2638 2450 50  0001 C CNN
@@
 $EndComp
 $Comp
-L C C2
+L C C4
 U 1 1 59EF94AB
 P 3650 2600
-F 0 "C2" H 3675 2700 50  0000 L CNN
+F 0 "C4" H 3675 2700 50  0000 L CNN
 F 1 "0,1" H 3675 2500 50  0000 L CNN
 F 2 "Capacitors_SMD:C_1206_HandSoldering" H 3688 2450 50  0001 C CNN
@@
 $EndComp
 $Comp
-L D_Zener D4
+L D_Zener D7
 U 1 1 59EF950A
 P 3900 2600
-F 0 "D4" V 4000 2700 50  0000 C CNN
+F 0 "D7" V 4000 2700 50  0000 C CNN
 F 1 "7,5v 1500a" V 4100 2700 50  0000 C CNN
 F 2 "Diodes_THT:D_DO-201AD_P5.08mm_Vertical_KathodeUp" H 3900 2600 50  0001 C CNN
@@
 $EndComp
 $Comp
-L IRF540N Q1
+L IRF540N-RESCUE-ss_relay Q1
 U 1 1 59EF955B
 P 4300 2400
@@
 $EndComp
 $Comp
-L R R5
+L R R7
 U 1 1 59EF9689
 P 3650 2300
-F 0 "R5" H 3800 2350 50  0000 C CNN
+F 0 "R7" H 3800 2350 50  0000 C CNN
 F 1 "470k 1W" H 3900 2250 50  0000 C CNN
 F 2 "Resistors_THT:R_Axial_DIN0617_L17.0mm_D6.0mm_P20.32mm_Horizontal" V 3580 2300 50  0001 C CNN
@@
 $EndComp
 $Comp
-L R R7
+L R R4
 U 1 1 59EF96EE
 P 4400 2050
-F 0 "R7" H 4500 2100 50  0000 C CNN
+F 0 "R4" H 4500 2100 50  0000 C CNN
 F 1 "56" H 4500 2000 50  0000 C CNN
 F 2 "Resistors_THT:R_Axial_DIN0617_L17.0mm_D6.0mm_P20.32mm_Horizontal" V 4330 2050 50  0001 C CNN
@@
 $EndComp
 $Comp
-L R R6
+L R R3
 U 1 1 59EF9745
 P 4150 2050
-F 0 "R6" H 4000 2100 50  0000 C CNN
+F 0 "R3" H 4000 2100 50  0000 C CNN
 F 1 "470k 1W" H 3900 2000 50  0000 C CNN
 F 2 "Resistors_THT:R_Axial_DIN0617_L17.0mm_D6.0mm_P20.32mm_Horizontal" V 4080 2050 50  0001 C CNN
@@
 $EndComp
 $Comp
-L D D6
+L D D5
 U 1 1 59EF97B0
 P 4700 2050
-F 0 "D6" V 4050 2000 50  0000 C CNN
+F 0 "D5" V 4050 2000 50  0000 C CNN
 F 1 "RL206" V 4150 2050 50  0000 C CNN
 F 2 "Diodes_THT:D_DO-15_P5.08mm_Vertical_AnodeUp" H 4700 2050 50  0001 C CNN
@@
 $EndComp
 $Comp
-L C C3
+L C C1
 U 1 1 59EF987A
 P 4150 1750
-F 0 "C3" H 4175 1850 50  0000 L CNN
+F 0 "C1" H 4175 1850 50  0000 L CNN
 F 1 "0,1" H 4175 1650 50  0000 L CNN
 F 2 "Capacitors_SMD:C_1206_HandSoldering" H 4188 1600 50  0001 C CNN
@@
 $EndComp
 $Comp
-L C C4
+L C C2
 U 1 1 59EF98D3
 P 4400 1750
-F 0 "C4" H 4425 1850 50  0000 L CNN
+F 0 "C2" H 4425 1850 50  0000 L CNN
 F 1 "0,1 400v" H 4425 1650 50  0000 L CNN
 F 2 "Capacitors_THT:C_Rect_L10.3mm_W5.0mm_P7.50mm_MKS4" H 4438 1600 50  0001 C CNN
@@
 $EndComp
 $Comp
-L LED D3
+L LED D1
 U 1 1 59EF99DE
 P 3350 1750
-F 0 "D3" H 3350 1850 50  0000 C CNN
+F 0 "D1" H 3350 1850 50  0000 C CNN
 F 1 "LED" H 3350 1650 50  0000 C CNN
 F 2 "LEDs:LED_D3.0mm" H 3350 1750 50  0001 C CNN
@@
 	4400 2750 4400 2600
 Connection ~ 3900 2750
-Wire Wire Line
-	3350 1900 4150 1900
 Connection ~ 3950 1900
 Wire Wire Line
@@
 	6800 2400 6800 2200
 $Comp
-L D_Zener D5
+L D_Zener D2
 U 1 1 59EFA527
 P 3950 1750
-F 0 "D5" V 3850 1550 50  0000 C CNN
+F 0 "D2" V 3850 1550 50  0000 C CNN
 F 1 "5v6" V 3950 1550 50  0000 C CNN
 F 2 "Diodes_SMD:D_1206" H 3950 1750 50  0001 C CNN
@@
 $EndComp
 $Comp
-L D_Bridge_+-AA D7
+L D_Bridge_+-AA D4
 U 1 1 59EFBBD9
 P 6100 2000
-F 0 "D7" V 5900 1700 50  0000 L CNN
+F 0 "D4" V 5900 1700 50  0000 L CNN
 F 1 "MB6S" V 5800 1650 50  0000 L CNN
 F 2 "Diodes_SMD:Diode_Bridge_TO-269AA" H 6100 2000 50  0001 C CNN
@@
 Connection ~ 6800 2400
 $Comp
-L CONN_01X02 P?
+L CONN_01X02 P2
 U 1 1 59F22711
 P 950 2700
-F 0 "P?" H 950 2850 50  0000 C CNN
+F 0 "P2" H 950 2850 50  0000 C CNN
 F 1 "DI_B" V 1050 2700 50  0000 C CNN
 F 2 "Pin_Headers:Pin_Header_Straight_1x02_Pitch2.54mm" H 950 2700 50  0001 C CNN
@@
 	1350 1950 1350 2750
 Connection ~ 1350 2750
+$Comp
+L R R1
+U 1 1 5AD1DBBD
+P 3700 1900
+F 0 "R1" H 3800 1900 50  0000 C CNN
+F 1 "1k" H 3800 2000 50  0000 C CNN
+F 2 "Resistors_SMD:R_1206_HandSoldering" V 3630 1900 50  0001 C CNN
+F 3 "" H 3700 1900 50  0000 C CNN
+	1    3700 1900
+	0    1    1    0
+$EndComp
+Wire Wire Line
+	3550 1900 3350 1900
+Wire Wire Line
+	3850 1900 4150 1900
 $EndSCHEMATC
