File: capacity_sensor/capacity_sensor.kicad_pcb (KiCad board)
At the start: 2 copper layers, 45.7 x 47 mm, 31 parts, among them J1 TP1, J2 Sensor, J3 TP2, J4 TP3, J5 Polarity, J6 TP4, J7 Pwr/Out, Q1 BC546, U1 ICM7555, U2 74HCT14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

Commit message: update
Parts:
- added C6: 0,1, Capacitors_SMD:C_0805_HandSoldering, B.Cu at (114.3, 95.2)
- added C7: 0,1, Capacitors_SMD:C_0805_HandSoldering, B.Cu at (133.3, 104.1)
- added C8: 4,7pF, Capacitors_SMD:C_0805_HandSoldering, B.Cu at (121.9, 116.8)
- moved J1 16.5 mm to (113.0, 100.3)
- moved R3 2.54 mm to (119.4, 110.5)
- moved C2 1.27 mm to (119.4, 118.1)
- turned C4 to 180 degrees
Connections:
- U1 pad 4: Net-(U1-Pad4) -> (no net)
- U1 pad 5: Net-(U1-Pad5) -> (no net)
- U3 pad 9: Net-(U3-Pad9) -> (no net)
Routing:
- net GND: track 0.00 -> 178.0 mm
- net +5V: track 0.00 -> 100.3 mm
- net Net-(J6-Pad1): track 0.00 -> 34.8 mm, vias 0 -> 2
- net Net-(R5-Pad2): track 0.00 -> 30.9 mm
- net Net-(C2-Pad1): track 0.00 -> 27.1 mm
- net Net-(J1-Pad1): track 0.00 -> 22.4 mm
- net Net-(U3-Pad12): track 0.00 -> 16.3 mm
- net Net-(J4-Pad1): track 0.00 -> 14.5 mm
- net Net-(J3-Pad1): track 0.00 -> 13.8 mm
- net Net-(J5-Pad3): track 0.00 -> 13.5 mm
- net Net-(C3-Pad1): track 0.00 -> 10.4 mm
- net Net-(U1-Pad3): track 0.00 -> 10.3 mm
- net Net-(J7-Pad2): track 0.00 -> 9.83 mm
- net Net-(C1-Pad1): track 0.00 -> 9.51 mm
- net Net-(J2-Pad1): track 0.00 -> 8.92 mm
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- added copper zone on B.Cu, net GND
- added copper zone on F.Cu, net GND
Other:
- board size 45.7 x 47 mm -> 41.9 x 47 mm
