File: ac_220_di/ac_220_di.kicad_pcb (KiCad board)
At the start: 2 copper layers, 14 parts, among them P1 In, P2 Led, P3 Out, U1 4N35

Commit message: template
Other:
- board outline added: 40.6 x 29.2 mm
Changed lines of the file:
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@@
-(kicad_pcb (version 4) (host pcbnew 4.0.5)
+(kicad_pcb (version 4) (host pcbnew 4.0.7)
   (general
     (links 22)
     (no_connects 1)
-    (area 130.104999 88.255 186.520001 129.570001)
+    (area 114.224999 90.094999 155.015001 119.455001)
     (thickness 1.6)
-    (drawings 0)
+    (drawings 4)
     (tracks 66)
     (zones 0)
@@
     (pad_to_mask_clearance 0.2)
     (aux_axis_origin 0 0)
-    (visible_elements FFFFFF7F)
+    (visible_elements 7FFFFFFF)
     (pcbplotparams
       (layerselection 0x00030_80000001)
@@
     )
   )
+  (gr_line (start 114.3 119.38) (end 154.94 119.38) (angle 90) (layer Edge.Cuts) (width 0.15))
+  (gr_line (start 114.3 90.17) (end 114.3 119.38) (angle 90) (layer Edge.Cuts) (width 0.15))
+  (gr_line (start 154.94 90.17) (end 114.3 90.17) (angle 90) (layer Edge.Cuts) (width 0.15))
+  (gr_line (start 154.94 119.38) (end 154.94 90.17) (angle 90) (layer Edge.Cuts) (width 0.15))
   (segment (start 139.7 99.695) (end 139.7 94.615) (width 0.25) (layer B.Cu) (net 1))
   (segment (start 130.81 107.73) (end 130.082 107.73) (width 0.25) (layer B.Cu) (net 1))
@@
   (segment (start 130.81 105.63) (end 134.205 105.63) (width 0.25) (layer B.Cu) (net 4))
   (segment (start 134.205 105.63) (end 135.128 106.553) (width 0.25) (layer B.Cu) (net 4))
-  (segment (start 151.13 103.886) (end 151.13 101.378) (width 0.25) (layer B.Cu) (net 5) (status C00000))
-  (segment (start 151.13 101.378) (end 151.098 101.346) (width 0.25) (layer B.Cu) (net 5) (status C00000))
-  (segment (start 151.098 101.346) (end 151.098 99.06) (width 0.25) (layer B.Cu) (net 5) (status C00000))
-  (segment (start 147.098 99.06) (end 147.098 101.346) (width 0.25) (layer B.Cu) (net 6) (status C00000))
-  (segment (start 147.098 101.346) (end 149.098 103.346) (width 0.25) (layer B.Cu) (net 6) (status 400000))
+  (segment (start 151.13 103.886) (end 151.13 101.378) (width 0.25) (layer B.Cu) (net 5))
+  (segment (start 151.13 101.378) (end 151.098 101.346) (width 0.25) (layer B.Cu) (net 5))
+  (segment (start 151.098 101.346) (end 151.098 99.06) (width 0.25) (layer B.Cu) (net 5))
+  (segment (start 147.098 99.06) (end 147.098 101.346) (width 0.25) (layer B.Cu) (net 6))
+  (segment (start 147.098 101.346) (end 149.098 103.346) (width 0.25) (layer B.Cu) (net 6))
   (segment (start 149.098 103.346) (end 149.098 106.934) (width 0.25) (layer B.Cu) (net 6))
-  (segment (start 149.098 106.934) (end 151.13 108.966) (width 0.25) (layer B.Cu) (net 6) (status 800000))
+  (segment (start 149.098 106.934) (end 151.13 108.966) (width 0.25) (layer B.Cu) (net 6))
   (segment (start 149.86 112.522) (end 149.86 112.268) (width 0.25) (layer B.Cu) (net 6))
   (segment (start 149.86 112.268) (end 151.13 110.998) (width 0.25) (layer B.Cu) (net 6))
@@
   (segment (start 152.908 105.41) (end 152.908 95.504) (width 0.25) (layer B.Cu) (net 8))
   (segment (start 152.908 95.504) (end 150.876 93.472) (width 0.25) (layer B.Cu) (net 8))
-  (segment (start 145.288 95.98) (end 147.606 95.98) (width 0.25) (layer B.Cu) (net 9) (status 400000))
-  (segment (start 148.336 95.25) (end 148.336 93.472) (width 0.25) (layer B.Cu) (net 9) (status 800000))
+  (segment (start 145.288 95.98) (end 147.606 95.98) (width 0.25) (layer B.Cu) (net 9))
+  (segment (start 148.336 95.25) (end 148.336 93.472) (width 0.25) (layer B.Cu) (net 9))
   (segment (start 147.606 95.98) (end 148.336 95.25) (width 0.25) (layer B.Cu) (net 9))
-  (segment (start 145.288 91.98) (end 146.018 91.98) (width 0.25) (layer B.Cu) (net 10) (status C00000))
-  (segment (start 146.018 91.98) (end 146.558 91.44) (width 0.25) (layer B.Cu) (net 10) (status 400000))
+  (segment (start 145.288 91.98) (end 146.018 91.98) (width 0.25) (layer B.Cu) (net 10))
+  (segment (start 146.018 91.98) (end 146.558 91.44) (width 0.25) (layer B.Cu) (net 10))
   (segment (start 146.558 91.44) (end 152.4 91.44) (width 0.25) (layer B.Cu) (net 10))
   (segment (start 152.4 91.44) (end 153.416 92.456) (width 0.25) (layer B.Cu) (net 10))
@@
   (segment (start 151.638 115.316) (end 146.05 115.316) (width 0.25) (layer B.Cu) (net 10))
   (segment (start 146.05 115.316) (end 144.78 114.046) (width 0.25) (layer B.Cu) (net 10))
-  (segment (start 144.78 114.046) (end 144.78 112.522) (width 0.25) (layer B.Cu) (net 10) (status 800000))
+  (segment (start 144.78 114.046) (end 144.78 112.522) (width 0.25) (layer B.Cu) (net 10))
 )
