File: audio_ta7281/audio_ta7281.kicad_pcb (KiCad board)
At the start: 2 copper layers, 52.1 x 69.8 mm, 24 parts, among them J1 PwrA, J2 PwrB, J3 Out, P1 In, U1 TA7281

Commit message: template
Parts:
- added ?: MountingHole_3.2mm_M3, Mounting_Holes:MountingHole_3.2mm_M3, F.Cu at (209.6, 44.5)
- added ?: MountingHole_3.2mm_M3, Mounting_Holes:MountingHole_3.2mm_M3, F.Cu at (212.1, 24.1)
- added ?: MountingHole_3.2mm_M3, Mounting_Holes:MountingHole_3.2mm_M3, F.Cu at (167.6, 24.1)
- added ?: MountingHole_3.2mm_M3, Mounting_Holes:MountingHole_3.2mm_M3, F.Cu at (212.1, 86.4)
- added ?: MountingHole_3.2mm_M3, Mounting_Holes:MountingHole_3.2mm_M3, F.Cu at (167.6, 86.4)
- added ?: MountingHole_3.2mm_M3, Mounting_Holes:MountingHole_3.2mm_M3, F.Cu at (168.9, 44.5)
Routing:
- net /OutB: track 32.2 -> 59.0 mm
- net Net-(C12-Pad2): track 0.00 -> 17.4 mm, vias 0 -> 1
- added copper zone on F.Cu, net GNDA
Other:
- outline, holes or cut-outs redrawn
