File: capacity_sensor_smd/capacity_sensor.kicad_pcb (KiCad board)
At the start: 2 copper layers, 41.9 x 45.7 mm, 37 parts, among them J1 TP1, J2 Sensor, J3 TP2, J4 TP3, J5 Polarity, J6 TP4, J7 Pwr/Out, P1 Prot. Diode, Q1 2N2222, U1 ICM7555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

Commit message: template
Parts:
- D1: value LED -> Out
- D4: value LED -> Pwr
- D5: value D -> 1N4148
Connections:
- Q1 pad 2: Net-(D2-Pad1) -> GND
- Q1 pad 3: GND -> Net-(D2-Pad1)
Routing:
- net GND: track 177.0 -> 188.5 mm, vias 2 -> 3
- net Net-(D2-Pad1): track 7.65 -> 9.41 mm
Other:
- board text added: "Freq"
- board text added: "Trigger"
