File: capacity_sensor_smd/capacity_sensor.sch (KiCad schematic (older format))
At the start: 34 parts, among them J1 TP1, J2 Sensor, J3 TP2, J4 TP3, J5 Polarity, J6 TP4, J7 Pwr/Out, Q1 BC546, U1 ICM7555, U2 74HCT14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

Commit message: update
Parts:
- removed D2: LED_Dual_CAC, LEDs:LED_D8.0mm-3, symbol LED_Dual_CAC
- removed Q1: BC546, TO_SOT_Packages_THT:TO-92_Molded_Narrow, symbol BC546
- added D1, D4: LED, LEDs:LED_1206_HandSoldering, symbol LED
- added D5: D, Diodes_SMD:D_PowerDI-123, symbol D
- added P1: Prot. Diode, Pin_Headers:Pin_Header_Straight_1x01_Pitch2.54mm, symbol CONN_01X01
- added Q1: 2N2222, TO_SOT_Packages_SMD:SOT-23_Handsoldering, symbol PZT2222A
- C4: renamed from C?; value 10pF -> 4,7pF
- C5: footprint Capacitors_Tantalum_SMD:CP_Tantalum_Case-B_EIA-3528-21_Hand -> Capacitors_Tantalum_SMD:CP_Tantalum_Case-A_EIA-3216-18_Hand
- C6: renamed from C3; value 10,0 -> 100,0
- J7: footprint TerminalBlocks_Phoenix:TerminalBlock_Phoenix_MKDS1.5-3pol -> Connectors_Terminal_Blocks:TerminalBlock_Altech_AK300-3_P5.00mm
- U2, U3: footprint Housings_DIP:DIP-14_W7.62mm -> Housings_SOIC:SOIC-14_3.9x8.7mm_Pitch1.27mm
- renumbered C6 to C1, C1 to C2, C2 to C3, C4 to C7, C7 to C8, D1 to D2
Connections:
- wire segments 47 -> 53
- no-connect marks 3 -> 4
Other:
- moved on the sheet: R9
Changed lines of the file:
@@
 Connection ~ 2300 1900
 $Comp
-L C C1
+L C C2
 U 1 1 5A57793B
 P 2300 2450
-F 0 "C1" H 2325 2550 50  0000 L CNN
+F 0 "C2" H 2325 2550 50  0000 L CNN
 F 1 "2n2" H 2325 2350 50  0000 L CNN
 F 2 "Capacitors_SMD:C_0805_HandSoldering" H 2338 2300 50  0001 C CNN
@@
 F 0 "U2" H 2900 1600 50  0000 C CNN
 F 1 "74HCT14" H 2950 1400 50  0000 C CNN
-F 2 "Housings_DIP:DIP-14_W7.62mm" H 2750 1500 50  0001 C CNN
+F 2 "Housings_SOIC:SOIC-14_3.9x8.7mm_Pitch1.27mm" H 2750 1500 50  0001 C CNN
 F 3 "" H 2750 1500 50  0001 C CNN
 	1    2750 1500
@@
 F 0 "U2" H 4400 1600 50  0000 C CNN
 F 1 "74HCT14" H 4450 1400 50  0000 C CNN
-F 2 "Housings_DIP:DIP-14_W7.62mm" H 4250 1500 50  0001 C CNN
+F 2 "Housings_SOIC:SOIC-14_3.9x8.7mm_Pitch1.27mm" H 4250 1500 50  0001 C CNN
 F 3 "" H 4250 1500 50  0001 C CNN
 	2    4250 1500
@@
 F 0 "U2" H 4400 2300 50  0000 C CNN
 F 1 "74HCT14" H 4450 2100 50  0000 C CNN
-F 2 "Housings_DIP:DIP-14_W7.62mm" H 4250 2200 50  0001 C CNN
+F 2 "Housings_SOIC:SOIC-14_3.9x8.7mm_Pitch1.27mm" H 4250 2200 50  0001 C CNN
 F 3 "" H 4250 2200 50  0001 C CNN
 	3    4250 2200
@@
 $Comp
 L 74HC14 U2
-U 6 1 5A577C29
+U 4 1 5A577C29
 P 6450 1500
 F 0 "U2" H 6600 1600 50  0000 C CNN
 F 1 "74HCT14" H 6650 1400 50  0000 C CNN
-F 2 "Housings_DIP:DIP-14_W7.62mm" H 6450 1500 50  0001 C CNN
+F 2 "Housings_SOIC:SOIC-14_3.9x8.7mm_Pitch1.27mm" H 6450 1500 50  0001 C CNN
 F 3 "" H 6450 1500 50  0001 C CNN
-	6    6450 1500
+	4    6450 1500
 	1    0    0    -1
 $EndComp
@@
 F 0 "U2" H 6600 2300 50  0000 C CNN
 F 1 "74HCT14" H 6650 2100 50  0000 C CNN
-F 2 "Housings_DIP:DIP-14_W7.62mm" H 6450 2200 50  0001 C CNN
+F 2 "Housings_SOIC:SOIC-14_3.9x8.7mm_Pitch1.27mm" H 6450 2200 50  0001 C CNN
 F 3 "" H 6450 2200 50  0001 C CNN
 	5    6450 2200
@@
 $Comp
 L 74HC14 U2
-U 4 1 5A577D6C
+U 6 1 5A577D6C
 P 8450 3200
 F 0 "U2" H 8600 3300 50  0000 C CNN
 F 1 "74HCT14" H 8650 3100 50  0000 C CNN
-F 2 "Housings_DIP:DIP-14_W7.62mm" H 8450 3200 50  0001 C CNN
+F 2 "Housings_SOIC:SOIC-14_3.9x8.7mm_Pitch1.27mm" H 8450 3200 50  0001 C CNN
 F 3 "" H 8450 3200 50  0001 C CNN
-	4    8450 3200
+	6    8450 3200
 	1    0    0    -1
 $EndComp
@@
 F 0 "U3" H 7650 2250 50  0000 C CNN
 F 1 "74HC74" H 7800 1655 50  0000 C CNN
-F 2 "Housings_DIP:DIP-14_W7.62mm" H 7500 1950 50  0001 C CNN
+F 2 "Housings_SOIC:SOIC-14_3.9x8.7mm_Pitch1.27mm" H 7500 1950 50  0001 C CNN
 F 3 "" H 7500 1950 50  0001 C CNN
 	1    7500 1950
 	1    0    0    -1
 $EndComp
-Wire Wire Line
-	6900 1750 6900 1500
-Wire Wire Line
-	6900 1950 6900 2200
 $Comp
 L Conn_01x03_Male J5
@@
 	8100 1850 8250 1850
 Wire Wire Line
-	8100 1150 8100 1850
-Wire Wire Line
 	8250 1950 8000 1950
 Wire Wire Line
@@
 Connection ~ 5300 2200
 $Comp
-L C C2
+L C C3
 U 1 1 5A5788DE
 P 5700 2350
-F 0 "C2" H 5725 2450 50  0000 L CNN
+F 0 "C3" H 5725 2450 50  0000 L CNN
 F 1 "10pF" H 5725 2250 50  0000 L CNN
 F 2 "Capacitors_SMD:C_0805_HandSoldering" H 5738 2200 50  0001 C CNN
@@
 $EndComp
 $Comp
-L CP C3
+L CP C6
 U 1 1 5A578B00
 P 8000 3550
-F 0 "C3" H 8025 3650 50  0000 L CNN
-F 1 "10,0" H 8025 3450 50  0000 L CNN
+F 0 "C6" H 8025 3650 50  0000 L CNN
+F 1 "100,0" H 8025 3450 50  0000 L CNN
 F 2 "Capacitors_Tantalum_SMD:CP_Tantalum_Case-B_EIA-3528-21_Hand" H 8038 3400 50  0001 C CNN
 F 3 "" H 8000 3550 50  0001 C CNN
@@
 $EndComp
 $Comp
-L BC546 Q1
-U 1 1 5A57953A
-P 9400 3200
-F 0 "Q1" H 9600 3275 50  0000 L CNN
-F 1 "BC546" H 9600 3200 50  0000 L CNN
-F 2 "TO_SOT_Packages_THT:TO-92_Molded_Narrow" H 9600 3125 50  0001 L CIN
-F 3 "" H 9400 3200 50  0001 L CNN
-	1    9400 3200
-	1    0    0    -1
-$EndComp
-$Comp
 L GND #PWR08
 U 1 1 5A5796EB
@@
 $EndComp
 $Comp
-L D D1
+L D D2
 U 1 1 5A5797B5
 P 9500 2650
-F 0 "D1" H 9500 2850 50  0000 C CNN
+F 0 "D2" H 9500 2850 50  0000 C CNN
 F 1 "1N4148" H 9500 2750 50  0000 C CNN
 F 2 "Diodes_SMD:D_1206" H 9500 2650 50  0001 C CNN
@@
 $EndComp
 $Comp
-L C C4
+L C C7
 U 1 1 5A579830
 P 10000 3150
-F 0 "C4" H 10025 3250 50  0000 L CNN
+F 0 "C7" H 10025 3250 50  0000 L CNN
 F 1 "0,1" H 10025 3050 50  0000 L CNN
 F 2 "Capacitors_SMD:C_0805_HandSoldering" H 10038 3000 50  0001 C CNN
@@
 L R R9
 U 1 1 5A579A7D
-P 9700 2250
-F 0 "R9" V 9500 2250 50  0000 C CNN
-F 1 "5k6" V 9600 2250 50  0000 C CNN
-F 2 "Resistors_SMD:R_0805_HandSoldering" V 9630 2250 50  0001 C CNN
-F 3 "" H 9700 2250 50  0001 C CNN
-	1    9700 2250
+P 9900 2250
+F 0 "R9" V 9700 2250 50  0000 C CNN
+F 1 "5k6" V 9800 2250 50  0000 C CNN
+F 2 "Resistors_SMD:R_0805_HandSoldering" V 9830 2250 50  0001 C CNN
+F 3 "" H 9900 2250 50  0001 C CNN
+	1    9900 2250
 	-1   0    0    1
 $EndComp
@@
 L GND #PWR010
 U 1 1 5A579B51
-P 9700 2400
-F 0 "#PWR010" H 9700 2150 50  0001 C CNN
-F 1 "GND" H 9700 2250 50  0000 C CNN
-F 2 "" H 9700 2400 50  0001 C CNN
-F 3 "" H 9700 2400 50  0001 C CNN
-	1    9700 2400
-	1    0    0    -1
-$EndComp
-$Comp
-L LED_Dual_CAC D2
-U 1 1 5A579B98
-P 9600 1800
-F 0 "D2" H 9600 2025 50  0000 C CNN
-F 1 "LED_Dual_CAC" H 9600 1550 50  0000 C CNN
-F 2 "LEDs:LED_D8.0mm-3" H 9650 1800 50  0001 C CNN
-F 3 "" H 9650 1800 50  0001 C CNN
-	1    9600 1800
-	0    1    1    0
+P 9900 2400
+F 0 "#PWR010" H 9900 2150 50  0001 C CNN
+F 1 "GND" H 9900 2250 50  0000 C CNN
+F 2 "" H 9900 2400 50  0001 C CNN
+F 3 "" H 9900 2400 50  0001 C CNN
+	1    9900 2400
+	1    0    0    -1
 $EndComp
 $Comp
@@
 F 0 "J7" H 10800 3200 50  0000 C CNN
 F 1 "Pwr/Out" H 10800 2800 50  0000 C CNN
-F 2 "TerminalBlocks_Phoenix:TerminalBlock_Phoenix_MKDS1.5-3pol" H 10800 3000 50  0001 C CNN
+F 2 "Connectors_Terminal_Blocks:TerminalBlock_Altech_AK300-3_P5.00mm" H 10800 3000 50  0001 C CNN
 F 3 "" H 10800 3000 50  0001 C CNN
 	1    10800 3000
@@
 F 0 "C5" H 7225 3400 50  0000 L CNN
 F 1 "10,0" H 7225 3200 50  0000 L CNN
-F 2 "Capacitors_Tantalum_SMD:CP_Tantalum_Case-B_EIA-3528-21_Hand" H 7238 3150 50  0001 C CNN
+F 2 "Capacitors_Tantalum_SMD:CP_Tantalum_Case-A_EIA-3216-18_Hand" H 7238 3150 50  0001 C CNN
 F 3 "" H 7200 3300 50  0001 C CNN
 	1    7200 3300
@@
 F 0 "U3" H 8900 1450 50  0000 C CNN
 F 1 "74HC74" H 9050 855 50  0000 C CNN
-F 2 "Housings_DIP:DIP-14_W7.62mm" H 8750 1150 50  0001 C CNN
+F 2 "Housings_SOIC:SOIC-14_3.9x8.7mm_Pitch1.27mm" H 8750 1150 50  0001 C CNN
 F 3 "" H 8750 1150 50  0001 C CNN
 	2    8750 1150
@@
 	7500 600  7500 1400
 Wire Wire Line
-	8750 1700 8350 1700
-Wire Wire Line
-	8350 1700 8350 600
-Connection ~ 8350 600
-Wire Wire Line
-	8150 950  8150 700
-Wire Wire Line
-	8150 700  9450 700
-Wire Wire Line
-	9450 700  9450 1350
-Wire Wire Line
-	9450 1350 9350 1350
-Wire Wire Line
-	8100 1150 8150 1150
-Connection ~ 8100 1750
+	8150 1700 8750 1700
 $Comp
 L VCC #PWR018
@@
 	6950 3150 7200 3150
 $Comp
-L C C6
+L C C1
 U 1 1 5A57C71D
 P 1550 1100
-F 0 "C6" H 1575 1200 50  0000 L CNN
+F 0 "C1" H 1575 1200 50  0000 L CNN
 F 1 "0,1" H 1575 1000 50  0000 L CNN
 F 2 "Capacitors_SMD:C_0805_HandSoldering" H 1588 950 50  0001 C CNN
@@
 $EndComp
 $Comp
-L C C7
+L C C8
 U 1 1 5A57CB5F
 P 10750 2700
-F 0 "C7" H 10775 2800 50  0000 L CNN
+F 0 "C8" H 10775 2800 50  0000 L CNN
 F 1 "0,1" H 10775 2600 50  0000 L CNN
 F 2 "Capacitors_SMD:C_0805_HandSoldering" H 10788 2550 50  0001 C CNN
@@
 $EndComp
 $Comp
-L C C?
+L C C4
 U 1 1 5A5F5345
 P 6000 2350
-F 0 "C?" H 6025 2450 50  0000 L CNN
-F 1 "10pF" H 6025 2250 50  0000 L CNN
+F 0 "C4" H 6025 2450 50  0000 L CNN
+F 1 "4,7pF" H 6025 2250 50  0000 L CNN
 F 2 "Capacitors_SMD:C_0805_HandSoldering" H 6038 2200 50  0001 C CNN
 F 3 "" H 6000 2350 50  0001 C CNN
@@
 $EndComp
 $Comp
-L GND #PWR?
+L GND #PWR021
 U 1 1 5A5F53D1
 P 6000 2500
-F 0 "#PWR?" H 6000 2250 50  0001 C CNN
+F 0 "#PWR021" H 6000 2250 50  0001 C CNN
 F 1 "GND" H 6000 2350 50  0000 C CNN
 F 2 "" H 6000 2500 50  0001 C CNN
@@
 $EndComp
 Connection ~ 6000 2200
+Wire Wire Line
+	8100 1850 8100 1750
+Wire Wire Line
+	8150 600  8150 1700
+Connection ~ 8150 1150
+Connection ~ 8150 600
+Connection ~ 8150 950
+$Comp
+L LED D1
+U 1 1 5A5F8987
+P 9500 1950
+F 0 "D1" H 9500 2050 50  0000 C CNN
+F 1 "LED" H 9500 1850 50  0000 C CNN
+F 2 "LEDs:LED_1206_HandSoldering" H 9500 1950 50  0001 C CNN
+F 3 "" H 9500 1950 50  0000 C CNN
+	1    9500 1950
+	0    -1   -1   0
+$EndComp
+$Comp
+L LED D4
+U 1 1 5A5F8B5C
+P 9900 1950
+F 0 "D4" H 9900 2050 50  0000 C CNN
+F 1 "LED" H 9900 1850 50  0000 C CNN
+F 2 "LEDs:LED_1206_HandSoldering" H 9900 1950 50  0001 C CNN
+F 3 "" H 9900 1950 50  0000 C CNN
+	1    9900 1950
+	0    -1   -1   0
+$EndComp
+Wire Wire Line
+	9500 1800 9500 1500
+Wire Wire Line
+	9500 1500 9900 1500
+Wire Wire Line
+	9900 1500 9900 1800
+Connection ~ 9600 1500
+$Comp
+L PZT2222A Q1
+U 1 1 5A5F8CA7
+P 9400 3200
+F 0 "Q1" H 9600 3275 50  0000 L CNN
+F 1 "2N2222" H 9600 3200 50  0000 L CNN
+F 2 "TO_SOT_Packages_SMD:SOT-23_Handsoldering" H 9600 3125 50  0000 L CIN
+F 3 "" H 9400 3200 50  0000 L CNN
+	1    9400 3200
+	1    0    0    -1
+$EndComp
+$Comp
+L D D5
+U 1 1 5A5F8E01
+P 10200 2850
+F 0 "D5" H 10200 2950 50  0000 C CNN
+F 1 "D" H 10200 2750 50  0000 C CNN
+F 2 "Diodes_SMD:D_PowerDI-123" H 10200 2850 50  0001 C CNN
+F 3 "" H 10200 2850 50  0000 C CNN
+	1    10200 2850
+	0    1    1    0
+$EndComp
+Connection ~ 10200 3000
+$Comp
+L CONN_01X01 P1
+U 1 1 5A5F8EB6
+P 10600 2000
+F 0 "P1" H 10600 2100 50  0000 C CNN
+F 1 "Prot. Diode" V 10700 2000 50  0000 C CNN
+F 2 "Pin_Headers:Pin_Header_Straight_1x01_Pitch2.54mm" H 10600 2000 50  0001 C CNN
+F 3 "" H 10600 2000 50  0000 C CNN
+	1    10600 2000
+	1    0    0    -1
+$EndComp
+Wire Wire Line
+	10200 2700 10200 2000
+Wire Wire Line
+	10200 2000 10400 2000
+NoConn ~ 9350 1350
+Wire Wire Line
+	6900 1500 6900 1600
+Wire Wire Line
+	6900 2200 6900 2050
+Wire Wire Line
+	6900 2050 6850 2050
+Wire Wire Line
+	6850 2050 6850 1750
+Wire Wire Line
+	6850 1750 6900 1750
+Wire Wire Line
+	6900 1950 6800 1950
+Wire Wire Line
+	6800 1950 6800 1600
+Wire Wire Line
+	6800 1600 6900 1600
 $EndSCHEMATC

Commit message: template
Parts:
- removed Q1: 2N2222, TO_SOT_Packages_SMD:SOT-23_Handsoldering, symbol PZT2222A
- added Q1: 2N2222, TO_SOT_Packages_SMD:SOT-23_Handsoldering, symbol 2N3055
- D1: value LED -> Out
- D4: value LED -> Pwr
- D5: value D -> 1N4148
Connections:
- net GND: now also Q1.2 (E)
- net at R7.1: now also Q1.1 (B)
- net at D2.1 (K), D3.1 (K): now also Q1.3 (C)
Changed lines of the file:
@@
 P 9500 1950
 F 0 "D1" H 9500 2050 50  0000 C CNN
-F 1 "LED" H 9500 1850 50  0000 C CNN
+F 1 "Out" H 9500 1850 50  0000 C CNN
 F 2 "LEDs:LED_1206_HandSoldering" H 9500 1950 50  0001 C CNN
 F 3 "" H 9500 1950 50  0000 C CNN
@@
 P 9900 1950
 F 0 "D4" H 9900 2050 50  0000 C CNN
-F 1 "LED" H 9900 1850 50  0000 C CNN
+F 1 "Pwr" H 9900 1850 50  0000 C CNN
 F 2 "LEDs:LED_1206_HandSoldering" H 9900 1950 50  0001 C CNN
 F 3 "" H 9900 1950 50  0000 C CNN
@@
 Connection ~ 9600 1500
 $Comp
-L PZT2222A Q1
-U 1 1 5A5F8CA7
-P 9400 3200
-F 0 "Q1" H 9600 3275 50  0000 L CNN
-F 1 "2N2222" H 9600 3200 50  0000 L CNN
-F 2 "TO_SOT_Packages_SMD:SOT-23_Handsoldering" H 9600 3125 50  0000 L CIN
-F 3 "" H 9400 3200 50  0000 L CNN
-	1    9400 3200
-	1    0    0    -1
-$EndComp
-$Comp
 L D D5
 U 1 1 5A5F8E01
 P 10200 2850
-F 0 "D5" H 10200 2950 50  0000 C CNN
-F 1 "D" H 10200 2750 50  0000 C CNN
+F 0 "D5" H 10250 2750 50  0000 C CNN
+F 1 "1N4148" H 10000 2750 50  0000 C CNN
 F 2 "Diodes_SMD:D_PowerDI-123" H 10200 2850 50  0001 C CNN
 F 3 "" H 10200 2850 50  0000 C CNN
@@
 Wire Wire Line
 	6800 1600 6900 1600
+$Comp
+L 2N3055 Q1
+U 1 1 5AD1BD32
+P 9400 3200
+F 0 "Q1" H 9600 3275 50  0000 L CNN
+F 1 "2N2222" H 9600 3200 50  0000 L CNN
+F 2 "TO_SOT_Packages_SMD:SOT-23_Handsoldering" H 9600 3125 50  0001 L CIN
+F 3 "" H 9400 3200 50  0001 L CNN
+	1    9400 3200
+	1    0    0    -1
+$EndComp
 $EndSCHEMATC
