File: mmnet_base/mmnet_base_00.kicad_pcb (KiCad board)
At the start: 2 copper layers, 66 x 76.2 mm, 52 parts, among them J1 24V, J2 RS485, J3 Ext_IO_0, J4 Ext_IO_1, J5 Ai0-1, J6 Ai2-3, J7 1Wire, P1 VR+In, P10 Extension, P11 JTAG/AnalogExt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

Commit message: template
Parts:
- added REF**: MountingHole_3.2mm_M3, Mounting_Holes:MountingHole_3.2mm_M3, F.Cu at (163.8, 49.5)
- added REF**: MountingHole_3.2mm_M3, Mounting_Holes:MountingHole_3.2mm_M3, F.Cu at (110.5, 48.3)
- added REF**: MountingHole_3.2mm_M3, Mounting_Holes:MountingHole_3.2mm_M3, F.Cu at (110.5, 125.7)
- added REF**: MountingHole_3.2mm_M3, Mounting_Holes:MountingHole_3.2mm_M3, F.Cu at (163.8, 125.7)
- moved D5 9.92 mm to (142.2, 45.7)
- moved D6 9.92 mm to (149.9, 45.7)
- moved D4 9.16 mm to (120.7, 45.7)
- moved D3 9.16 mm to (123.2, 45.7)
Routing:
- net +5V: track 245.5 -> 255.8 mm
- net GND: track 290.3 -> 300.1 mm
- net Net-(D6-Pad1): track 71.8 -> 80.5 mm
- net Net-(D4-Pad2): track 27.7 -> 32.1 mm
- net Net-(D3-Pad2): track 13.8 -> 16.3 mm
- net Net-(D5-Pad1): track 12.5 -> 14.5 mm
- added copper zone on F.Cu, net GND
Other:
- board size 66 x 76.2 mm -> 66 x 90.2 mm
