File: pi_adc_rtc_etc/pi_adc_rtc_etc.kicad_pcb (KiCad board)
At the start: 2 copper layers, 85 x 56 mm, 51 parts, among them J1 Power, J2 Ir_IO, J3 Twi0, J4 Twi1, J5 Serial_CO2, M1 dcdc5v, P1 CONN_13X2, P10 Ai0, P11 Ai1, P12 Ai2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

Commit message: template
Parts:
- C5: footprint Capacitors_THT:CP_Radial_D10.0mm_P2.50mm -> Capacitors_THT:CP_Radial_D10.0mm_P5.00mm
- D1: value D -> SS34; footprint Diodes_SMD:D_MELF_Handsoldering -> Diodes_SMD:D_MiniMELF_Handsoldering
- U2: value DS1307N+ -> DS1307
Routing:
- net GND: track 361.8 -> 359.3 mm
Other:
- rule pad_to_mask_clearance: 0 -> 0.2
