File: ss_relay/ss_relay.sch (KiCad schematic (older format))
At the start: 26 parts, among them J1 DC Load, J2 AC220, P1 CONN_01X02, Q1 IRF730, U1 PC817

Commit message: template
Parts:
- Q1: symbol IRF540N -> IRF540N-RESCUE-ss_relay
Changed lines of the file:
@@
 EESchema Schematic File Version 2
+LIBS:ss_relay-rescue
 LIBS:power
 LIBS:device
@@
 $EndComp
 $Comp
-L IRF540N Q1
+L IRF540N-RESCUE-ss_relay Q1
 U 1 1 59EF955B
 P 4300 2400
