File: step_up/step_up.sch (KiCad schematic (older format))
At the start: 30 parts, among them J1 Screw_Terminal_1x03, Q1 kt503, Q2 IRFR024, U1 74HC04, U2 LM2903

Commit message: template
Parts:
- removed C2, C5: 10,0, Capacitors_SMD:c_elec_5x5.7, symbol CP
- removed C6, C7: 0,1, Capacitors_SMD:C_1206_HandSoldering, symbol C
- removed D1: 3v3, Diodes_THT:Diode_DO-41_SOD81_Vertical_AnodeUp, symbol D_Zener
- removed Q1: kt503, TO_SOT_Packages_THT:TO-92_Inline_Narrow_Oval, symbol Q_NPN_CBE
- added C1, C16, C17, C8: 0,1, Capacitors_SMD:C_1206_HandSoldering, symbol C
- added C12, C13: 0,33, Capacitors_SMD:C_1206_HandSoldering, symbol C
- added C15: 10,0, Capacitors_SMD:CP_Elec_4x5.3, symbol CP
- added C2: 1,0, Capacitors_SMD:C_1206_HandSoldering, symbol C
- added C3: 47,0, SMD_Packages:SMD-2112_Pol, symbol CP
- added R11: 3,3k, Resistors_SMD:R_1206_HandSoldering, symbol R
- added R7: 200k, Resistors_SMD:R_1206_HandSoldering, symbol R
- added RV1: 50k, Potentiometers:Potentiometer_Trimmer_Bourns_3296W, symbol POT_TRIM
- added U3: L78L33_TO92, TO_SOT_Packages_THT:TO-92_Inline_Narrow_Oval, symbol L78L33_TO92
- C11: value 47,0 -> 10,0; footprint SMD_Packages:SMD-2112_Pol -> Capacitors_SMD:CP_Elec_4x5.3
- C7: renamed from C3; value 1000 -> 1n
- C9: value 1,0 -> 0,1
- D1: renamed from D2; footprint Diodes_THT:Diode_P600_Vertical_AnodeUp -> Diodes_SMD:D_3220
- J1: value Screw_Terminal_1x03 -> Power; footprint Connectors_Terminal_Blocks:TerminalBlock_Pheonix_MPT-2.54mm_3pol -> Connectors_Terminal_Blocks:TerminalBlock_bornier-3_P5.08mm
- L1: footprint Choke_Toroid_ThroughHole:Choke_Toroid_horizontal_Diameter9mm_Amidon-T30 -> Choke_Toroid_ThroughHole:Choke_Toroid_8x16mm_Vertical
- Q1: renamed from Q2; footprint (none) -> TO_SOT_Packages_SMD:TO-252-3_TabPin2
- R10: renamed from R3; value 390 -> 1,5k
- R4: value 390 -> 0,1; footprint Resistors_SMD:R_1206_HandSoldering -> Resistors_SMD:R_2512_HandSoldering
- R8: value 470 -> 1k
- RV2: renamed from RV1; footprint Potentiometers:Potentiometer_Trimmer-Suntan-TSR-3386C -> Potentiometers:Potentiometer_Trimmer_Bourns_3296W
- renumbered C4 to C10, C1 to C14, C8 to C4, C10 to C5, C12 to C6, R7 to R1, R1 to R2, R2 to R3, R9 to R6, R6 to R9
Connections:
- net +3V3: now also C11.2, C12.1, C16.1, C17.1, R7.1, U3.1 (VO); no longer R6.2, U1.5, U2.8 (V+)
- net GND: now also C11.1, C9.2, R4.1, C1.2, C12.2, C13.2, C15.2, C16.2, C17.2, C2.2, C3.2, C8.1, R11.2, RV1.1, U3.2 (GND); no longer C11.2, C9.1, Q1.3 (S), R4.2, R8.2, U2.4 (V-), U2.5 (+)
- net at R1.1: now also U1.9, U2.1, U2.7; no longer U1.11
- net at R1.2: now also U1.6; no longer U1.8
- net at C7.1, U1.4: now also U1.5; no longer U1.9
- net +2V5: now reaches C14.1, R10.2, R5.2
- net +2V5: now also C15.1, R11.1; no longer R4.1
- net at Q1.2 (G): now also U1.10, U1.12; no longer U1.12
- net at R8.1: now also RV1.2
- net at R6.1: now also Q1.3 (S), R4.2; no longer U2.6 (_)
- net +6vBatt renamed +6V
- net +6V: now also C1.1, C13.1, C2.1, C3.1, U3.3 (VI); no longer C11.1, C9.2
- new net: U1.11, U1.13, U1.8
- new net: C9.1, R8.2, U2.5 (+)
- new net: C8.2, R6.2, U2.6 (_)
- new net: R7.2, RV1.3
- no-connect marks 2 -> 0
Other:
- moved on the sheet: C14, R10, R5, R6, U1C, U1D, U2B
