File: wall_board/wall_board_00.sch (KiCad schematic (older format))
At the start: 55 parts, among them J1 Di, J2 1WireExt, J3 +24, P1 Buttons 0-3, P2 CONN_01X20, P3 CONN_01X20, P4 Enc, P5 LCD2004, P6 LCD LED -, P7 2401 1W serial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

Commit message: template
Parts:
- removed P8: Reg5V, symbol CONN_01X04
- added M1: dcdc5v, dz_lib:dcdc5v, symbol dcdc5v
- C1, C2, C3, C4: footprint (none) -> Capacitors_SMD:C_1206_HandSoldering
- C5: value CP -> 470,0; footprint (none) -> Capacitors_THT:CP_Radial_D22.0mm_P10.00mm_SnapIn
- D1, D10, D2, D3, D4, D7, D8, D9: footprint (none) -> LEDs:LED_1206_HandSoldering
- D11, D12, D13, D5, D6: footprint (none) -> Diodes_SMD:D_1206
- F1: footprint (none) -> SMD_Packages:Fuse_SMD
- J1, J2: footprint (none) -> Connectors_Terminal_Blocks:TerminalBlock_bornier-3_P5.08mm
- J3: footprint (none) -> Connectors_Terminal_Blocks:TerminalBlock_bornier-2_P5.08mm
- L1, L2: footprint (none) -> Relays_THT:Relay_SPDT_OMRON-G5LE-1
- P1: footprint (none) -> Pin_Headers:Pin_Header_Straight_1x05_Pitch2.54mm
- P2, P3: footprint (none) -> Socket_Strips:Socket_Strip_Straight_1x20_Pitch2.54mm
- P4: footprint (none) -> Pin_Headers:Pin_Header_Straight_1x04_Pitch2.54mm
- P5: footprint (none) -> Socket_Strips:Socket_Strip_Straight_1x16_Pitch2.54mm
- P6: footprint (none) -> Pin_Headers:Pin_Header_Straight_1x01_Pitch2.54mm
- P7: footprint (none) -> Pin_Headers:Pin_Header_Straight_1x03_Pitch2.54mm
- Q1, Q2, Q3: footprint TO-92 -> TO_SOT_Packages_THT:TO-92_Inline_Narrow_Oval
- R1, R10, R11, R12, R13, R14, R15, R16, R2, R3, R4, R5, R6, R7, R8, R9: footprint (none) -> Resistors_SMD:R_1206_HandSoldering
- R17: value R -> 4,7k; footprint (none) -> Resistors_SMD:R_1206_HandSoldering
- RV1: footprint (none) -> Potentiometers:Potentiometer_Trimmer_Bourns_3339H_Horizontal
- RV2, RV3: footprint (none) -> Varistors:RV_Disc_D12_W3.9_P7.5
Connections:
- net +5V: now also M1.3 (+5_Out)
- net GND: now also M1.1 (GND_In), M1.4 (GND_Out)
- net at C5.1, D13.1 (K): now also M1.2 (Pwr_In)
