File: _Sensors/capacity_sensor_smd/capacity_sensor.kicad_pcb (KiCad board)
At the start: 2 copper layers, 41.9 x 45.7 mm, 39 parts, among them J1 TP1, J2 Sensor, J3 TP2, J4 TP3, J6 TP4, J7 Pwr/Out, P1 Prot. Diode, Q1 2N2222, U1 ICM7555, U2 74HCT14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

Commit message: update
Parts:
- removed P1: Prot. Diode, Pin_Headers:Pin_Header_Straight_1x01_Pitch2.54mm
- removed hole (x4): hole, Mounting_Holes:MountingHole_3.2mm_M3
- added C10: 0,1, Capacitors_SMD:C_0805_HandSoldering, B.Cu at (151.9, 117.1)
- added C11: 10,0, Capacitors_Tantalum_SMD:CP_Tantalum_Case-A_EIA-3216-18_Hand, B.Cu at (140.4, 101.6)
- added C12: 0,33, Capacitors_SMD:C_0805_HandSoldering, B.Cu at (137.8, 104.1)
- added C13: 0,33, Capacitors_SMD:C_0805_HandSoldering, B.Cu at (137.8, 111.1)
- added C9: 0,1, Capacitors_SMD:C_0805_HandSoldering, B.Cu at (145.5, 91.4)
- added JP1: Jumper_NO_Small, Jumper:SolderJumper-2_P1.3mm_Open_TrianglePad1.0x1.5mm, B.Cu at (133.3, 104.9)
- added MH1: MountingHole, MountingHole:MountingHole_3.2mm_M3, F.Cu at (157.5, 87.6)
- added MH2: MountingHole, MountingHole:MountingHole_3.2mm_M3, F.Cu at (123.2, 125.7)
- added MH3: MountingHole, MountingHole:MountingHole_3.2mm_M3, F.Cu at (157.5, 125.7)
- added MH4: MountingHole, MountingHole:MountingHole_3.2mm_M3, F.Cu at (123.2, 87.6)
- added R11: 200, Resistors_SMD:R_2512_HandSoldering, B.Cu at (147.2, 95.2)
- added U4: L78L05_SOT89, TO_SOT_Packages_SMD:SOT89-3_Housing, B.Cu at (138.4, 107.5)
- moved D5 10.8 mm to (146.1, 100.3), turned to 270 degrees
- moved C1 4.58 mm to (139.7, 117.3)
Connections:
- D5 pad 1: Net-(D5-Pad1) -> +24V
- J7 pad 1: +5V -> +24V
- U1 pad 4: (no net) -> Net-(U1-Pad4)
- U1 pad 5: (no net) -> Net-(U1-Pad5)
- U3 pad 5: (no net) -> Net-(U3-Pad5)
- U3 pad 8: (no net) -> Net-(U3-Pad8)
- U3 pad 9: (no net) -> Net-(U3-Pad9)
Routing:
- net GND: track 188.5 -> 242.1 mm
- net Net-(C11-Pad1): track 0.00 -> 17.3 mm
- net +24V: track 0.00 -> 10.9 mm
- net Net-(C7-Pad1): track 19.5 -> 9.82 mm
- net Net-(D5-Pad1): track 4.51 -> 0.00 mm
- net +5V: track 108.7 -> 111.5 mm, vias 3 -> 4
