File: _Sensors/capacity_sensor_smd/capacity_sensor.sch (KiCad schematic (older format))
At the start: 35 parts, among them J1 TP1, J2 Sensor, J3 TP2, J4 TP3, J6 TP4, J7 Pwr/Out, P1 Prot. Diode, Q1 2N2222, U1 ICM7555, U2 74HCT14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

Commit message: update
Parts:
- removed P1: Prot. Diode, Pin_Headers:Pin_Header_Straight_1x01_Pitch2.54mm, symbol capacity_sensor-rescue:CONN_01X01
- added C10, C9: 0,1, Capacitors_SMD:C_0805_HandSoldering, symbol Device:C
- added C11: 10,0, Capacitors_Tantalum_SMD:CP_Tantalum_Case-A_EIA-3216-18_Hand, symbol Device:CP
- added C12, C13: 0,33, Capacitors_SMD:C_0805_HandSoldering, symbol Device:C
- added JP1: Jumper_NO_Small, Jumper:SolderJumper-2_P1.3mm_Open_TrianglePad1.0x1.5mm, symbol Device:Jumper_NO_Small
- added MH1, MH2, MH3, MH4: MountingHole, MountingHole:MountingHole_3.2mm_M3, symbol Mechanical:MountingHole
- added R11: 200, Resistors_SMD:R_2512_HandSoldering, symbol Device:R
- added U4: L78L05_SOT89, TO_SOT_Packages_SMD:SOT89-3_Housing, symbol regul:L78L05_SOT89
Connections:
- net labels added: +24V
- wire segments 55 -> 73
