File: _Modular/dz_ChorusDelSol/classic_mod.kicad_sch (KiCad schematic)
At the start: 79 parts, among them J1 Fast Depth 10k, J10 Modulator Out, J13 Power, J2 Fast Freq 1m, J3 Slow Depth 10k, J4 Slow Freq 1m, U1 LM2902, U2 LM2902, U3 LM2902

Commit message: update
Parts:
- C1, C10, C2, C3, C4, C5, C6, C7, C9: footprint (none) -> Capacitor_SMD:C_0805_2012Metric_Pad1.18x1.45mm_HandSolder
- C11, C14, C98, C99: footprint (none) -> Capacitor_SMD:C_Elec_6.3x5.8
- C12, C13, C15, C16, C17, C18, C19, C20, C21, C8: footprint (none) -> Capacitor_SMD:C_1206_3216Metric_Pad1.33x1.80mm_HandSolder
- D1, D2, D3: footprint (none) -> Diode_SMD:D_MiniMELF_Handsoldering
- J1, J13, J2, J3, J4, JP7: footprint (none) -> Connector_PinHeader_2.54mm:PinHeader_1x03_P2.54mm_Vertical
- J10: footprint (none) -> Connector_PinHeader_2.54mm:PinHeader_1x05_P2.54mm_Vertical
- R1, R10, R11, R12, R13, R14, R15, R16, R17, R18, R19, R2, R20, R21, R22, R23, R24, R25, R26, R27, R28, R29, R3, R30, R31, R32, R33, R34, R35, R36, R37, R38, R39, R4, R40, R41, R42, R5, R6, R7, R8, R9: footprint (none) -> Resistor_SMD:R_1206_3216Metric_Pad1.30x1.75mm_HandSolder
- RV1: footprint (none) -> Potentiometer_THT:Potentiometer_Runtron_RM-065_Vertical
- U1, U2, U3: footprint (none) -> Package_DIP:DIP-14_W7.62mm
