File: _Modular/dz_ChorusDelSol/dz_ChorusDelSol.kicad_sch (KiCad schematic)
At the start: 1 part

Commit message: update
Parts:
- JP1: footprint (none) -> Connector_PinHeader_2.54mm:PinHeader_1x03_P2.54mm_Vertical
Other:
- sheet Preamp ports: added none; removed BBD Drive, Dry
