File: _Modular/dz_ChorusDelSol/mixer.kicad_sch (KiCad schematic)
At the start: 119 parts, among them J11 20k, J12 20k, J14 10k, J15 L Out, J16 L In, J17 R Out, J18 R In, J19 A Out, J20 20k, J21 C Out, J22 Dry LMR In, J23 Phase ABC Out, J24 Power, J27 B Out, J28 Wet Out, U6 LM2904, U7 LM2902, U8 LM2902, U9 LM2904

Commit message: update
Parts:
- removed J15: L Out, symbol Connector:AudioJack3
- removed J16: L In, symbol Connector:AudioJack3
- removed J17: R Out, symbol Connector:AudioJack3
- removed J18: R In, symbol Connector:AudioJack3
- removed J19: A Out, symbol Connector:AudioJack3
- removed J21: C Out, symbol Connector:AudioJack3
- removed J27: B Out, symbol Connector:AudioJack3
- removed J28: Wet Out, symbol Connector:AudioJack3
- added J15: L Out, Connector_Audio:Jack_6.35mm_Neutrik_NMJ6HCD2_Horizontal, symbol Connector:AudioJack3_Switch
- added J16: L/Mono In, Connector_Audio:Jack_6.35mm_Neutrik_NMJ6HCD2_Horizontal, symbol Connector:AudioJack3_Switch
- added J17: R Out, Connector_Audio:Jack_6.35mm_Neutrik_NMJ6HCD2_Horizontal, symbol Connector:AudioJack3_Switch
- added J18: R In, Connector_Audio:Jack_6.35mm_Neutrik_NMJ6HCD2_Horizontal, symbol Connector:AudioJack3_Switch
- added J19: A Out, Connector_Audio:Jack_6.35mm_Neutrik_NMJ6HCD2_Horizontal, symbol Connector:AudioJack3_Switch
- added J21: C Out, Connector_Audio:Jack_6.35mm_Neutrik_NMJ6HCD2_Horizontal, symbol Connector:AudioJack3_Switch
- added J27: B Out, Connector_Audio:Jack_6.35mm_Neutrik_NMJ6HCD2_Horizontal, symbol Connector:AudioJack3_Switch
- added J28: Wet Out, Connector_Audio:Jack_6.35mm_Neutrik_NMJ6HCD2_Horizontal, symbol Connector:AudioJack3_Switch
- C54, C55, C58, C59, C62, C63, C66, C67, C75, C76, C78, C79, C80, C81, C84, C85, C86, C87, C88, C92, C93, C94, C95, C96: footprint (none) -> Capacitor_SMD:C_1206_3216Metric_Pad1.33x1.80mm_HandSolder
- C56, C57, C65, C69, C70, C71, C72, C82, C90: footprint (none) -> Capacitor_SMD:C_0805_2012Metric_Pad1.18x1.45mm_HandSolder
- C60, C61, C64, C68, C83, C89, C91: footprint (none) -> Capacitor_THT:C_Disc_D5.0mm_W2.5mm_P2.50mm
- C73, C74, C77: footprint (none) -> Capacitor_SMD:C_Elec_6.3x5.8
- J11, J12, J14, J20, J24, JP2, JP5: footprint (none) -> Connector_PinHeader_2.54mm:PinHeader_1x03_P2.54mm_Vertical
- J22, J23: footprint (none) -> Connector_PinHeader_2.54mm:PinHeader_1x05_P2.54mm_Vertical
- JP3, JP4: footprint (none) -> Connector_PinHeader_2.54mm:PinHeader_1x02_P2.54mm_Vertical
- R100, R101, R102, R105, R106, R113, R114, R115, R116, R117, R118, R119, R120, R121, R122, R123, R124, R125, R126, R127, R128, R129, R130, R50, R53, R70, R72, R74, R75, R76, R77, R78, R79, R80, R81, R82, R83, R84, R85, R86, R87, R88, R89, R90, R91, R92, R93, R94, R95, R96, R97, R98, R99: footprint (none) -> Resistor_SMD:R_1206_3216Metric_Pad1.30x1.75mm_HandSolder
- U6, U9: footprint (none) -> Package_DIP:DIP-8_W7.62mm
- U7, U8: footprint (none) -> Package_DIP:DIP-14_W7.62mm
Connections:
- net GND: now also J15.S, J16.R, J16.RN, J16.S, J16.SN, J16.TN, J17.S, J18.R, J18.RN, J18.S, J18.SN, J19.S, J21.S, J27.S, J28.S
- net at R101.2: now also J27.R
- net at R53.2: now also J21.T
- net at R72.2: now also J21.R
- net at R91.2: now also J17.T
- net at C82.2, R119.2: now also J16.T, J18.TN
- net at C90.2, R127.2: now also J18.T
- net at R99.2: now also J27.T
- net at R100.2: now also J28.T
- net at R102.2: now also J28.R
- net at R70.2: now also J19.R
- net at R93.2: now also J17.R
- net at R77.2: now also J15.T
- net at R81.2: now also J15.R
- net at R50.2: now also J19.T
- no-connect marks 0 -> 18
Other:
- moved on the sheet: R101, R102, R70, R72, R81, R93
