File: _Modular/dz_ChorusDelSol/power.kicad_sch (KiCad schematic)
At the start: 0 parts

Commit message: update
Parts:
- added C121: 2200x25v, Capacitor_THT:CP_Radial_D13.0mm_P5.00mm, symbol Device:C_Polarized
- added C122: 470x25v, Capacitor_THT:CP_Radial_D13.0mm_P5.00mm, symbol Device:C_Polarized
- added C123, C124: 0,33, Capacitor_SMD:C_0805_2012Metric_Pad1.18x1.45mm_HandSolder, symbol Device:C
- added D12: D, Diode_SMD:D_SMA-SMB_Universal_Handsoldering, symbol Device:D
- added D13: LED, LED_SMD:LED_1206_3216Metric_Pad1.42x1.75mm_HandSolder, symbol Device:LED
- added D14: MB6S, Diode_SMD:Diode_Bridge_OnSemi_SDIP-4L, symbol Device:D_Bridge_+-AA
- added F1: Fuse, Fuse:Fuseholder_Clip-5x20mm_Keystone_3512_Inline_P23.62x7.27mm_D1.02x1.57mm_Horizontal, symbol Device:Fuse
- added J33, J34, J35, J36, J37, J38: Power, Connector_PinHeader_2.54mm:PinHeader_1x03_P2.54mm_Vertical, symbol Connector:Conn_01x03_Male
- added JP13: GND Polarity, Connector_PinHeader_2.54mm:PinHeader_1x03_P2.54mm_Vertical, symbol Jumper:Jumper_3_Bridged12
- added R144: 10k, Resistor_SMD:R_1206_3216Metric_Pad1.30x1.75mm_HandSolder, symbol Device:R
- added R145, R146: 15, Resistor_THT:R_Axial_Power_L20.0mm_W6.4mm_P30.48mm, symbol Device:R
- added TP10, TP11: Power Switch, TestPoint:TestPoint_THTPad_2.0x2.0mm_Drill1.0mm, symbol Connector:TestPoint
- added TP12, TP8: Trans 220, TestPoint:TestPoint_THTPad_2.0x2.0mm_Drill1.0mm, symbol Connector:TestPoint
- added TP3, TP4: Trans Low, TestPoint:TestPoint_THTPad_2.0x2.0mm_Drill1.0mm, symbol Connector:TestPoint
- added TP5, TP6: Trans Conn, TestPoint:TestPoint_THTPad_2.0x2.0mm_Drill1.0mm, symbol Connector:TestPoint
- added TP7, TP9: Mains, TestPoint:TestPoint_THTPad_2.0x2.0mm_Drill1.0mm, symbol Connector:TestPoint
- added U14: L7815, Package_TO_SOT_THT:TO-220-3_Vertical, symbol Regulator_Linear:L7815
Connections:
- new net: TP5.1, TP6.1
- new net: C124.1, D12.2 (A), J33.1 (Pin_1), J34.1 (Pin_1), J35.1 (Pin_1), J36.1 (Pin_1), J37.1 (Pin_1), J38.1 (Pin_1), JP13.3 (B), R144.2, U14.3 (OUT)
- new net: J33.2 (Pin_2), J34.2 (Pin_2), J35.2 (Pin_2), J36.2 (Pin_2), J37.2 (Pin_2), J38.2 (Pin_2), JP13.2 (C)
- new net: C121.2, C122.2, C123.2, C124.2, D13.1 (K), D14.2 (-), J33.3 (Pin_3), J34.3 (Pin_3), J35.3 (Pin_3), J36.3 (Pin_3), J37.3 (Pin_3), J38.3 (Pin_3), JP13.1 (A), U14.2 (GND)
- new net: D13.2 (A), R144.1
- new net: D14.1 (+), R145.1
- new net: D14.3, TP3.1
- new net: D14.4, TP4.1
- new net: TP11.1, TP12.1
- new net: C122.1, C123.1, D12.1 (K), R146.2, U14.1 (IN)
- new net: TP10.1, TP9.1
- new net: C121.1, R145.2, R146.1
- new net: F1.2, TP8.1
- new net: F1.1, TP7.1
