File: _Modular/dz_ChorusDelSol/preamp.kicad_sch (KiCad schematic)
At the start: 75 parts, among them J25 Dry LMR In, J26 Power, J5 Filter Switch, J6 BBD Drive, J7 Eq Pot 10k, J8 Eq Pot 10k, J9 Eq Pot 10k, U10 MCP601-xP, U4 LM2904, U5 LM2902

Commit message: update
Parts:
- C22, C26, C27, C34, C47, C48, C49, C51, C52, C97: footprint (none) -> Capacitor_SMD:C_1206_3216Metric_Pad1.33x1.80mm_HandSolder
- C23, C25, C43, C44: footprint (none) -> Capacitor_THT:C_Disc_D5.0mm_W2.5mm_P2.50mm
- C24, C28, C29, C30, C31, C32, C35, C36, C37, C38, C39, C40, C41, C42, C45: footprint (none) -> Capacitor_SMD:C_0805_2012Metric_Pad1.18x1.45mm_HandSolder
- C33, C46, C50, C53: footprint (none) -> Capacitor_SMD:C_Elec_6.3x5.8
- J25: footprint (none) -> Connector_PinHeader_2.54mm:PinHeader_1x05_P2.54mm_Vertical
- J26, J6, J7, J8, J9, JP6: footprint (none) -> Connector_PinHeader_2.54mm:PinHeader_1x03_P2.54mm_Vertical
- J5: footprint (none) -> Connector_PinHeader_2.54mm:PinHeader_1x06_P2.54mm_Vertical
- R43, R44, R45, R46, R47, R48, R49, R51, R52, R54, R55, R56, R57, R58, R59, R60, R61, R62, R63, R64, R65, R66, R67, R68, R69, R71, R73: footprint (none) -> Resistor_SMD:R_1206_3216Metric_Pad1.30x1.75mm_HandSolder
- RV2, RV3, RV4, RV5: footprint (none) -> Potentiometer_THT:Potentiometer_Runtron_RM-065_Vertical
- U4: footprint (none) -> Package_DIP:DIP-8_W7.62mm
- U5: footprint (none) -> Package_DIP:DIP-14_W7.62mm
