File: _Modular/dz_ChorusDelSol/voice.kicad_sch (KiCad schematic)
At the start: 72 parts

Commit message: update
Parts:
- C100, C102, C103, C107, C108, C109: renamed from C?; footprint (none) -> Capacitor_THT:C_Disc_D5.0mm_W2.5mm_P2.50mm
- C101, C110, C117, C119: renamed from C?; footprint (none) -> Capacitor_SMD:C_Elec_6.3x5.8
- C104, C105, C106, C112, C113: renamed from C?; footprint (none) -> Capacitor_SMD:C_1206_3216Metric_Pad1.33x1.80mm_HandSolder
- C111, C114, C115, C116, C118, C120: renamed from C?; footprint (none) -> Capacitor_SMD:C_0805_2012Metric_Pad1.18x1.45mm_HandSolder
- D10, D8, D9: renamed from D?; footprint (none) -> Diode_THT:D_5W_P12.70mm_Horizontal
- D11, D4, D5, D6, D7: renamed from D?; footprint (none) -> Diode_SMD:D_MiniMELF_Handsoldering
- J29, J30, J31: renamed from J?; footprint (none) -> Connector_PinHeader_2.54mm:PinHeader_1x02_P2.54mm_Vertical
- J32: renamed from J?; footprint (none) -> Connector_PinHeader_2.54mm:PinHeader_1x03_P2.54mm_Vertical
- JP10, JP11, JP12, JP8, JP9: renamed from JP?; footprint (none) -> Connector_PinHeader_2.54mm:PinHeader_1x03_P2.54mm_Vertical
- L1, L2: renamed from L?; footprint (none) -> Inductor_THT:L_Radial_D10.0mm_P5.00mm_Fastron_07P
- Q1, Q2: renamed from Q?; footprint (none) -> Package_TO_SOT_THT:TO-92
- R103, R104, R107, R108, R109, R110, R111, R112, R131, R132, R133, R134, R135, R136, R137, R138, R139, R140, R141, R142, R143: renamed from R?; footprint (none) -> Resistor_SMD:R_1206_3216Metric_Pad1.30x1.75mm_HandSolder
- TP1, TP2: renamed from TP?; footprint (none) -> Connector_PinHeader_2.54mm:PinHeader_1x01_P2.54mm_Vertical
- U11: renamed from U?; footprint (none) -> Package_DIP:DIP-14_W7.62mm
- U12: renamed from U?; footprint (none) -> Package_DIP:DIP-8_W7.62mm
- gave numbers to parts that had none: 1
