File: _Modular/dz_ChorusDelSol_modules_1.1/DelSol_Mixer.kicad_sch (KiCad schematic)
At the start: 124 parts, among them J1 L Out, J10 A Out, J11 C Out, J12 B Out, J13 Wet Out, J14 Phase ABC Out, J15 Power, J2 Dry LMR In, J3 20k, J4 20k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

Commit message: headph amp, level meter
Parts:
- removed C27: 0,1, Capacitor_SMD:C_1206_3216Metric_Pad1.33x1.80mm_HandSolder, symbol Device:C
- removed C33, C38: 100,0, Capacitor_SMD:C_Elec_6.3x5.8, symbol Device:C
- added C27, C33: 47,0 25v, Capacitor_THT:CP_Radial_D5.0mm_P2.50mm, symbol Device:C_Polarized
- added J16: ModPower, Connector_PinHeader_2.54mm:PinHeader_2x05_P2.54mm_Vertical, symbol Connector_Generic:Conn_02x05_Odd_Even
- added J17: Out, Connector_PinHeader_2.54mm:PinHeader_1x03_P2.54mm_Vertical, symbol Connector:Conn_01x03_Male
- C12, C13, C14, C15, C18, C19, C2, C3, C4, C5, C7, C8: value 20,0 -> 10,0
- C32: footprint Capacitor_SMD:C_Elec_6.3x5.8 -> Capacitor_SMD:C_0805_2012Metric_Pad1.18x1.45mm_HandSolder
- J3, J4, J7, J8: value 20k -> 50k
Connections:
- net +15V: now also J16.1 (Pin_1), J16.2 (Pin_2)
- net -15V: now also J16.10 (Pin_10), J16.9 (Pin_9)
- net GND: now also C27.2, C33.1, J16.3 (Pin_3), J16.4 (Pin_4), J16.5 (Pin_5), J16.6 (Pin_6), J16.7 (Pin_7), J16.8 (Pin_8), J17.2 (Pin_2)
- net V+: now also C27.1
- net V-: now also C33.2
- net Out R: now reaches C20.2, R20.1, R23.2, U2.1
- net Out R: now also J17.1 (Pin_1)
- net Out L: now reaches C9.2, R5.1, R8.2, U2.7
- net Out L: now also J17.3 (Pin_3)
