File: _Modular/dz_ChorusDelSol_modules_1.1/DelSol_Mixer.kicad_pcb (KiCad board)
At the start: 2 copper layers, 254 x 55.9 mm, 124 parts, among them J1 L Out, J10 A Out, J11 C Out, J12 B Out, J13 Wet Out, J14 Phase ABC Out, J15 Power, J2 Dry LMR In, J3 20k, J4 20k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

Commit message: headph amp, level meter
Parts:
- removed C38: 100,0, Capacitor_SMD:C_Elec_6.3x5.8
- added J16: ModPower, Connector_PinHeader_2.54mm:PinHeader_2x05_P2.54mm_Vertical, F.Cu at (259.1, 49.5)
- added J17: Out, Connector_PinHeader_2.54mm:PinHeader_1x03_P2.54mm_Vertical, F.Cu at (189.9, 39.4)
- C12, C13, C14, C15, C18, C19, C2, C3, C4, C5, C7, C8: value 20,0 -> 10,0
- C16, C20, C6, C9: value 30p -> 15p
- C27: value 0,1 -> 47,0 25v; footprint Capacitor_SMD:C_1206_3216Metric_Pad1.33x1.80mm_HandSolder -> Capacitor_THT:CP_Radial_D5.0mm_P2.50mm; moved to F.Cu
- C32: footprint Capacitor_SMD:C_Elec_6.3x5.8 -> Capacitor_SMD:C_0805_2012Metric_Pad1.18x1.45mm_HandSolder; moved to B.Cu
- C33: value 100,0 -> 47,0 25v; footprint Capacitor_SMD:C_Elec_6.3x5.8 -> Capacitor_THT:CP_Radial_D5.0mm_P2.50mm
- C44: value 30p -> 33p
- J3, J4, J7, J8: value 20k -> 50k
- moved C27 225.1 mm to (252.7, 40.1), turned to -90 degrees
- moved C32 24.4 mm to (237.5, 44.5), turned to 180 degrees
- moved C43 18.6 mm to (238.1, 48.3)
- moved R53 15.9 mm to (244.5, 47.0), turned to 180 degrees
- moved C1 11.8 mm to (34.3, 51.4), turned to 180 degrees
- moved C33 11.1 mm to (261.0, 40.0)
- moved R51 10.0 mm to (244.5, 43.8), turned to 180 degrees
- moved R35 7.75 mm to (171.4, 36.2)
- moved R41 6.02 mm to (145.4, 36.2)
- moved R34 6.02 mm to (22.2, 23.5)
- moved C10 5.85 mm to (49.5, 29.8)
- moved R15 5.85 mm to (49.5, 24.8)
- moved C21 4.84 mm to (22.2, 29.8)
- moved R16 4.75 mm to (211.5, 26.7)
- moved R1 4.58 mm to (236.2, 26.7)
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Connections:
- net Net-(C20-Pad2) renamed /Out R
- net Net-(C9-Pad2) renamed /Out L
- C27 pad 1: GND -> /V+
- C27 pad 2: /1/2 -> GND
- C33 pad 1: /V+ -> GND
- C33 pad 2: GND -> /V-
Routing:
- net GND: track 721.7 -> 649.2 mm, vias 4 -> 5
- net /1/2: track 492.7 -> 448.8 mm, vias 11 -> 8
- net /Out L: track 19.3 -> 58.5 mm, vias 0 -> 1
- net -15V: track 11.1 -> 49.0 mm
- net /Dry L: track 300.2 -> 271.9 mm, vias 5 -> 6
- net +15V: track 11.1 -> 37.1 mm
- net /Out R: track 17.1 -> 38.8 mm, vias 0 -> 2
- net /V-: track 445.2 -> 458.8 mm, vias 10 -> 9
- net /V+: track 422.0 -> 411.4 mm
- net Net-(R35-Pad1): track 100.6 -> 110.3 mm
- net Net-(R41-Pad1): track 64.3 -> 71.7 mm
- net Net-(C10-Pad2): track 15.2 -> 20.8 mm
- net Net-(C21-Pad2): track 5.99 -> 11.4 mm
- net Net-(J12-PadT): track 2.38 -> 6.32 mm
- net Net-(J10-PadR): track 3.09 -> 6.90 mm
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Other:
- board size 254 x 55.9 mm -> 254 x 54 mm
- board text added: "Out"
- board text added: "Power"
