File: _Modular/dz_ChorusDelSol_modules_1.1/DelSol_Preamp.kicad_sch (KiCad schematic)
At the start: 79 parts, among them J1 Filter Switch, J2 BBD Drive, J3 Dry LMR In, J4 Eq Pot 10k, J5 Eq Pot 10k, J6 Eq Pot 10k, J7 Power, U1 LM2904, U2 MCP601-xP, U3 LM2902

Commit message: up
Parts:
- removed C12: 0,1, Capacitor_SMD:C_1206_3216Metric_Pad1.33x1.80mm_HandSolder, symbol Device:C
- removed J2: BBD Drive, Connector_PinHeader_2.54mm:PinHeader_1x03_P2.54mm_Vertical, symbol Connector:Conn_01x03_Male
- added J2: BBD Drive, Connector_JST:JST_XH_B5B-XH-AM_1x05_P2.50mm_Vertical, symbol Connector:Conn_01x05_Male
- C11: value 47,0 -> 10,0; footprint Capacitor_SMD:C_Elec_6.3x5.8 -> Capacitor_SMD:C_0805_2012Metric_Pad1.18x1.45mm_HandSolder
- C17: value 47n -> 47
- C21, C22: footprint Capacitor_THT:C_Disc_D5.0mm_W2.5mm_P2.50mm -> Capacitor_SMD:C_0805_2012Metric_Pad1.18x1.45mm_HandSolder
- J3: footprint Connector_PinHeader_2.54mm:PinHeader_1x05_P2.54mm_Vertical -> Connector_JST:JST_XH_B5B-XH-AM_1x05_P2.50mm_Vertical
- J4, J5, J6: footprint Connector_PinHeader_2.54mm:PinHeader_1x03_P2.54mm_Vertical -> Potentiometer_THT:Potentiometer_Alps_RK097_Single_Horizontal
- RV3: footprint Potentiometer_THT:Potentiometer_Runtron_RM-065_Vertical -> Potentiometer_THT:Potentiometer_Bourns_3296W_Vertical
- U2: value MCP601-xP -> TL071
Connections:
- net GND: now also J2.1 (Pin_1), J2.5 (Pin_5)
- net at C6.1, R4.2, U2.6: now also J2.2 (Pin_2), J2.3 (Pin_3), J2.4 (Pin_4)
Other:
- moved on the sheet: R1, R2
