File: _Modular/dz_Distortion_1U/dz_Distortion_Main.kicad_sch (KiCad schematic)
At the start: 112 parts, among them J1 ModPower, J10 Inst In', J11 In, J12 In', J2 Heater Pwr, J3 Heater, J4 Anode, J5 Anode Pwr, J6 Heater', J7 Chan Switch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

Commit message: footpr
Parts:
- added D22, D23: LL4148, Diode_SMD:D_MiniMELF, symbol Diode:LL4148
- C10, C15, C17, C20, C21, C22, C24, C9: footprint (none) -> Capacitor_SMD:C_0805_2012Metric_Pad1.18x1.45mm_HandSolder
- C11, C6: footprint (none) -> Capacitor_THT:CP_Radial_D13.0mm_P5.00mm
- C12, C7: footprint (none) -> Capacitor_THT:C_Rect_L7.0mm_W3.5mm_P5.00mm
- C13, C18, C8: footprint (none) -> Capacitor_THT:C_Disc_D5.0mm_W2.5mm_P2.50mm
- C14, C16, C26, C27, C3, C4, C5: footprint (none) -> Capacitor_SMD:C_1206_3216Metric_Pad1.33x1.80mm_HandSolder
- C19: footprint (none) -> Capacitor_THT:CP_Radial_D10.0mm_P2.50mm_P5.00mm
- C23, C25, U4: footprint (none) -> Capacitor_THT:CP_Radial_D22.0mm_P10.00mm_SnapIn
- D1, D20, D6: footprint (none) -> LED_SMD:LED_1206_3216Metric_Pad1.42x1.75mm_HandSolder
- D7: footprint (none) -> LED_THT:LED_D3.0mm
- J10, J2, J3, J4, J5, J6, J7, J9: footprint (none) -> Connector_PinHeader_2.54mm:PinHeader_1x02_P2.54mm_Vertical
- J11, J12: footprint (none) -> Connector_PinHeader_2.54mm:PinHeader_1x05_P2.54mm_Vertical
- J8: footprint (none) -> Connector_PinHeader_2.54mm:PinHeader_1x01_P2.54mm_Vertical
- L1, L2: footprint (none) -> Inductor_THT:L_Radial_D10.0mm_P5.00mm_Fastron_07M
- Q1: footprint (none) -> Package_TO_SOT_THT:TO-92
- Q2: footprint (none) -> Package_TO_SOT_THT:TO-220-3_Vertical
- R12, R3, R5, R9: footprint Resistor_SMD:R_1206_3216Metric_Pad1.30x1.75mm_HandSolder -> Resistor_THT:R_Axial_DIN0309_L9.0mm_D3.2mm_P5.08mm_Vertical
- R13, R17, R22, R23, R24, R28, R31, R6, R7, R8: footprint Resistor_SMD:R_1206_3216Metric_Pad1.30x1.75mm_HandSolder -> Resistor_THT:R_Axial_DIN0309_L9.0mm_D3.2mm_P12.70mm_Horizontal
- RV1, RV2, RV3, RV4, RV5, RV6, RV8: footprint (none) -> Potentiometer_THT:Potentiometer_Runtron_RM-065_Vertical
- RV7: footprint (none) -> Connector_PinHeader_2.54mm:PinHeader_1x03_P2.54mm_Vertical
- SW1: footprint (none) -> Connector_PinHeader_2.54mm:PinHeader_1x04_P2.54mm_Vertical
- U1: footprint (none) -> Package_DIP:DIP-8_W7.62mm_LongPads
Connections:
- net +15V: now also D23.1 (K)
- net GND: now also D22.2 (A)
- net at C12.1, RV4.1: now also D22.1 (K), D23.2 (A)

Commit message: separate power pcb
Parts:
- U2: footprint Valve:Valve_Noval_P -> Valve:Valve_ECC-83-2
Changed lines of the file:
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@@
       (effects (font (size 1.27 1.27)) (justify left))
     )
-    (property "Footprint" "Valve:Valve_Noval_P" (id 2) (at 187.198 146.05 0)
+    (property "Footprint" "Valve:Valve_ECC-83-2" (id 2) (at 187.198 146.05 0)
       (effects (font (size 1.27 1.27)) hide)
     )
@@
       (effects (font (size 1.27 1.27)) (justify left))
     )
-    (property "Footprint" "Valve:Valve_Noval_P" (id 2) (at 217.678 146.05 0)
+    (property "Footprint" "Valve:Valve_ECC-83-2" (id 2) (at 217.678 146.05 0)
       (effects (font (size 1.27 1.27)) hide)
     )
@@
       (effects (font (size 1.27 1.27)) (justify left))
     )
-    (property "Footprint" "Valve:Valve_Noval_P" (id 2) (at 264.668 134.62 0)
+    (property "Footprint" "Valve:Valve_ECC-83-2" (id 2) (at 264.668 134.62 0)
       (effects (font (size 1.27 1.27)) hide)
     )
@@
     )
     (path "/48b0637a-c3e9-4cb0-b347-c41bded4a332"
-      (reference "U2") (unit 1) (value "ECC88") (footprint "Valve:Valve_Noval_P")
+      (reference "U2") (unit 1) (value "ECC88") (footprint "Valve:Valve_ECC-83-2")
     )
     (path "/a2064ccf-0679-42a2-9a40-149226a0a3d3"
-      (reference "U2") (unit 2) (value "ECC88") (footprint "Valve:Valve_Noval_P")
+      (reference "U2") (unit 2) (value "ECC88") (footprint "Valve:Valve_ECC-83-2")
     )
     (path "/ff1f60f5-a872-466d-b582-6faafd6c1452"
-      (reference "U2") (unit 3) (value "ECC88") (footprint "Valve:Valve_Noval_P")
+      (reference "U2") (unit 3) (value "ECC88") (footprint "Valve:Valve_ECC-83-2")
     )
     (path "/821b83e5-9401-447e-a583-42ebefdc5367"

Commit message: up
Parts:
- removed C17: 1000, Capacitor_SMD:C_0805_2012Metric_Pad1.18x1.45mm_HandSolder, symbol Device:C
- removed C19: 100,0, Capacitor_THT:CP_Radial_D10.0mm_P2.50mm_P5.00mm, symbol Device:C_Polarized
- removed C20: 22n, Capacitor_SMD:C_0805_2012Metric_Pad1.18x1.45mm_HandSolder, symbol Device:C
- removed C21, C22, C24: 4,7, Capacitor_SMD:C_0805_2012Metric_Pad1.18x1.45mm_HandSolder, symbol Device:C
- removed C23, C25: 100,0 x 450v, Capacitor_THT:CP_Radial_D22.0mm_P10.00mm_SnapIn, symbol Device:C_Polarized
- removed D14: КД641Е, Package_TO_SOT_THT:TO-220-2_Vertical, symbol Device:D_Schottky
- removed D18: 1N4148, Diode_THT:D_DO-35_SOD27_P7.62mm_Horizontal, symbol Diode:1N4148
- removed D20: LED, LED_SMD:LED_1206_3216Metric_Pad1.42x1.75mm_HandSolder, symbol Device:LED
- removed D23: LL4148, Diode_SMD:D_MiniMELF, symbol Diode:LL4148
- removed J2: Heater Pwr, Connector_PinHeader_2.54mm:PinHeader_1x02_P2.54mm_Vertical, symbol Connector:Conn_01x02_Male
- removed J5: Anode Pwr, Connector_PinHeader_2.54mm:PinHeader_1x02_P2.54mm_Vertical, symbol Connector:Conn_01x02_Male
- removed J6: Heater', Connector_PinHeader_2.54mm:PinHeader_1x02_P2.54mm_Vertical, symbol Connector:Conn_01x02_Male
- removed L1: 680uH, Inductor_THT:L_Radial_D10.0mm_P5.00mm_Fastron_07M, symbol Device:L_Ferrite
- removed L2: 50uH, Inductor_THT:L_Radial_D10.0mm_P5.00mm_Fastron_07M, symbol Device:L_Ferrite
- removed Q1: KT3107, Package_TO_SOT_THT:TO-92, symbol Device:Q_PNP_CBE
- removed Q2: IRF830, Package_TO_SOT_THT:TO-220-3_Vertical, symbol Device:Q_NMOS_GDS
- removed R22: 0,47 2w, Resistor_THT:R_Axial_DIN0309_L9.0mm_D3.2mm_P12.70mm_Horizontal, symbol Device:R
- removed R23, R24: 510k, Resistor_THT:R_Axial_DIN0309_L9.0mm_D3.2mm_P12.70mm_Horizontal, symbol Device:R
- removed R27: 1k, Resistor_SMD:R_1206_3216Metric_Pad1.30x1.75mm_HandSolder, symbol Device:R
- removed R28, R31: 100k 1w, Resistor_THT:R_Axial_DIN0309_L9.0mm_D3.2mm_P12.70mm_Horizontal, symbol Device:R
- removed R29: 47, Resistor_SMD:R_1206_3216Metric_Pad1.30x1.75mm_HandSolder, symbol Device:R
- removed RV8: 10k, Potentiometer_THT:Potentiometer_Runtron_RM-065_Vertical, symbol Device:R_Potentiometer_Trim
- removed U3: MC34063AP, Package_DIP:DIP-8_W7.62mm, symbol Regulator_Switching:MC34063AP
- added H1, H2, H3, H4: MountingHole, MountingHole:MountingHole_3.2mm_M3, symbol Mechanical:MountingHole
- D22: value LL4148 -> Z 5v6
- J4: value Anode -> Anode +300v
- SW1: value SW_SP3T -> Mode
- U4: footprint Capacitor_THT:CP_Radial_D22.0mm_P10.00mm_SnapIn -> Package_DIP:DIP-8_W7.62mm
Connections:
- net GND: now also RV5.3; no longer RV5.1
- net at R14.1, SW1.3: now also RV5.1; no longer RV5.3
- net VCC: now reaches C1.1, C26.2, C3.2, R1.2, U1.8 (V+), U4.8 (V+)
Other:
- note removed: "C19 was 4700 - why?"
- note removed: "Originally P4NK60Z is used"
- moved on the sheet: D22
