File: _Modular/dz_Distortion_1U/dz_Distortion_Main.kicad_pcb (KiCad board)
At the start: 2 copper layers, 114 parts, among them J1 ModPower, J10 Inst In', J11 In, J12 In', J2 Heater Pwr, J3 Heater, J4 Anode, J5 Anode Pwr, J6 Heater', J7 Chan Switch, J8 Instrument Switch, J9 Inst In, Q1 KT3107, Q2 IRF830, SW1 SW_SP3T, U1 TL072, U2 ECC88, U3 MC34063AP, U4 TL072

Commit message: up
Parts:
- removed C17: 1000, Capacitor_SMD:C_0805_2012Metric_Pad1.18x1.45mm_HandSolder
- removed C19: 100,0, Capacitor_THT:CP_Radial_D10.0mm_P2.50mm_P5.00mm
- removed C20: 22n, Capacitor_SMD:C_0805_2012Metric_Pad1.18x1.45mm_HandSolder
- removed C21, C22, C24: 4,7, Capacitor_SMD:C_0805_2012Metric_Pad1.18x1.45mm_HandSolder
- removed C23, C25: 100,0 x 450v, Capacitor_THT:CP_Radial_D22.0mm_P10.00mm_SnapIn
- removed D14: КД641Е, Package_TO_SOT_THT:TO-220-2_Vertical
- removed D18: 1N4148, Diode_THT:D_DO-35_SOD27_P7.62mm_Horizontal
- removed D20: LED, LED_SMD:LED_1206_3216Metric_Pad1.42x1.75mm_HandSolder
- removed D23: LL4148, Diode_SMD:D_MiniMELF
- removed J2: Heater Pwr, Connector_PinHeader_2.54mm:PinHeader_1x02_P2.54mm_Vertical
- removed J5: Anode Pwr, Connector_PinHeader_2.54mm:PinHeader_1x02_P2.54mm_Vertical
- removed J6: Heater', Connector_PinHeader_2.54mm:PinHeader_1x02_P2.54mm_Vertical
- removed L1: 680uH, Inductor_THT:L_Radial_D10.0mm_P5.00mm_Fastron_07M
- removed L2: 50uH, Inductor_THT:L_Radial_D10.0mm_P5.00mm_Fastron_07M
- removed Q1: KT3107, Package_TO_SOT_THT:TO-92
- removed Q2: IRF830, Package_TO_SOT_THT:TO-220-3_Vertical
- removed R22: 0,47 2w, Resistor_THT:R_Axial_DIN0309_L9.0mm_D3.2mm_P12.70mm_Horizontal
- removed R23, R24: 510k, Resistor_THT:R_Axial_DIN0309_L9.0mm_D3.2mm_P12.70mm_Horizontal
- removed R27: 1k, Resistor_SMD:R_1206_3216Metric_Pad1.30x1.75mm_HandSolder
- removed R28, R31: 100k 1w, Resistor_THT:R_Axial_DIN0309_L9.0mm_D3.2mm_P12.70mm_Horizontal
- removed R29: 47, Resistor_SMD:R_1206_3216Metric_Pad1.30x1.75mm_HandSolder
- removed RV8: 10k, Potentiometer_THT:Potentiometer_Runtron_RM-065_Vertical
- removed U3: MC34063AP, Package_DIP:DIP-8_W7.62mm
- added H1: MountingHole, MountingHole:MountingHole_3.2mm_M3, F.Cu at (134.6, 105.4)
- added H2: MountingHole, MountingHole:MountingHole_3.2mm_M3, F.Cu at (52.1, 105.4)
- added H3: MountingHole, MountingHole:MountingHole_3.2mm_M3, F.Cu at (52.1, 40.6)
- added H4: MountingHole, MountingHole:MountingHole_3.2mm_M3, F.Cu at (134.6, 40.6)
- C10, C15, C26, C27, C3, C4, C5, C9, D1, D15, D16, D17, D19, D2, D21, D3, D4, D5, D6, D8, D9, R1, R10, R11, R14, R15, R16, R18, R19, R2, R20, R21, R25, R26, R30, R32, R4: moved to B.Cu
- D22: value LL4148 -> Z 5v6; moved to B.Cu
- J4: value Anode -> Anode +300v
- SW1: value SW_SP3T -> Mode
- U4: footprint Capacitor_THT:CP_Radial_D22.0mm_P10.00mm_SnapIn -> Package_DIP:DIP-8_W7.62mm
- moved D22 173.0 mm to (51.3, 67.1), turned to 180 degrees
- moved J4 171.2 mm to (60.1, 80.0)
- moved R25 159.5 mm to (74.7, 48.0), turned to 90 degrees
- moved RV6 153.5 mm to (54.6, 52.1), turned to 180 degrees
- moved R11 146.6 mm to (84.1, 59.7)
- moved R16 136.9 mm to (67.3, 73.6), turned to -90 degrees
- moved R30 136.0 mm to (61.2, 48.0), turned to -90 degrees
- moved D6 135.3 mm to (104.1, 61.0), turned to -90 degrees
- moved R4 133.2 mm to (91.2, 59.7), turned to 180 degrees
- moved R18 133.2 mm to (108.9, 73.7)
- moved C27 130.8 mm to (92.7, 44.2), turned to -90 degrees
- moved D12 129.8 mm to (115.6, 69.8), turned to 180 degrees
- moved C4 126.6 mm to (78.7, 78.4), turned to 90 degrees
- moved R26 125.5 mm to (85.1, 44.7), turned to 90 degrees
- moved D4 119.5 mm to (75.7, 57.2)
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Connections:
- C1 pad 1: Net-(C1-Pad1) -> VCC
- C26 pad 2: Net-(C1-Pad1) -> VCC
- C3 pad 2: Net-(C1-Pad1) -> VCC
- R1 pad 2: Net-(C1-Pad1) -> VCC
- RV5 pad 1: GND -> Net-(R14-Pad1)
- RV5 pad 3: Net-(R14-Pad1) -> GND
- U1 pad 8: Net-(C1-Pad1) -> VCC
Routing:
- net GND: track 0.00 -> 405.0 mm
- net +15V: track 0.00 -> 160.9 mm, vias 0 -> 2
- net Net-(C2-Pad2): track 0.00 -> 127.6 mm, vias 0 -> 1
- net VCC: track 0.00 -> 82.3 mm, vias 0 -> 1
- net Net-(C6-Pad1): track 0.00 -> 69.8 mm
- net Net-(R14-Pad1): track 0.00 -> 61.7 mm
- net Net-(C11-Pad1): track 0.00 -> 51.3 mm
- net Net-(D2-Pad1): track 0.00 -> 48.3 mm, vias 0 -> 3
- net /A In: track 0.00 -> 48.0 mm
- net Net-(C12-Pad1): track 0.00 -> 41.8 mm
- net Net-(R3-Pad1): track 0.00 -> 38.3 mm
- net Net-(R8-Pad1): track 0.00 -> 32.3 mm
- net Net-(C15-Pad2): track 0.00 -> 30.4 mm
- net Net-(J10-Pad2): track 0.00 -> 29.1 mm
- net Net-(C12-Pad2): track 0.00 -> 28.5 mm
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Other:
- board outline added: 90.2 x 72.4 mm
- board text added: "Drive"

Commit message: up
Routing:
- net /A In: track 48.0 -> 60.0 mm
- added copper zone on F.Cu, net GND
