File: _Modular/dz_Distortion_1U/dz_Distortion_1U.kicad_sch (KiCad schematic)
At the start: 72 parts, among them J1 Inst In, J10 Compression meter, J2 ModPower, J3 Auto/Line/Inst Sw, J4 Gate off Sw, J5 Guit/Line Relay, J6 Guit/Line Relay, J7 Guit/Line Relay, J8 Guit Clean Out, J9 Comp on/off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

Commit message: up
Parts:
- removed D1, D10, D11, D12, D2, D3, D4, D5, D6, D7, D8, D9: D, symbol Device:D
- added D? (x12): LL4148, Diode_SMD:D_MiniMELF, symbol Diode:LL4148
Connections:
- net +15V: now also D?.1 (K)
- net at U2.1: now also D?.1 (K), D?.2 (A)
- net at C13.2, R18.1, U2.2 (-): now also D?.2 (A)
- net at C16.1, RV7.2: now also D?.2 (A)
- net at R20.2, U2.9 (-): now also D?.1 (K), D?.1 (K)
- net at U2.5 (+), U2.8: now also D?.2 (A), D?.2 (A)
- net at U1.8: now also D?.1 (K)
- net at RV6.1: now also D?.2 (A)
- net at J3.2 (Pin_2), J5.2 (Pin_2), J6.2 (Pin_2)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: now also D?.2 (A)
- net at U2.14: now also D?.1 (K), D?.1 (K), D?.2 (A), D?.2 (A)
- net at C14.1, R18.2, U2.12 (+): now also D?.1 (K)
- net at U2.13 (-): now also D?.1 (K), D?.2 (A)
- net at C10.2, J4.1 (Pin_1), R13.2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: now also D?.2 (A)
- net at RV5.3: now also D?.1 (K)
- net at Q2.2 (G), R16.1: now also D?.1 (K), D?.1 (K)
- net at R13.1: now also D?.2 (A)
