File: _Modular/TapeDelay/dz_TapeDelay_Control.kicad_sch (KiCad schematic)
At the start: 111 parts, among them J1 +20v Unreg, J10 Pinch Solenoid, J11 ModPower, J12 Meter in 1-2, J13 Meter in 3-4, J14 Step Motor 1 Driver, J15 Step Motor 2 Driver, J16 Motor power, J17 Motor power, J18 Erase Head, J19 Gen, J2 OLED, J20 Aux1, J21 Mute, J22 Aux2, J3 DCDC Pwr, J4 DCDC Gnd, J5 DCDC +5, J6 DCDC Gnd, J7 Encoder/Enter/ESC, J8 Transport ctl/leds, J9 AVR-ISP-10, Q1 IRF7303, Q2 KT3107, Q3 KT603A, Q4 KT603A, Q5 MMBT3904, U1 ATmega8-16P, U2 TL064, U3 PCF8574, Y1 8 MHz

Commit message: up
Parts:
- gave numbers to parts that had none: 4
Changed lines of the file:
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@@
   (symbol (lib_id "Mechanical:MountingHole") (at 124.46 178.435 0) (unit 1)
     (in_bom yes) (on_board yes) (fields_autoplaced)
-    (property "Reference" "H?" (id 0) (at 127 177.6003 0)
+    (property "Reference" "H4" (id 0) (at 127 177.6003 0)
       (effects (font (size 1.27 1.27)) (justify left) hide)
     )
@@
   (symbol (lib_id "Mechanical:MountingHole") (at 124.46 173.355 0) (unit 1)
     (in_bom yes) (on_board yes) (fields_autoplaced)
-    (property "Reference" "H?" (id 0) (at 127 172.5203 0)
+    (property "Reference" "H3" (id 0) (at 127 172.5203 0)
       (effects (font (size 1.27 1.27)) (justify left) hide)
     )
@@
   (symbol (lib_id "Mechanical:MountingHole") (at 119.38 178.435 0) (unit 1)
     (in_bom yes) (on_board yes) (fields_autoplaced)
-    (property "Reference" "H?" (id 0) (at 121.92 177.6003 0)
+    (property "Reference" "H2" (id 0) (at 121.92 177.6003 0)
       (effects (font (size 1.27 1.27)) (justify left) hide)
     )
@@
   (symbol (lib_id "Mechanical:MountingHole") (at 119.38 173.355 0) (unit 1)
     (in_bom yes) (on_board yes) (fields_autoplaced)
-    (property "Reference" "H?" (id 0) (at 121.92 172.5203 0)
+    (property "Reference" "H1" (id 0) (at 121.92 172.5203 0)
       (effects (font (size 1.27 1.27)) (justify left) hide)
     )
@@
       (reference "D10") (unit 1) (value "SS34") (footprint "Diode_SMD:D_SMA-SMB_Universal_Handsoldering")
     )
+    (path "/c7203091-36ec-4943-9189-8bc0da9b6f6e"
+      (reference "H1") (unit 1) (value "MountingHole") (footprint "MountingHole:MountingHole_3.2mm_M3")
+    )
+    (path "/a02c2d3a-f9a0-4c0f-8472-523b8dbd678b"
+      (reference "H2") (unit 1) (value "MountingHole") (footprint "MountingHole:MountingHole_3.2mm_M3")
+    )
+    (path "/5b35710d-1a85-4003-9f46-b7929f24b900"
+      (reference "H3") (unit 1) (value "MountingHole") (footprint "MountingHole:MountingHole_3.2mm_M3")
+    )
     (path "/0d28539d-746f-451f-a767-4a526f61e008"
-      (reference "H?") (unit 1) (value "MountingHole") (footprint "MountingHole:MountingHole_3.2mm_M3")
-    )
-    (path "/5b35710d-1a85-4003-9f46-b7929f24b900"
-      (reference "H?") (unit 1) (value "MountingHole") (footprint "MountingHole:MountingHole_3.2mm_M3")
-    )
-    (path "/a02c2d3a-f9a0-4c0f-8472-523b8dbd678b"
-      (reference "H?") (unit 1) (value "MountingHole") (footprint "MountingHole:MountingHole_3.2mm_M3")
-    )
-    (path "/c7203091-36ec-4943-9189-8bc0da9b6f6e"
-      (reference "H?") (unit 1) (value "MountingHole") (footprint "MountingHole:MountingHole_3.2mm_M3")
+      (reference "H4") (unit 1) (value "MountingHole") (footprint "MountingHole:MountingHole_3.2mm_M3")
     )
     (path "/4c3e4926-ace7-442d-bbc1-b3f725dd4262"
