File: _Modular/TapeDelay/dz_TapeDelay_Control.kicad_sch (KiCad schematic)
At the start: 113 parts, among them J1 +20v Unreg, J10 Pinch Solenoid, J11 ModPower, J12 Meter in 1-2, J13 Meter in 3-4, J14 Step Motor 1 Driver, J15 Step Motor 2 Driver, J16 Motor power, J17 Motor power, J18 Erase Head, J19 Gen, J2 OLED, J20 Sens1, J21 Mute, J22 Sens2, J3 DCDC Pwr, J4 DCDC Gnd, J5 DCDC +5, J6 DCDC Gnd, J7 Encoder/Enter/ESC, J8 Transport ctl/leds, J9 AVR-ISP-10, Q1 IRF7303, Q2 KT3107, Q3 KT603A, Q4 KT603A, Q5 MMBT3904, U1 ATmega8-16P, U2 TL064, U3 PCF8574, Y1 8 MHz

Commit message: meter
Parts:
- added C27: 0,1, Capacitor_SMD:C_0805_2012Metric_Pad1.18x1.45mm_HandSolder, symbol Device:C
- C25: value 27 -> 100
- C26: value 0,01 -> 470
Connections:
- net +15V: now also C27.2
- net GND: now also C27.1
Other:
- note added: "~200v 200Khz"
Changed lines of the file:
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@@
   (junction (at 88.9 149.225) (diameter 0) (color 0 0 0 0)
   )
+  (junction (at 58.42 115.57) (diameter 0) (color 0 0 0 0)
+  )
   (junction (at 90.17 193.04) (diameter 0) (color 0 0 0 0)
   )
@@
     (stroke (width 0) (type default) (color 0 0 0 0))
   )
+  (wire (pts (xy 58.42 111.76) (xy 58.42 115.57))
+    (stroke (width 0) (type default) (color 0 0 0 0))
+  )
   (wire (pts (xy 180.975 138.43) (xy 206.375 138.43))
     (stroke (width 0) (type default) (color 0 0 0 0))
@@
     (stroke (width 0) (type default) (color 0 0 0 0))
   )
+  (wire (pts (xy 58.42 115.57) (xy 58.42 117.475))
+    (stroke (width 0) (type default) (color 0 0 0 0))
+  )
   (wire (pts (xy 104.14 78.105) (xy 99.06 78.105))
     (stroke (width 0) (type default) (color 0 0 0 0))
@@
     (stroke (width 0) (type default) (color 0 0 0 0))
   )
+  (text "~200v 200Khz" (at 96.52 154.94 0)
+    (effects (font (size 1.27 1.27)) (justify left bottom))
+  )
   (label "S2" (at 59.69 81.28 0)
     (effects (font (size 1.27 1.27)) (justify left bottom))
@@
     (pin "2")
   )
+  (symbol (lib_id "power:GND") (at 66.04 115.57 90) (unit 1)
+    (in_bom yes) (on_board yes) (fields_autoplaced)
+    (property "Reference" "#PWR0103" (id 0) (at 72.39 115.57 0)
+      (effects (font (size 1.27 1.27)) hide)
+    )
+    (property "Value" "GND" (id 1) (at 69.215 116.0038 90)
+      (effects (font (size 1.27 1.27)) (justify right))
+    )
+    (property "Footprint" "" (id 2) (at 66.04 115.57 0)
+      (effects (font (size 1.27 1.27)) hide)
+    )
+    (property "Datasheet" "" (id 3) (at 66.04 115.57 0)
+      (effects (font (size 1.27 1.27)) hide)
+    )
+    (pin "1")
+  )
   (symbol (lib_id "Device:R") (at 176.53 127 180) (unit 1)
     (in_bom yes) (on_board yes)
@@
     (pin "1")
   )
+  (symbol (lib_id "Device:C") (at 62.23 115.57 270) (unit 1)
+    (in_bom yes) (on_board yes) (fields_autoplaced)
+    (property "Reference" "C27" (id 0) (at 62.23 107.95 90))
+    (property "Value" "0,1" (id 1) (at 62.23 110.49 90))
+    (property "Footprint" "Capacitor_SMD:C_0805_2012Metric_Pad1.18x1.45mm_HandSolder" (id 2) (at 58.42 116.5352 0)
+      (effects (font (size 1.27 1.27)) hide)
+    )
+    (property "Datasheet" "~" (id 3) (at 62.23 115.57 0)
+      (effects (font (size 1.27 1.27)) hide)
+    )
+    (pin "1")
+    (pin "2")
+  )
   (symbol (lib_id "Device:C") (at 24.13 52.07 0) (unit 1)
     (in_bom yes) (on_board yes) (fields_autoplaced)
@@
   (symbol (lib_id "Device:C") (at 88.9 155.575 180) (unit 1)
     (in_bom yes) (on_board yes) (fields_autoplaced)
-    (property "Reference" "C26" (id 0) (at 92.71 154.3049 0)
+    (property "Reference" "C26" (id 0) (at 91.821 154.7403 0)
       (effects (font (size 1.27 1.27)) (justify right))
     )
-    (property "Value" "0,01" (id 1) (at 92.71 156.8449 0)
+    (property "Value" "470" (id 1) (at 91.821 157.2772 0)
       (effects (font (size 1.27 1.27)) (justify right))
     )
@@
       (effects (font (size 1.27 1.27)) (justify right))
     )
-    (property "Value" "27" (id 1) (at 82.55 156.8449 0)
+    (property "Value" "100" (id 1) (at 82.55 156.8449 0)
       (effects (font (size 1.27 1.27)) (justify right))
     )
@@
     (pin "2")
   )
-  (symbol (lib_id "power:+15V") (at 58.42 117.475 0) (unit 1)
+  (symbol (lib_id "power:+15V") (at 58.42 111.76 0) (unit 1)
     (in_bom yes) (on_board yes) (fields_autoplaced)
-    (property "Reference" "#PWR051" (id 0) (at 58.42 121.285 0)
+    (property "Reference" "#PWR051" (id 0) (at 58.42 115.57 0)
       (effects (font (size 1.27 1.27)) hide)
     )
-    (property "Value" "+15V" (id 1) (at 58.42 112.395 0))
-    (property "Footprint" "" (id 2) (at 58.42 117.475 0)
+    (property "Value" "+15V" (id 1) (at 58.42 106.68 0))
+    (property "Footprint" "" (id 2) (at 58.42 111.76 0)
       (effects (font (size 1.27 1.27)) hide)
     )
-    (property "Datasheet" "" (id 3) (at 58.42 117.475 0)
+    (property "Datasheet" "" (id 3) (at 58.42 111.76 0)
       (effects (font (size 1.27 1.27)) hide)
     )
@@
       (reference "#PWR0102") (unit 1) (value "+15V") (footprint "")
     )
+    (path "/215d39d7-14c7-4bc9-8476-9338a88ccff8"
+      (reference "#PWR0103") (unit 1) (value "GND") (footprint "")
+    )
     (path "/a3908678-a5b7-4102-88c1-2baf66da67d4"
       (reference "C1") (unit 1) (value "0,1") (footprint "Capacitor_SMD:C_1206_3216Metric_Pad1.33x1.80mm_HandSolder")
@@
     )
     (path "/9abc5987-15fa-441a-b3b8-3298ac0849e6"
-      (reference "C25") (unit 1) (value "27") (footprint "Capacitor_THT:C_Disc_D5.0mm_W2.5mm_P2.50mm")
+      (reference "C25") (unit 1) (value "100") (footprint "Capacitor_THT:C_Disc_D5.0mm_W2.5mm_P2.50mm")
     )
     (path "/7210febf-af05-4166-911c-319c06d8dd5d"
-      (reference "C26") (unit 1) (value "0,01") (footprint "Capacitor_THT:C_Disc_D5.0mm_W2.5mm_P2.50mm")
+      (reference "C26") (unit 1) (value "470") (footprint "Capacitor_THT:C_Disc_D5.0mm_W2.5mm_P2.50mm")
+    )
+    (path "/410d2f6a-35b3-4522-ba94-1c59fb067927"
+      (reference "C27") (unit 1) (value "0,1") (footprint "Capacitor_SMD:C_0805_2012Metric_Pad1.18x1.45mm_HandSolder")
     )
     (path "/b16ed1ea-881a-4c0c-82ee-0b64e9eefc1c"
