File: _Modular/TapeDelay/_autosave-dz_TapeDelay_Control.kicad_sch (KiCad schematic)
At the start: 113 parts, among them J1 +20v Unreg, J10 Pinch Solenoid, J11 ModPower, J12 Meter in 1-2, J13 Meter in 3-4, J14 Step Motor 1 Driver, J15 Step Motor 2 Driver, J16 Motor power, J17 Motor power, J18 Erase Head, J19 Gen, J2 OLED, J20 Sens1, J21 Mute, J22 Sens2, J3 DCDC Pwr, J4 DCDC Gnd, J5 DCDC +5, J6 DCDC Gnd, J7 Encoder/Enter/ESC, J8 Transport ctl/leds, J9 AVR-ISP-10, Q1 IRF7303, Q2 KT3107, Q3 KT603A, Q4 KT603A, Q5 MMBT3904, U1 ATmega8-16P, U2 TL064, U3 PCF8574, Y1 8 MHz

Commit message: Sensors
Parts:
- gave numbers to parts that had none: 2
Changed lines of the file:
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@@
   (symbol (lib_id "Device:R") (at 138.43 29.21 270) (unit 1)
     (in_bom yes) (on_board yes)
-    (property "Reference" "R?" (id 0) (at 137.795 27.305 0)
+    (property "Reference" "R40" (id 0) (at 137.795 27.305 0)
       (effects (font (size 1.27 1.27)) (justify right))
     )
@@
   (symbol (lib_id "power:+5V") (at 134.62 29.21 90) (mirror x) (unit 1)
     (in_bom yes) (on_board yes)
-    (property "Reference" "#PWR?" (id 0) (at 138.43 29.21 0)
+    (property "Reference" "#PWR053" (id 0) (at 138.43 29.21 0)
       (effects (font (size 1.27 1.27)) hide)
     )
@@
   (symbol (lib_id "Device:R") (at 138.43 35.56 270) (unit 1)
     (in_bom yes) (on_board yes)
-    (property "Reference" "R?" (id 0) (at 137.795 33.655 0)
+    (property "Reference" "R41" (id 0) (at 137.795 33.655 0)
       (effects (font (size 1.27 1.27)) (justify right))
     )
@@
       (reference "#PWR052") (unit 1) (value "GND") (footprint "")
     )
+    (path "/27ed5892-3b55-41c1-ac33-93af08384b6f"
+      (reference "#PWR053") (unit 1) (value "+5V") (footprint "")
+    )
     (path "/7960e7d6-4e1c-4b58-a7c5-b29953fe0b42"
       (reference "#PWR0101") (unit 1) (value "GND") (footprint "")
@@
       (reference "#PWR0102") (unit 1) (value "+15V") (footprint "")
     )
-    (path "/27ed5892-3b55-41c1-ac33-93af08384b6f"
-      (reference "#PWR?") (unit 1) (value "+5V") (footprint "")
-    )
     (path "/a3908678-a5b7-4102-88c1-2baf66da67d4"
       (reference "C1") (unit 1) (value "0,1") (footprint "Capacitor_SMD:C_1206_3216Metric_Pad1.33x1.80mm_HandSolder")
@@
     )
     (path "/1d124c3d-50a1-4b01-9c10-1853aa60cbc7"
-      (reference "R?") (unit 1) (value "47k") (footprint "Resistor_SMD:R_1206_3216Metric_Pad1.30x1.75mm_HandSolder")
+      (reference "R40") (unit 1) (value "47k") (footprint "Resistor_SMD:R_1206_3216Metric_Pad1.30x1.75mm_HandSolder")
     )
     (path "/4e4715dc-36ee-4478-9f0a-8e834ac0c4d9"
-      (reference "R?") (unit 1) (value "47k") (footprint "Resistor_SMD:R_1206_3216Metric_Pad1.30x1.75mm_HandSolder")
+      (reference "R41") (unit 1) (value "47k") (footprint "Resistor_SMD:R_1206_3216Metric_Pad1.30x1.75mm_HandSolder")
     )
     (path "/06fe2f17-3328-45cb-8459-2e8bcbd16b01"
