File: _Modular/TapeDelay/TapeDelay.kicad_pcb (KiCad board)
At the start: 2 copper layers, 108 x 77.5 mm, 138 parts, among them J1 PB Head 1, J10 Meter Sw, J11 Erase Head, J12 Gen, J13 Dry In, J14 50k, J15 Dry In', J16 Out', J17 Out, J18 XMix 1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

Commit message: tape
Parts:
- removed C15, C35: 10,0, Capacitor_SMD:C_0805_2012Metric_Pad1.18x1.45mm_HandSolder
- removed C17, C27: 4,7, Capacitor_SMD:C_0805_2012Metric_Pad1.18x1.45mm_HandSolder
- removed C18, C28: 220,0, Capacitor_THT:CP_Radial_D7.5mm_P2.50mm
- removed C34: 0,1, Capacitor_SMD:C_0805_2012Metric_Pad1.18x1.45mm_HandSolder
- removed C36: 1,0, Capacitor_SMD:C_0805_2012Metric_Pad1.18x1.45mm_HandSolder
- removed C37: 27, Capacitor_THT:C_Disc_D5.0mm_W2.5mm_P2.50mm
- removed C38: 0,01, Capacitor_THT:C_Disc_D5.0mm_W2.5mm_P2.50mm
- removed C53: 47,0, Capacitor_THT:CP_Radial_D6.3mm_P2.50mm
- removed D1, D2: К174УН13, Package_DIP:DIP-16_W7.62mm_LongPads
- removed D3: SS34, Diode_SMD:D_SMA-SMB_Universal_Handsoldering
- removed J12: Gen, Connector_PinHeader_2.54mm:PinHeader_1x02_P2.54mm_Vertical
- removed Q1: KT3107, Package_TO_SOT_THT:TO-92
- removed Q2, Q3: KT603A, Package_TO_SOT_THT:TO-92_Wide
- removed R15, R16, R27, R28: 10k, Resistor_SMD:R_1206_3216Metric_Pad1.30x1.75mm_HandSolder
- removed R17, R29: 120k, Resistor_SMD:R_1206_3216Metric_Pad1.30x1.75mm_HandSolder
- removed R18, R30: 1m, Resistor_SMD:R_1206_3216Metric_Pad1.30x1.75mm_HandSolder
- removed R35, R40: 470, Resistor_SMD:R_1206_3216Metric_Pad1.30x1.75mm_HandSolder
- removed R36, R37: 30k, Resistor_SMD:R_1206_3216Metric_Pad1.30x1.75mm_HandSolder
- removed R38: 10, Resistor_THT:R_Axial_DIN0309_L9.0mm_D3.2mm_P2.54mm_Vertical
- removed R39: 4,3k, Resistor_SMD:R_1206_3216Metric_Pad1.30x1.75mm_HandSolder
- removed R41: 43, Resistor_THT:R_Axial_DIN0309_L9.0mm_D3.2mm_P2.54mm_Vertical
- added U3: L78L12, Package_TO_SOT_THT:TO-92_Inline, F.Cu at (109.2, 28.3)
- added U4: TL072, Package_DIP:DIP-8_W7.62mm_LongPads, F.Cu at (97.8, 70.5)
- J11: value Erase Head -> Gen
- U1: value L78L12_TO92 -> К174УН13; footprint Package_TO_SOT_THT:TO-92_Inline -> Package_DIP:DIP-16_W7.62mm_LongPads
- U2: value TL072 -> К174УН13; footprint Package_DIP:DIP-8_W7.62mm_LongPads -> Package_DIP:DIP-16_W7.62mm_LongPads
- moved U1 54.1 mm to (56.5, 31.8)
- moved J11 48.6 mm to (76.2, 29.2), turned to 90 degrees
- moved U2 38.2 mm to (94.0, 31.8)
- moved C16 25.8 mm to (77.7, 33.0)
- moved TP1 22.9 mm to (68.6, 36.8)
- moved RV1 20.7 mm to (76.8, 37.8), turned to 180 degrees
- moved C29 16.0 mm to (108.0, 35.6)
- moved J8 16.0 mm to (115.6, 35.7)
- moved R31 16.0 mm to (111.8, 37.2)
- moved R32 16.0 mm to (111.8, 44.5)
- moved C30 16.0 mm to (108.0, 43.3)
- moved R13 9.55 mm to (74.3, 43.8), turned to 90 degrees
- moved C14 8.10 mm to (67.4, 43.2)
- moved J16 7.24 mm to (123.8, 59.1)
- moved J17 7.24 mm to (123.8, 54.0)
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Connections:
- J11 pad 1: Net-(D3-Pad2) -> /Gen
- J3 pad 1: Net-(J3-Pad1) -> GND
- J3 pad 2: +12VA -> Net-(C13-Pad1)
- J5 pad 1: Net-(J5-Pad1) -> GND
- J5 pad 2: +12VA -> /PB Mix
- R1 pad 1: Net-(D1-Pad2) -> Net-(U1-Pad2)
- R19 pad 1: Net-(D2-Pad2) -> Net-(U2-Pad2)
- R2 pad 1: Net-(D1-Pad2) -> Net-(U1-Pad2)
- R20 pad 1: Net-(D2-Pad2) -> Net-(U2-Pad2)
- R23 pad 1: Net-(D2-Pad7) -> Net-(U2-Pad7)
- R24 pad 1: Net-(D2-Pad7) -> Net-(U2-Pad7)
- R26 pad 2: Net-(D2-Pad7) -> Net-(U2-Pad7)
- U1 pad 1: +12VA -> Net-(C1-Pad2)
- U1 pad 2: GND -> Net-(U1-Pad2)
- U1 pad 3: Net-(C31-Pad2) -> Net-(C6-Pad1)
- U2 pad 1: Net-(C42-Pad2) -> Net-(C19-Pad2)
- U2 pad 2: Net-(C41-Pad2) -> Net-(U2-Pad2)
- U2 pad 3: GND -> Net-(C25-Pad1)
- U2 pad 4: -15V -> Net-(C21-Pad2)
- U2 pad 6: Net-(C51-Pad1) -> GND
- U2 pad 7: Net-(C51-Pad2) -> Net-(U2-Pad7)
- U2 pad 8: +15V -> Net-(C26-Pad1)
