File: _Modular/TapeDelay/dz_TapeDelay_Control.kicad_pcb (KiCad board)
At the start: 2 copper layers, 106.7 x 58.4 mm, 111 parts, among them J1 +20v Unreg, J10 Pinch Solenoid, J11 ModPower, J12 Meter in 1-2, J13 Meter in 3-4, J14 Step Motor 1 Driver, J15 Step Motor 2 Driver, J16 Motor power, J17 Motor power, J18 Erase Head, J19 Gen, J2 OLED, J20 Aux1, J21 Mute, J22 Aux2, J3 DCDC Pwr, J4 DCDC Gnd, J5 DCDC +5, J6 DCDC Gnd, J7 Encoder/Enter/ESC, J8 Transport ctl/leds, J9 AVR-ISP-10, Q1 IRF7303, Q2 KT3107, Q3 KT603A, Q4 KT603A, Q5 MMBT3904, U1 ATmega8-16P, U2 TL064, U3 PCF8574, Y1 8 MHz

Commit message: pcb
Routing:
- net GND: track 419.9 -> 444.5 mm
Other:
- board text added: "Erase Head"

Commit message: up
Routing:
- added copper zone on F.Cu, net GND
Other:
- board text added: "dz@dz.ru Tape Delay Control Board"

Commit message: Sensors
Parts:
- added R40: 47k, Resistor_SMD:R_1206_3216Metric_Pad1.30x1.75mm_HandSolder, B.Cu at (81.2, 54.6)
- added R41: 47k, Resistor_SMD:R_1206_3216Metric_Pad1.30x1.75mm_HandSolder, B.Cu at (81.3, 67.3)
- J20: value Aux1 -> Sens1
- J22: value Aux2 -> Sens2
Connections:
- net Net-(U1-Pad11) renamed /S2
- net Net-(U1-Pad6) renamed /S1
Routing:
- net +5V: track 176.8 -> 188.7 mm
- net /S2: track 10.1 -> 12.4 mm
- net /S1: track 9.21 -> 11.4 mm
Other:
- board text added: "+"
- board text added: "+5"
- board text added: "-"
- board text added: "A"
- board text added: "B"
- board text added: "Esc"
- board text added: "Gnd"
- board text added: "LEDs"
- board text added: "Ok"
- board text added: "Pause"
- board text added: "Run"
- board text added: "SCL"
- board text added: "SDA"
- board text added: "Stop"

Commit message: meter
Parts:
- added C27: 0,1, Capacitor_SMD:C_0805_2012Metric_Pad1.18x1.45mm_HandSolder, B.Cu at (56.5, 66.0)
- C25: value 27 -> 100
- C26: value 0,01 -> 470
Routing:
- net GND: track 444.5 -> 447.2 mm
- net +15V: track 138.2 -> 139.6 mm
Changed lines of the file:
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@@
       (effects (font (size 1 1) (thickness 0.15)))
     )
-    (fp_text value "0,01" (at 3.79 3.81) (layer "F.Fab")
+    (fp_text value "470" (at 3.79 3.81) (layer "F.Fab")
       (effects (font (size 1 1) (thickness 0.15)))
     )
@@
       (effects (font (size 1 1) (thickness 0.15)))
     )
-    (fp_text value "27" (at 1.25 2.5) (layer "F.Fab")
+    (fp_text value "100" (at 1.25 2.5) (layer "F.Fab")
       (effects (font (size 1 1) (thickness 0.15)))
     )
@@
     )
   )
+  (footprint "Capacitor_SMD:C_0805_2012Metric_Pad1.18x1.45mm_HandSolder" (layer "B.Cu")
+    (at 56.515 66.04 180)
+    (descr "Capacitor SMD 0805 (2012 Metric), square (rectangular) end terminal, IPC_7351 nominal with elongated pad for handsoldering. (Body size source: IPC-SM-782 page 76, https://www.pcb-3d.com/wordpress/wp-content/uploads/ipc-sm-782a_amendment_1_and_2.pdf, https://docs.google.com/spreadsheets/d/1BsfQQcO9C6DZCsRaXUlFlo91Tg2WpOkGARC1WS5S8t0/edit?usp=sharing), generated with kicad-footprint-generator")
+    (tags "capacitor handsolder")
+    (property "Sheetfile" "dz_TapeDelay_Control.kicad_sch")
+    (property "Sheetname" "")
+    (attr smd)
+    (fp_text reference "C27" (at 0 1.68) (layer "B.SilkS")
+      (effects (font (size 1 1) (thickness 0.15)) (justify mirror))
+    )
+    (fp_text value "0,1" (at 0 -1.68) (layer "B.Fab")
+      (effects (font (size 1 1) (thickness 0.15)) (justify mirror))
+    )
+    (fp_text user "${REFERENCE}" (at 0 0) (layer "B.Fab")
+      (effects (font (size 0.5 0.5) (thickness 0.08)) (justify mirror))
+    )
+    (fp_line (start -0.261252 -0.735) (end 0.261252 -0.735) (layer "B.SilkS") (width 0.12))
+    (fp_line (start -0.261252 0.735) (end 0.261252 0.735) (layer "B.SilkS") (width 0.12))
+    (fp_line (start -1.88 -0.98) (end -1.88 0.98) (layer "B.CrtYd") (width 0.05))
+    (fp_line (start 1.88 -0.98) (end -1.88 -0.98) (layer "B.CrtYd") (width 0.05))
+    (fp_line (start -1.88 0.98) (end 1.88 0.98) (layer "B.CrtYd") (width 0.05))
+    (fp_line (start 1.88 0.98) (end 1.88 -0.98) (layer "B.CrtYd") (width 0.05))
+    (fp_line (start -1 -0.625) (end -1 0.625) (layer "B.Fab") (width 0.1))
+    (fp_line (start -1 0.625) (end 1 0.625) (layer "B.Fab") (width 0.1))
+    (fp_line (start 1 -0.625) (end -1 -0.625) (layer "B.Fab") (width 0.1))
+    (fp_line (start 1 0.625) (end 1 -0.625) (layer "B.Fab") (width 0.1))
+    (pad "1" smd roundrect (at -1.0375 0 180) (size 1.175 1.45) (layers "B.Cu" "B.Paste" "B.Mask") (roundrect_rratio 0.212766)
+      (net 1 "GND") (pintype "passive"))
+    (pad "2" smd roundrect (at 1.0375 0 180) (size 1.175 1.45) (layers "B.Cu" "B.Paste" "B.Mask") (roundrect_rratio 0.212766)
+      (net 54 "+15V") (pintype "passive"))
+    (model "${KICAD6_3DMODEL_DIR}/Capacitor_SMD.3dshapes/C_0805_2012Metric.wrl"
+      (offset (xyz 0 0 0))
+      (scale (xyz 1 1 1))
+      (rotate (xyz 0 0 0))
+    )
+  )
   (footprint "Resistor_SMD:R_1206_3216Metric_Pad1.30x1.75mm_HandSolder" (layer "B.Cu")
     (at 127.635 39.66 90)
@@
   (segment (start 52.705 83.185) (end 53.485 82.405) (width 0.25) (layer "B.Cu") (net 1))
   (segment (start 95.25 62.23) (end 102.67 62.23) (width 0.25) (layer "B.Cu") (net 1))
+  (segment (start 58.46 66.04) (end 59.73 64.77) (width 0.25) (layer "B.Cu") (net 1))
   (segment (start 113.65 49.535) (end 111.1575 49.535) (width 0.25) (layer "B.Cu") (net 1))
   (segment (start 125.095 80.01) (end 125.095 77.47) (width 0.25) (layer "B.Cu") (net 1))
@@
   (segment (start 130.805 74.935) (end 130.805 77.475) (width 0.25) (layer "B.Cu") (net 1))
   (segment (start 125.095 77.47) (end 125.095 75.3325) (width 0.25) (layer "B.Cu") (net 1))
+  (segment (start 57.5525 66.04) (end 58.46 66.04) (width 0.25) (layer "B.Cu") (net 1))
   (segment (start 47.979879 61.547379) (end 48.26 61.8275) (width 0.25) (layer "B.Cu") (net 1))
   (segment (start 103.2775 44.455) (end 102.235 45.4975) (width 0.25) (layer "B.Cu") (net 1))
@@
   (segment (start 62.23 85.725) (end 66.04 85.725) (width 0.25) (layer "B.Cu") (net 54))
   (segment (start 135.89 83.06) (end 135.89 72.39) (width 0.25) (layer "B.Cu") (net 54))
-  (segment (start 54.12 63.355) (end 54.12 76.07163) (width 0.25) (layer "B.Cu") (net 54))
+  (segment (start 54.265 66.04) (end 54.12 66.185) (width 0.25) (layer "B.Cu") (net 54))
   (segment (start 130.805 72.395) (end 133.345 72.395) (width 0.25) (layer "B.Cu") (net 54))
   (segment (start 54.12 76.07163) (end 61.017379 82.969009) (width 0.25) (layer "B.Cu") (net 54))
   (segment (start 61.017379 82.969009) (end 61.017379 84.512379) (width 0.25) (layer "B.Cu") (net 54))
+  (segment (start 55.4775 66.04) (end 54.265 66.04) (width 0.25) (layer "B.Cu") (net 54))
   (segment (start 66.04 85.725) (end 66.04 90.17) (width 0.25) (layer "B.Cu") (net 54))
+  (segment (start 54.12 66.185) (end 54.12 76.07163) (width 0.25) (layer "B.Cu") (net 54))
   (segment (start 127.99 75.21) (end 127 75.21) (width 0.25) (layer "B.Cu") (net 54))
   (segment (start 68.455 92.585) (end 126.365 92.585) (width 0.25) (layer "B.Cu") (net 54))
   (segment (start 66.04 90.17) (end 67.31 91.44) (width 0.25) (layer "B.Cu") (net 54))
+  (segment (start 54.12 63.355) (end 54.12 66.185) (width 0.25) (layer "B.Cu") (net 54))
   (segment (start 61.017379 84.512379) (end 62.23 85.725) (width 0.25) (layer "B.Cu") (net 54))
   (segment (start 130.805 72.395) (end 127.99 75.21) (width 0.25) (layer "B.Cu") (net 54))

Commit message: tape
Routing:
- net Net-(Q1-Pad5): track 5.78 -> 9.55 mm
- net Net-(D1-Pad2): track 17.4 -> 20.3 mm
- net +24V: track 84.9 -> 87.6 mm, vias 1 -> 0
- net +15V: track 139.6 -> 137.3 mm
Changed lines of the file:
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@@
   (segment (start 54.54 38.17) (end 81.61 38.17) (width 0.25) (layer "B.Cu") (net 4))
   (segment (start 79.7175 57.15) (end 77.49 57.15) (width 0.25) (layer "B.Cu") (net 4))
-  (segment (start 79.7175 44.4625) (end 79.73 44.45) (width 0.25) (layer "B.Cu") (net 4))
   (segment (start 79.73 44.45) (end 79.73 47.98) (width 0.25) (layer "B.Cu") (net 4))
   (segment (start 109.845 69.215) (end 113.03 69.215) (width 0.25) (layer "B.Cu") (net 4))
@@
   (segment (start 113.65 46.995) (end 111.6775 46.995) (width 0.25) (layer "B.Cu") (net 7))
   (segment (start 111.6775 46.995) (end 111.125 46.4425) (width 0.25) (layer "B.Cu") (net 7))
-  (segment (start 104.14 77.47) (end 123.19 77.47) (width 0.25) (layer "F.Cu") (net 8))
-  (via (at 104.14 77.47) (size 0.8) (drill 0.4) (layers "F.Cu" "B.Cu") (net 8))
-  (segment (start 77.790991 71.12) (end 84.140991 77.47) (width 0.25) (layer "B.Cu") (net 8))
-  (segment (start 65.13 71.12) (end 77.790991 71.12) (width 0.25) (layer "B.Cu") (net 8))
-  (segment (start 84.140991 77.47) (end 104.14 77.47) (width 0.25) (layer "B.Cu") (net 8))
-  (segment (start 62.235 77.47) (end 62.235 74.015) (width 0.25) (layer "B.Cu") (net 8))
-  (segment (start 62.142379 83.185) (end 62.142379 77.562621) (width 0.25) (layer "B.Cu") (net 8))
+  (segment (start 62.142379 83.185) (end 87.63 83.185) (width 2) (layer "F.Cu") (net 8))
+  (segment (start 93.345 77.47) (end 123.19 77.47) (width 2) (layer "F.Cu") (net 8))
+  (segment (start 87.63 83.185) (end 93.345 77.47) (width 2) (layer "F.Cu") (net 8))
+  (segment (start 62.235 77.47) (end 62.235 83.092379) (width 2) (layer "B.Cu") (net 8))
+  (segment (start 62.235 83.092379) (end 62.142379 83.185) (width 2) (layer "B.Cu") (net 8))
+  (segment (start 62.235 77.47) (end 62.235 74.015) (width 2) (layer "B.Cu") (net 8))
   (segment (start 116.84 71.12) (end 116.84 69.215) (width 2) (layer "B.Cu") (net 8))
-  (segment (start 62.142379 77.562621) (end 62.235 77.47) (width 0.25) (layer "B.Cu") (net 8))
-  (segment (start 62.235 74.015) (end 65.13 71.12) (width 0.25) (layer "B.Cu") (net 8))
   (segment (start 123.19 77.47) (end 116.84 71.12) (width 2) (layer "B.Cu") (net 8))
+  (segment (start 62.235 74.015) (end 65.13 71.12) (width 2) (layer "B.Cu") (net 8))
   (segment (start 118.4175 59.705) (end 118.4025 59.69) (width 0.25) (layer "B.Cu") (net 9))
   (segment (start 123.19 59.705) (end 118.4175 59.705) (width 0.25) (layer "B.Cu") (net 9))
@@
   (segment (start 50.165 78.745) (end 50.165 81.285) (width 0.25) (layer "B.Cu") (net 28))
   (segment (start 41.95 81.28) (end 43.075 82.405) (width 0.25) (layer "B.Cu") (net 28))
-  (segment (start 55.245 73.66) (end 59.755 73.66) (width 0.25) (layer "F.Cu") (net 29))
-  (segment (start 59.755 72.39) (end 59.755 73.66) (width 0.25) (layer "F.Cu") (net 29))
-  (segment (start 55.245 73.66) (end 56.79 73.66) (width 0.25) (layer "B.Cu") (net 29))
-  (segment (start 56.79 73.66) (end 59.33 71.12) (width 0.25) (layer "B.Cu") (net 29))
-  (segment (start 59.695 77.47) (end 59.695 71.485) (width 0.25) (layer "B.Cu") (net 29))
-  (segment (start 59.695 71.485) (end 59.33 71.12) (width 0.25) (layer "B.Cu") (net 29))
+  (segment (start 56.515 72.39) (end 55.245 73.66) (width 1) (layer "F.Cu") (net 29))
+  (segment (start 59.755 72.39) (end 56.515 72.39) (width 1) (layer "F.Cu") (net 29))
+  (segment (start 59.755 73.66) (end 55.245 73.66) (width 1) (layer "F.Cu") (net 29))
+  (segment (start 59.695 77.47) (end 59.695 73.655) (width 2) (layer "B.Cu") (net 29))
+  (segment (start 55.445 73.655) (end 55.445 73.66) (width 2) (layer "B.Cu") (net 29))
+  (segment (start 59.695 73.655) (end 55.445 73.655) (width 2) (layer "B.Cu") (net 29))
+  (segment (start 59.695 71.485) (end 59.33 71.12) (width 2) (layer "B.Cu") (net 29))
+  (segment (start 59.695 73.655) (end 59.695 71.485) (width 2) (layer "B.Cu") (net 29))
   (segment (start 102.235 38.33) (end 104.985 38.33) (width 0.25) (layer "B.Cu") (net 30))
   (segment (start 102.015 38.11) (end 102.235 38.33) (width 0.25) (layer "B.Cu") (net 30))
@@
   (via (at 135.89 72.39) (size 0.8) (drill 0.4) (layers "F.Cu" "B.Cu") (net 54))
   (segment (start 67.31 91.44) (end 68.455 92.585) (width 0.25) (layer "B.Cu") (net 54))
+  (segment (start 55.245 66.2725) (end 55.4775 66.04) (width 0.25) (layer "B.Cu") (net 54))
   (segment (start 126.365 92.585) (end 135.89 83.06) (width 0.25) (layer "B.Cu") (net 54))
   (segment (start 54.61 62.865) (end 54.12 63.355) (width 0.25) (layer "B.Cu") (net 54))
+  (segment (start 64.84 73.795) (end 66.04 72.595) (width 0.25) (layer "B.Cu") (net 54))
   (segment (start 66.04 77.75) (end 66.04 85.725) (width 0.25) (layer "B.Cu") (net 54))
-  (segment (start 62.23 85.725) (end 66.04 85.725) (width 0.25) (layer "B.Cu") (net 54))
+  (segment (start 66.04 72.595) (end 67.06462 72.595) (width 0.25) (layer "B.Cu") (net 54))
+  (segment (start 66.04 77.75) (end 64.84 76.55) (width 0.25) (layer "B.Cu") (net 54))
+  (segment (start 65.405 67.945) (end 55.88 67.945) (width 0.25) (layer "B.Cu") (net 54))
   (segment (start 135.89 83.06) (end 135.89 72.39) (width 0.25) (layer "B.Cu") (net 54))
   (segment (start 54.265 66.04) (end 54.12 66.185) (width 0.25) (layer "B.Cu") (net 54))
   (segment (start 130.805 72.395) (end 133.345 72.395) (width 0.25) (layer "B.Cu") (net 54))
-  (segment (start 54.12 76.07163) (end 61.017379 82.969009) (width 0.25) (layer "B.Cu") (net 54))
-  (segment (start 61.017379 82.969009) (end 61.017379 84.512379) (width 0.25) (layer "B.Cu") (net 54))
+  (segment (start 55.88 67.945) (end 55.245 67.31) (width 0.25) (layer "B.Cu") (net 54))
+  (segment (start 67.06462 72.595) (end 67.255 72.40462) (width 0.25) (layer "B.Cu") (net 54))
+  (segment (start 55.245 67.31) (end 55.245 66.2725) (width 0.25) (layer "B.Cu") (net 54))
   (segment (start 55.4775 66.04) (end 54.265 66.04) (width 0.25) (layer "B.Cu") (net 54))
   (segment (start 66.04 85.725) (end 66.04 90.17) (width 0.25) (layer "B.Cu") (net 54))
-  (segment (start 54.12 66.185) (end 54.12 76.07163) (width 0.25) (layer "B.Cu") (net 54))
+  (segment (start 64.84 76.55) (end 64.84 73.795) (width 0.25) (layer "B.Cu") (net 54))
   (segment (start 127.99 75.21) (end 127 75.21) (width 0.25) (layer "B.Cu") (net 54))
   (segment (start 68.455 92.585) (end 126.365 92.585) (width 0.25) (layer "B.Cu") (net 54))
   (segment (start 66.04 90.17) (end 67.31 91.44) (width 0.25) (layer "B.Cu") (net 54))
+  (segment (start 67.255 69.795) (end 65.405 67.945) (width 0.25) (layer "B.Cu") (net 54))
   (segment (start 54.12 63.355) (end 54.12 66.185) (width 0.25) (layer "B.Cu") (net 54))
-  (segment (start 61.017379 84.512379) (end 62.23 85.725) (width 0.25) (layer "B.Cu") (net 54))
   (segment (start 130.805 72.395) (end 127.99 75.21) (width 0.25) (layer "B.Cu") (net 54))
+  (segment (start 67.255 72.40462) (end 67.255 69.795) (width 0.25) (layer "B.Cu") (net 54))
   (segment (start 130.805 82.555) (end 127.98 79.73) (width 0.25) (layer "B.Cu") (net 55))
   (segment (start 127.98 79.73) (end 127 79.73) (width 0.25) (layer "B.Cu") (net 55))
@@
   (segment (start 74.305 69.86) (end 77.48 69.86) (width 0.25) (layer "B.Cu") (net 68))
   (segment (start 74.295 69.85) (end 74.305 69.86) (width 0.25) (layer "B.Cu") (net 68))
-  (segment (start 59.755 71.12) (end 59.755 69.85) (width 0.25) (layer "F.Cu") (net 69))
-  (segment (start 55.245 71.12) (end 59.755 71.12) (width 0.25) (layer "F.Cu") (net 69))
+  (segment (start 59.755 69.85) (end 56.515 69.85) (width 1) (layer "F.Cu") (net 69))
+  (segment (start 56.515 69.85) (end 55.245 71.12) (width 1) (layer "F.Cu") (net 69))
+  (segment (start 59.755 71.12) (end 55.245 71.12) (width 1) (layer "F.Cu") (net 69))
   (segment (start 42.545 71.755) (end 43.18 71.12) (width 0.25) (layer "B.Cu") (net 70))
   (segment (start 42.545 74.295) (end 42.545 71.755) (width 0.25) (layer "B.Cu") (net 70))
