File: _Modular/TapeDelay/interconnect.kicad_sch (KiCad schematic)
At the start: 37 parts, among them J13 Dry In, J14 50k, J15 Dry In', J16 Out', J17 Out, J18 XMix 1, J19 XMix 2, J20 XMix 1', J21 XMix 2', J22 50k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

Commit message: up
Parts:
- U2: footprint Package_DIP:DIP-16_W7.62mm_LongPads -> Package_DIP:DIP-8_W7.62mm_LongPads
Changed lines of the file:
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@@
       (effects (font (size 1.27 1.27)) (justify left))
     )
-    (property "Footprint" "Package_DIP:DIP-16_W7.62mm_LongPads" (id 2) (at 158.75 184.15 0)
+    (property "Footprint" "Package_DIP:DIP-8_W7.62mm_LongPads" (id 2) (at 158.75 184.15 0)
       (effects (font (size 1.27 1.27)) hide)
     )
@@
     (property "Reference" "U2" (id 0) (at 73.66 15.24 0))
     (property "Value" "TL072" (id 1) (at 73.66 17.78 0))
-    (property "Footprint" "Package_DIP:DIP-16_W7.62mm_LongPads" (id 2) (at 73.66 25.4 0)
+    (property "Footprint" "Package_DIP:DIP-8_W7.62mm_LongPads" (id 2) (at 73.66 25.4 0)
       (effects (font (size 1.27 1.27)) hide)
     )
@@
     (property "Reference" "U2" (id 0) (at 248.92 19.05 0))
     (property "Value" "TL072" (id 1) (at 248.92 21.59 0))
-    (property "Footprint" "Package_DIP:DIP-16_W7.62mm_LongPads" (id 2) (at 248.92 29.21 0)
-      (effects (font (size 1.27 1.27)) hide)
-    )
+    (property "Footprint" "Package_DIP:DIP-8_W7.62mm_LongPads" (id 2) (at 248.92 29.21 0)
+      (effects (font (size 1.27 1.27)) hide)
+    )

Commit message: tape
Parts:
- renumbered U2 to U4
Changed lines of the file:
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@@
   (symbol (lib_id "Amplifier_Operational:TL072") (at 158.75 184.15 0) (unit 3)
     (in_bom yes) (on_board yes) (fields_autoplaced)
-    (property "Reference" "U2" (id 0) (at 157.48 182.8799 0)
-      (effects (font (size 1.27 1.27)) (justify left))
-    )
-    (property "Value" "TL072" (id 1) (at 157.48 185.4199 0)
+    (property "Reference" "U4" (id 0) (at 156.845 183.3153 0)
+      (effects (font (size 1.27 1.27)) (justify left))
+    )
+    (property "Value" "TL072" (id 1) (at 156.845 185.8522 0)
       (effects (font (size 1.27 1.27)) (justify left))
     )
@@
   (symbol (lib_id "Amplifier_Operational:TL072") (at 73.66 25.4 0) (unit 1)
     (in_bom yes) (on_board yes) (fields_autoplaced)
-    (property "Reference" "U2" (id 0) (at 73.66 15.24 0))
-    (property "Value" "TL072" (id 1) (at 73.66 17.78 0))
+    (property "Reference" "U4" (id 0) (at 73.66 16.6202 0))
+    (property "Value" "TL072" (id 1) (at 73.66 19.1571 0))
     (property "Footprint" "Package_DIP:DIP-8_W7.62mm_LongPads" (id 2) (at 73.66 25.4 0)
       (effects (font (size 1.27 1.27)) hide)
@@
   (symbol (lib_id "Amplifier_Operational:TL072") (at 248.92 29.21 0) (unit 2)
     (in_bom yes) (on_board yes) (fields_autoplaced)
-    (property "Reference" "U2" (id 0) (at 248.92 19.05 0))
-    (property "Value" "TL072" (id 1) (at 248.92 21.59 0))
+    (property "Reference" "U4" (id 0) (at 248.92 20.4302 0))
+    (property "Value" "TL072" (id 1) (at 248.92 22.9671 0))
     (property "Footprint" "Package_DIP:DIP-8_W7.62mm_LongPads" (id 2) (at 248.92 29.21 0)
       (effects (font (size 1.27 1.27)) hide)
