File: _Modular/TapeDelay/TapeDelay.kicad_sch (KiCad schematic)
At the start: 91 parts, among them J1 PB Head 1, J2 Rec Head, J3 Rec Meter, J4 PB Head 2, J5 PB Meter

Commit message: up
Parts:
- removed J?: Meter switch, symbol Connector:Conn_01x05_Male
- removed J?: Audio, symbol Connector:Conn_01x08_Male
- added C30, C32: 47,0, Capacitor_THT:CP_Radial_D6.3mm_P2.50mm, symbol Device:C_Polarized
- added J10: Meter Sw, Connector_PinHeader_2.54mm:PinHeader_1x03_P2.54mm_Vertical, symbol Connector:Conn_01x03_Male
- added J6: PB NR 1, Connector_PinHeader_2.54mm:PinHeader_1x02_P2.54mm_Vertical, symbol Connector:Conn_01x02_Male
- added J7: PB NR 2, Connector_PinHeader_2.54mm:PinHeader_1x02_P2.54mm_Vertical, symbol Connector:Conn_01x02_Male
- added J9: Rec NR, Connector_PinHeader_2.54mm:PinHeader_1x02_P2.54mm_Vertical, symbol Connector:Conn_01x02_Male
- added R31, R32: 100, Resistor_SMD:R_1206_3216Metric_Pad1.30x1.75mm_HandSolder, symbol Device:R
- added R33, R34: 47k, Resistor_SMD:R_1206_3216Metric_Pad1.30x1.75mm_HandSolder, symbol Device:R
- added TP1: TP Rec, Connector_PinHeader_2.54mm:PinHeader_1x01_P2.54mm_Vertical, symbol Connector:TestPoint
- C1, C10, C11, C12, C13, C15, C16, C17, C19, C2, C20, C21, C24, C3, C5, C7, C8: footprint (none) -> Capacitor_SMD:C_0805_2012Metric_Pad1.18x1.45mm_HandSolder
- C14, C4: footprint (none) -> Capacitor_THT:CP_Radial_D5.0mm_P2.50mm
- C18, C25, C28, C6: footprint (none) -> Capacitor_THT:CP_Radial_D7.5mm_P2.50mm
- C22, C23: footprint (none) -> Capacitor_SMD:C_1206_3216Metric_Pad1.33x1.80mm_HandSolder
- C26, C27, C9: footprint (none) -> Capacitor_THT:CP_Radial_D6.3mm_P2.50mm
- C29: renamed from C?; footprint (none) -> Capacitor_THT:CP_Radial_D6.3mm_P2.50mm
- C31, C33, C34, C35, C36, C38: renamed from C?; footprint (none) -> Capacitor_SMD:C_0805_2012Metric_Pad1.18x1.45mm_HandSolder
- C37: renamed from C?; footprint (none) -> Capacitor_THT:C_Disc_D5.0mm_W2.5mm_P2.50mm
- D1, D2: footprint (none) -> Package_DIP:DIP-16_W7.62mm_LongPads
- J1, J2, J3, J4, J5: footprint (none) -> Connector_PinHeader_2.54mm:PinHeader_1x02_P2.54mm_Vertical
- J11, J12: renamed from J?; footprint (none) -> Connector_PinHeader_2.54mm:PinHeader_1x02_P2.54mm_Vertical
- R1, R10, R11, R12, R15, R16, R17, R18, R19, R2, R20, R21, R22, R25, R26, R27, R28, R29, R3, R30, R4, R5, R6, R7, R8, R9: footprint (none) -> Resistor_SMD:R_1206_3216Metric_Pad1.30x1.75mm_HandSolder
- R13, R14, RV1: footprint (none) -> Resistor_THT:R_Axial_DIN0309_L9.0mm_D3.2mm_P2.54mm_Vertical
- R23, R24: value 100k -> 47k; footprint (none) -> Resistor_SMD:R_1206_3216Metric_Pad1.30x1.75mm_HandSolder
- R35, R36, R37, R39, R40: renamed from R?; footprint (none) -> Resistor_SMD:R_1206_3216Metric_Pad1.30x1.75mm_HandSolder
- R38, R41: renamed from R?; footprint (none) -> Resistor_THT:R_Axial_DIN0309_L9.0mm_D3.2mm_P2.54mm_Vertical
- gave numbers to parts that had none: 6
Connections:
- net +15V: now also R31.1; no longer C31.2, J8.1 (Pin_1), J8.2 (Pin_2), U1.3 (VI)
- net GND: now also C30.1, C32.2
- net PB Mix: now also C35.1
- net PB1: now also J6.1 (Pin_1), R33.2; no longer C5.2, R23.2
- net PB2: now also J7.1 (Pin_1), R34.2; no longer C24.2, R24.2
- net Rec: now also J9.2 (Pin_2); no longer C7.1
- net at J8.10 (Pin_10): now also J8.9 (Pin_9), R32.2
- net at R12.2, R13.2, RV1.2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: now also TP1.1
- new net: C31.2, J8.1 (Pin_1), J8.2 (Pin_2), R31.2, U1.3 (VI)
- new net: J10.3 (Pin_3), R24.2, R34.1
- new net: C5.2, J6.2 (Pin_2)
- new net: C24.2, J7.2 (Pin_2)
- new net: C32.1, J10.2 (Pin_2)
- new net: J10.1 (Pin_1), R23.2, R33.1
- new net: C7.1, J9.1 (Pin_1)
- new net -15V: C30.2, R32.1
- no-connect marks 2 -> 0
Other:
- added sheet Interconnect (interconnect.kicad_sch)
- note added: "Turns off metering for PB1/PB2 in side positions, in center pos enables both"
- moved on the sheet: C29, R24

Commit message: up
Parts:
- added C53: 47,0, Capacitor_THT:CP_Radial_D6.3mm_P2.50mm, symbol Device:C_Polarized
- C27: footprint Capacitor_THT:CP_Radial_D6.3mm_P2.50mm -> Capacitor_SMD:C_0805_2012Metric_Pad1.18x1.45mm_HandSolder
- C38: footprint Capacitor_SMD:C_0805_2012Metric_Pad1.18x1.45mm_HandSolder -> Capacitor_THT:C_Disc_D5.0mm_W2.5mm_P2.50mm
- D3: value D -> SS34; footprint (none) -> Diode_SMD:D_SMA-SMB_Universal_Handsoldering
- Q1: footprint (none) -> Package_TO_SOT_THT:TO-92
- Q2, Q3: footprint (none) -> Package_TO_SOT_THT:TO-92_Wide
- RV1: footprint Resistor_THT:R_Axial_DIN0309_L9.0mm_D3.2mm_P2.54mm_Vertical -> Potentiometer_THT:Potentiometer_Runtron_RM-065_Vertical
Connections:
- net GND: now also C53.2
- net at R13.2, RV1.2, RV1.3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: now also C14.2; no longer R12.2
- net at C13.1, C15.1, D1.9 (RecOut)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: now also R12.1; no longer C14.1
- net at C34.1, Q2.2 (C), R36.2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: now also C53.1
- new net: C14.1, R12.2
Other:
- moved on the sheet: C14, R12
Changed lines of the file:
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@@
   (junction (at 93.98 175.26) (diameter 0) (color 0 0 0 0)
   )
+  (junction (at 168.91 36.83) (diameter 0) (color 0 0 0 0)
+  )
   (junction (at 46.99 39.37) (diameter 0) (color 0 0 0 0)
   )
@@
   (junction (at 130.81 109.22) (diameter 0) (color 0 0 0 0)
   )
-  (junction (at 168.91 36.83) (diameter 0) (color 0 0 0 0)
-  )
   (junction (at 123.19 109.22) (diameter 0) (color 0 0 0 0)
   )
@@
       (effects (font (size 1.27 1.27)) (justify left))
     )
-    (property "Footprint" "" (id 2) (at 227.33 146.05 0)
+    (property "Footprint" "Package_TO_SOT_THT:TO-92" (id 2) (at 227.33 146.05 0)
       (effects (font (size 1.27 1.27)) hide)
     )
@@
       (effects (font (size 1.27 1.27)) (justify right))
     )
-    (property "Footprint" "Resistor_THT:R_Axial_DIN0309_L9.0mm_D3.2mm_P2.54mm_Vertical" (id 2) (at 190.5 33.02 0)
+    (property "Footprint" "Potentiometer_THT:Potentiometer_Runtron_RM-065_Vertical" (id 2) (at 190.5 33.02 0)
       (effects (font (size 1.27 1.27)) hide)
     )
@@
     (pin "2")
   )
+  (symbol (lib_id "power:GND") (at 217.17 111.76 180) (unit 1)
+    (in_bom yes) (on_board yes) (fields_autoplaced)
+    (property "Reference" "#PWR023" (id 0) (at 217.17 105.41 0)
+      (effects (font (size 1.27 1.27)) hide)
+    )
+    (property "Value" "GND" (id 1) (at 219.71 110.4899 0)
+      (effects (font (size 1.27 1.27)) (justify right))
+    )
+    (property "Footprint" "" (id 2) (at 217.17 111.76 0)
+      (effects (font (size 1.27 1.27)) hide)
+    )
+    (property "Datasheet" "" (id 3) (at 217.17 111.76 0)
+      (effects (font (size 1.27 1.27)) hide)
+    )
+    (pin "1")
+  )
   (symbol (lib_id "power:+12VA") (at 165.1 92.71 270) (unit 1)
     (in_bom yes) (on_board yes) (fields_autoplaced)
@@
       (effects (font (size 1.27 1.27)) (justify left))
     )
-    (property "Footprint" "Capacitor_THT:CP_Radial_D6.3mm_P2.50mm" (id 2) (at 229.5652 99.06 0)
+    (property "Footprint" "Capacitor_SMD:C_0805_2012Metric_Pad1.18x1.45mm_HandSolder" (id 2) (at 229.5652 99.06 0)
       (effects (font (size 1.27 1.27)) hide)
     )
@@
     (pin "2")
   )
+  (symbol (lib_id "Device:C_Polarized") (at 217.17 115.57 180) (unit 1)
+    (in_bom yes) (on_board yes)
+    (property "Reference" "C53" (id 0) (at 222.25 114.3 0))
+    (property "Value" "47,0" (id 1) (at 222.25 116.84 0))
+    (property "Footprint" "Capacitor_THT:CP_Radial_D6.3mm_P2.50mm" (id 2) (at 216.2048 111.76 0)
+      (effects (font (size 1.27 1.27)) hide)
+    )
+    (property "Datasheet" "~" (id 3) (at 217.17 115.57 0)
+      (effects (font (size 1.27 1.27)) hide)
+    )
+    (pin "1")
+    (pin "2")
+  )
   (symbol (lib_id "Device:R") (at 269.24 40.64 180) (unit 1)
     (in_bom yes) (on_board yes) (fields_autoplaced)
@@
       (effects (font (size 1.27 1.27)) (justify right))
     )
-    (property "Footprint" "Capacitor_SMD:C_0805_2012Metric_Pad1.18x1.45mm_HandSolder" (id 2) (at 261.9248 146.05 0)
+    (property "Footprint" "Capacitor_THT:C_Disc_D5.0mm_W2.5mm_P2.50mm" (id 2) (at 261.9248 146.05 0)
       (effects (font (size 1.27 1.27)) hide)
     )
@@
       (effects (font (size 1.27 1.27)) (justify left))
     )
-    (property "Footprint" "" (id 2) (at 242.57 146.05 0)
+    (property "Footprint" "Package_TO_SOT_THT:TO-92_Wide" (id 2) (at 242.57 146.05 0)
       (effects (font (size 1.27 1.27)) hide)
     )
@@
     (pin "2")
   )
-  (symbol (lib_id "Device:R") (at 180.34 36.83 90) (unit 1)
+  (symbol (lib_id "Device:R") (at 172.72 36.83 90) (unit 1)
     (in_bom yes) (on_board yes) (fields_autoplaced)
-    (property "Reference" "R12" (id 0) (at 180.34 30.48 90))
-    (property "Value" "6,8k" (id 1) (at 180.34 33.02 90))
-    (property "Footprint" "Resistor_SMD:R_1206_3216Metric_Pad1.30x1.75mm_HandSolder" (id 2) (at 180.34 38.608 90)
+    (property "Reference" "R12" (id 0) (at 172.72 30.48 90))
+    (property "Value" "6,8k" (id 1) (at 172.72 33.02 90))
+    (property "Footprint" "Resistor_SMD:R_1206_3216Metric_Pad1.30x1.75mm_HandSolder" (id 2) (at 172.72 38.608 90)
       (effects (font (size 1.27 1.27)) hide)
     )
-    (property "Datasheet" "~" (id 3) (at 180.34 36.83 0)
+    (property "Datasheet" "~" (id 3) (at 172.72 36.83 0)
       (effects (font (size 1.27 1.27)) hide)
     )
@@
       (effects (font (size 1.27 1.27)) (justify left))
     )
-    (property "Footprint" "" (id 2) (at 242.57 124.46 0)
+    (property "Footprint" "Package_TO_SOT_THT:TO-92_Wide" (id 2) (at 242.57 124.46 0)
       (effects (font (size 1.27 1.27)) hide)
     )
@@
       (effects (font (size 1.27 1.27)) (justify right))
     )
-    (property "Value" "D" (id 1) (at 250.19 140.9699 90)
+    (property "Value" "SS34" (id 1) (at 250.19 140.9699 90)
       (effects (font (size 1.27 1.27)) (justify right))
     )
-    (property "Footprint" "" (id 2) (at 247.65 139.7 0)
+    (property "Footprint" "Diode_SMD:D_SMA-SMB_Universal_Handsoldering" (id 2) (at 247.65 139.7 0)
       (effects (font (size 1.27 1.27)) hide)
     )
@@
     (pin "2")
   )
-  (symbol (lib_id "Device:C_Polarized") (at 172.72 36.83 90) (unit 1)
+  (symbol (lib_id "Device:C_Polarized") (at 180.34 36.83 90) (unit 1)
     (in_bom yes) (on_board yes) (fields_autoplaced)
-    (property "Reference" "C14" (id 0) (at 171.831 29.21 90))
-    (property "Value" "10,0" (id 1) (at 171.831 31.75 90))
-    (property "Footprint" "Capacitor_THT:CP_Radial_D5.0mm_P2.50mm" (id 2) (at 176.53 35.8648 0)
+    (property "Reference" "C14" (id 0) (at 179.451 29.21 90))
+    (property "Value" "10,0" (id 1) (at 179.451 31.75 90))
+    (property "Footprint" "Capacitor_THT:CP_Radial_D5.0mm_P2.50mm" (id 2) (at 184.15 35.8648 0)
       (effects (font (size 1.27 1.27)) hide)
     )
-    (property "Datasheet" "~" (id 3) (at 172.72 36.83 0)
+    (property "Datasheet" "~" (id 3) (at 180.34 36.83 0)
       (effects (font (size 1.27 1.27)) hide)
     )
@@
       (reference "#PWR022") (unit 1) (value "+12VA") (footprint "")
     )
+    (path "/2dab14a1-84a4-455d-bfdb-0364709026e9"
+      (reference "#PWR023") (unit 1) (value "GND") (footprint "")
+    )
     (path "/bc136873-ed84-4d0d-b036-84a2fb1efa68"
       (reference "#PWR0101") (unit 1) (value "GND") (footprint "")
@@
     )
     (path "/7e5caa1f-f1d1-49cf-9f99-9d02e9193aca"
-      (reference "C27") (unit 1) (value "4,7") (footprint "Capacitor_THT:CP_Radial_D6.3mm_P2.50mm")
+      (reference "C27") (unit 1) (value "4,7") (footprint "Capacitor_SMD:C_0805_2012Metric_Pad1.18x1.45mm_HandSolder")
     )
     (path "/13ad48bd-4181-4a6a-9f5b-b6b8772fa516"
@@
     )
     (path "/c407ddd8-26fd-4217-b7b0-6bd9cc265d1e"
-      (reference "C38") (unit 1) (value "0,01") (footprint "Capacitor_SMD:C_0805_2012Metric_Pad1.18x1.45mm_HandSolder")
+      (reference "C38") (unit 1) (value "0,01") (footprint "Capacitor_THT:C_Disc_D5.0mm_W2.5mm_P2.50mm")
     )
     (path "/3ce054ec-f5d0-4ba0-80ab-69acb624d505/8ad43a07-66fd-4c3e-b7ad-57b516a3ab59"
@@
       (reference "C52") (unit 1) (value "10,0") (footprint "Capacitor_SMD:C_1206_3216Metric_Pad1.33x1.80mm_HandSolder")
     )
+    (path "/b2f8d0bc-d4f1-4b7c-b8cb-ac8c0c5aecd0"
+      (reference "C53") (unit 1) (value "47,0") (footprint "Capacitor_THT:CP_Radial_D6.3mm_P2.50mm")
+    )
     (path "/1213eb54-00c5-48a4-b2c0-a1ad34d4d51b"
       (reference "D1") (unit 1) (value "К174УН13") (footprint "Package_DIP:DIP-16_W7.62mm_LongPads")
@@
     )
     (path "/e952a00e-40e6-4e15-9f61-608074d61c84"
-      (reference "D3") (unit 1) (value "D") (footprint "")
+      (reference "D3") (unit 1) (value "SS34") (footprint "Diode_SMD:D_SMA-SMB_Universal_Handsoldering")
     )
     (path "/38a2a1d3-853e-4498-8432-eeda026af4a7"
@@
     )
     (path "/0a1a7f08-ef8b-41d3-8ec1-b123cefac08e"
-      (reference "Q1") (unit 1) (value "KT3107") (footprint "")
+      (reference "Q1") (unit 1) (value "KT3107") (footprint "Package_TO_SOT_THT:TO-92")
     )
     (path "/e8208e7a-b420-4ae1-9bd9-08fa3f922f4f"
-      (reference "Q2") (unit 1) (value "KT603A") (footprint "")
+      (reference "Q2") (unit 1) (value "KT603A") (footprint "Package_TO_SOT_THT:TO-92_Wide")
     )
     (path "/cb03f1fe-8aee-40f7-87c8-8509f917f530"
-      (reference "Q3") (unit 1) (value "KT603A") (footprint "")
+      (reference "Q3") (unit 1) (value "KT603A") (footprint "Package_TO_SOT_THT:TO-92_Wide")
     )
     (path "/5e00a4eb-6f40-4bc7-aa95-8ae2784598fc"
@@
     )
     (path "/0d446b2f-0d30-4eab-bdb2-d80f0f94ce27"
-      (reference "RV1") (unit 1) (value "100k") (footprint "Resistor_THT:R_Axial_DIN0309_L9.0mm_D3.2mm_P2.54mm_Vertical")
+      (reference "RV1") (unit 1) (value "100k") (footprint "Potentiometer_THT:Potentiometer_Runtron_RM-065_Vertical")
     )
     (path "/a03be65a-2b6a-4db8-9bfa-1f87799f0c73"
@@
     )
     (path "/3ce054ec-f5d0-4ba0-80ab-69acb624d505/5a26ff6a-3c17-4ccb-8d4b-b05f9438fb77"
-      (reference "U2") (unit 1) (value "TL072") (footprint "Package_DIP:DIP-16_W7.62mm_LongPads")
+      (reference "U2") (unit 1) (value "TL072") (footprint "Package_DIP:DIP-8_W7.62mm_LongPads")
     )
     (path "/3ce054ec-f5d0-4ba0-80ab-69acb624d505/71718834-8634-4371-aa26-abc98d842440"
-      (reference "U2") (unit 2) (value "TL072") (footprint "Package_DIP:DIP-16_W7.62mm_LongPads")
+      (reference "U2") (unit 2) (value "TL072") (footprint "Package_DIP:DIP-8_W7.62mm_LongPads")
     )
     (path "/3ce054ec-f5d0-4ba0-80ab-69acb624d505/2d77aceb-6985-4313-8fe0-1c707dedbd38"
-      (reference "U2") (unit 3) (value "TL072") (footprint "Package_DIP:DIP-16_W7.62mm_LongPads")
+      (reference "U2") (unit 3) (value "TL072") (footprint "Package_DIP:DIP-8_W7.62mm_LongPads")
     )
   )

Commit message: meter
Parts:
- removed C34: 0,1, Capacitor_SMD:C_0805_2012Metric_Pad1.18x1.45mm_HandSolder, symbol Device:C
- removed C36: 1,0, Capacitor_SMD:C_0805_2012Metric_Pad1.18x1.45mm_HandSolder, symbol Device:C
- removed C37: 27, Capacitor_THT:C_Disc_D5.0mm_W2.5mm_P2.50mm, symbol Device:C
- removed C38: 0,01, Capacitor_THT:C_Disc_D5.0mm_W2.5mm_P2.50mm, symbol Device:C
- removed C53: 47,0, Capacitor_THT:CP_Radial_D6.3mm_P2.50mm, symbol Device:C_Polarized
- removed D3: SS34, Diode_SMD:D_SMA-SMB_Universal_Handsoldering, symbol Device:D
- removed J11: Erase Head, Connector_PinHeader_2.54mm:PinHeader_1x02_P2.54mm_Vertical, symbol Connector:Conn_01x02_Male
- removed J12: Gen, Connector_PinHeader_2.54mm:PinHeader_1x02_P2.54mm_Vertical, symbol Connector:Conn_01x02_Male
- removed Q1: KT3107, Package_TO_SOT_THT:TO-92, symbol Device:Q_PNP_CBE
- removed Q2, Q3: KT603A, Package_TO_SOT_THT:TO-92_Wide, symbol Device:Q_NPN_BCE
- removed R35, R40: 470, Resistor_SMD:R_1206_3216Metric_Pad1.30x1.75mm_HandSolder, symbol Device:R
- removed R36, R37: 30k, Resistor_SMD:R_1206_3216Metric_Pad1.30x1.75mm_HandSolder, symbol Device:R
- removed R38: 10, Resistor_THT:R_Axial_DIN0309_L9.0mm_D3.2mm_P2.54mm_Vertical, symbol Device:R
- removed R39: 4,3k, Resistor_SMD:R_1206_3216Metric_Pad1.30x1.75mm_HandSolder, symbol Device:R
- removed R41: 43, Resistor_THT:R_Axial_DIN0309_L9.0mm_D3.2mm_P2.54mm_Vertical, symbol Device:R
- added R? (x2): 1k, Resistor_SMD:R_1206_3216Metric_Pad1.30x1.75mm_HandSolder, symbol Device:R
Connections:
- net +12VA: now also R?.2, R?.2
- net at D2.6 (AlcOut), R29.1: now also R?.1
- net at D1.6 (AlcOut), R17.1: now also R?.1
Other:
- note removed: "Erase head generator is soldered on one board only, connects to other with Gen connector"

Commit message: tape
Parts:
- removed C15: 10,0, Capacitor_SMD:C_0805_2012Metric_Pad1.18x1.45mm_HandSolder, symbol Device:C_Polarized
- removed C17, C27: 4,7, Capacitor_SMD:C_0805_2012Metric_Pad1.18x1.45mm_HandSolder, symbol Device:C_Polarized
- removed C18, C28: 220,0, Capacitor_THT:CP_Radial_D7.5mm_P2.50mm, symbol Device:C_Polarized
- removed C35: 10,0, Capacitor_SMD:C_0805_2012Metric_Pad1.18x1.45mm_HandSolder, symbol Device:C
- removed R15, R16, R27, R28: 10k, Resistor_SMD:R_1206_3216Metric_Pad1.30x1.75mm_HandSolder, symbol Device:R
- removed R17, R29: 120k, Resistor_SMD:R_1206_3216Metric_Pad1.30x1.75mm_HandSolder, symbol Device:R
- removed R18, R30: 1m, Resistor_SMD:R_1206_3216Metric_Pad1.30x1.75mm_HandSolder, symbol Device:R
- removed R? (x2): 1k, Resistor_SMD:R_1206_3216Metric_Pad1.30x1.75mm_HandSolder, symbol Device:R
- added J11: Gen, Connector_PinHeader_2.54mm:PinHeader_1x02_P2.54mm_Vertical, symbol Connector:Conn_01x02_Male
- U3: renamed from U1; value L78L12_TO92 -> L78L12
- renumbered D1 to U1, D2 to U2
Connections:
- net +12VA: no longer J3.2 (Pin_2), J5.2 (Pin_2)
- net GND: now also J3.1 (Pin_1), J5.1 (Pin_1), U1.11 (AlcSpeedCap), U1.12 (AlcRC), U1.13 (AlcIn1), U1.14 (AlcIn2), U1.6 (AlcOut), U2.11 (AlcSpeedCap), U2.12 (AlcRC), U2.13 (AlcIn1), U2.14 (AlcIn2), U2.6 (AlcOut)
- net Gen: now also J11.1 (Pin_1), J11.2 (Pin_2)
- net PB Mix: now also J5.2 (Pin_2)
- net at C13.1, R10.2, R12.1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: now also J3.2 (Pin_2)
Other:
- moved on the sheet: J3, J5

Commit message: up
Parts:
- removed C26, C32: 47,0, Capacitor_THT:CP_Radial_D6.3mm_P2.50mm, symbol Device:C_Polarized
- added C? (x2): 4,7, Capacitor_SMD:C_0805_2012Metric_Pad1.18x1.45mm_HandSolder, symbol Device:C
- added C? (x5): 10,0, Capacitor_SMD:C_0805_2012Metric_Pad1.18x1.45mm_HandSolder, symbol Device:C
- added C?: 22n, Capacitor_SMD:C_0805_2012Metric_Pad1.18x1.45mm_HandSolder, symbol Device:C
- added C?: 1,0, Capacitor_SMD:C_0805_2012Metric_Pad1.18x1.45mm_HandSolder, symbol Device:C
- added D? (x2): LED, symbol Device:LED
- added R? (x4): 10k, Resistor_SMD:R_1206_3216Metric_Pad1.30x1.75mm_HandSolder, symbol Device:R
- added R? (x2): 470k, Resistor_SMD:R_1206_3216Metric_Pad1.30x1.75mm_HandSolder, symbol Device:R
- added R? (x2): 2,2k, Resistor_SMD:R_1206_3216Metric_Pad1.30x1.75mm_HandSolder, symbol Device:R
- added R? (x2): 5,6k, Resistor_SMD:R_1206_3216Metric_Pad1.30x1.75mm_HandSolder, symbol Device:R
- C25: value 100,0 -> 100,0 x 6v
Connections:
- net +12VA: now also R?.2, R?.2, R?.2, R?.2
- net GND: now also J10.2 (Pin_2), C?.1, C?.1, C?.1, C?.1, C?.1, C?.2, R?.1, R?.1; no longer U1.11 (AlcSpeedCap), U1.12 (AlcRC), U1.13 (AlcIn1), U1.14 (AlcIn2), U1.6 (AlcOut), U2.11 (AlcSpeedCap), U2.12 (AlcRC), U2.13 (AlcIn1), U2.14 (AlcIn2), U2.6 (AlcOut)
- net PB Mix: now also C?.1, C?.1
- net Rec: now also C13.1, J3.2 (Pin_2), R10.2, R12.1, R9.2, U1.9 (RecOut), C?.1
- net at R23.1, R24.1: now also C?.1; no longer R26.2, U2.7 (RecFB)
- net at R22.1, R25.2, U2.8 (RecIn): now also C?.2
- new net: C?.2, U2.11 (AlcSpeedCap)
- new net: C?.2, R?.2, U2.12 (AlcRC)
- new net: R?.2, U2.13 (AlcIn1)
- new net: R?.1, U2.14 (AlcIn2)
- new net: D?.1 (K), R?.1, U2.6 (AlcOut)
- new net: C?.2, U1.11 (AlcSpeedCap)
- new net: C?.2, R?.2, U1.12 (AlcRC)
- new net: R?.2, U1.13 (AlcIn1)
- new net: R?.1, U1.14 (AlcIn2)
- new net: D?.1 (K), R?.1, U1.6 (AlcOut)
- new net: C?.2, R?.1, R?.2 (x2)
- new net: C?.2, R26.2, U2.7 (RecFB)
- new net: D?.2 (A), R?.1 (x2)
Other:
- moved on the sheet: J10, R23, R24, R33, R34, U1C, U2C

Commit message: up
Parts:
- R7: value 180 -> 1k
Changed lines of the file:
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@@
       (effects (font (size 1.27 1.27)) (justify right))
     )
-    (property "Value" "180" (id 1) (at 130.81 69.85 0)
+    (property "Value" "1k" (id 1) (at 130.81 69.85 0)
       (effects (font (size 1.27 1.27)) (justify right))
     )
@@
     )
     (path "/ff93e7c0-f31a-42b6-8c22-060a826bd04d"
-      (reference "R7") (unit 1) (value "180") (footprint "Resistor_SMD:R_1206_3216Metric_Pad1.30x1.75mm_HandSolder")
+      (reference "R7") (unit 1) (value "1k") (footprint "Resistor_SMD:R_1206_3216Metric_Pad1.30x1.75mm_HandSolder")
     )
     (path "/2c8b108f-1ea1-4fc8-94e9-a5b04c76d2e3"
