File: _Modular/dz_HeadPhones_Amp/dz_HeadPhones_Amp.kicad_pcb (KiCad board)
At the start: 2 copper layers, 76.2 x 69.8 mm, 83 parts, among them J1 In, J2 Through, J3 Power, J4 ModPower, J5 Phones, J6 Meter, J7 Meter, Q1 BC547, Q2 BC557, Q3 BC547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

Commit message: upd
Parts:
- J6: value Meter -> Meter R
- J7: value Meter -> Meter L
- Q1, Q3: value BC547 -> КТ503
- Q2, Q4: value BC557 -> КТ502
Routing:
- added copper zone on F.Cu, net GND
Other:
- board text added: "+"
- board text added: "-"
- board text added: "100uA"
- board text added: "12..15v"
- board text removed: "Power"

Commit message: meter pcb
Parts:
- removed C23, C26: 1,0, Capacitor_SMD:C_0805_2012Metric_Pad1.18x1.45mm_HandSolder
- removed D6, D9: 1N4148, Diode_THT:D_DO-35_SOD27_P2.54mm_Vertical_KathodeUp
- added C14: 56, Capacitor_THT:C_Disc_D5.0mm_W2.5mm_P2.50mm, F.Cu at (236.2, 74.9)
- added C19: 56, Capacitor_THT:C_Disc_D5.0mm_W2.5mm_P2.50mm, F.Cu at (236.2, 59.7)
- added R25: 560, Resistor_THT:R_Axial_DIN0207_L6.3mm_D2.5mm_P2.54mm_Vertical, F.Cu at (255.3, 52.1)
- added R26: 9.1k, Resistor_THT:R_Axial_DIN0207_L6.3mm_D2.5mm_P2.54mm_Vertical, F.Cu at (261.6, 52.1)
- R19: value 120k -> 560
- R22: value 120k -> 9.1k
- moved R22 38.3 mm to (261.6, 85.1), turned to 180 degrees
- moved R19 34.2 mm to (253.4, 87.4), turned to 90 degrees
- moved D10 29.0 mm to (261.6, 88.9)
- moved D8 26.2 mm to (229.2, 83.2)
- moved D7 17.9 mm to (252.7, 55.2), turned to 0 degrees
- moved C21 16.4 mm to (234.3, 66.7)
- moved C25 15.9 mm to (245.7, 85.1)
- moved C22 14.6 mm to (247.0, 52.1)
- moved D5 14.6 mm to (240.7, 53.3)
- moved C24 12.4 mm to (232.8, 78.7)
- moved R24 6.26 mm to (232.4, 72.6), turned to -90 degrees
- moved R21 1.83 mm to (232.4, 54.6)
Connections:
- C24 pad 2: Net-(C24-Pad2) -> Net-(RV3-Pad3)
- D10 pad 1: Net-(C26-Pad2) -> Net-(C25-Pad2)
- D5 pad 4: Net-(D5-Pad4) -> Net-(RV2-Pad1)
- D7 pad 1: Net-(C23-Pad2) -> Net-(C22-Pad2)
- D7 pad 2: Net-(D5-Pad4) -> Net-(D7-Pad2)
- D8 pad 4: Net-(D10-Pad2) -> Net-(D8-Pad4)
- J6 pad 1: Net-(C22-Pad1) -> Net-(J6-Pad1)
- J7 pad 1: Net-(C25-Pad1) -> Net-(J7-Pad1)
- R19 pad 1: Net-(C23-Pad1) -> Net-(D10-Pad2)
- R19 pad 2: Net-(C21-Pad2) -> Net-(C25-Pad1)
- R21 pad 2: Net-(D5-Pad4) -> Net-(RV2-Pad1)
- R22 pad 1: Net-(C26-Pad1) -> Net-(J7-Pad1)
- R22 pad 2: Net-(C24-Pad2) -> Net-(C25-Pad1)
- R24 pad 2: Net-(D10-Pad2) -> Net-(D8-Pad4)
- RV2 pad 2: Net-(C23-Pad1) -> Net-(U2-Pad2)
- RV2 pad 3: GND -> Net-(C21-Pad2)
- RV3 pad 1: Net-(RV3-Pad1) -> Net-(D8-Pad4)
- RV3 pad 2: Net-(C26-Pad1) -> Net-(RV3-Pad2)
- RV3 pad 3: GND -> Net-(RV3-Pad3)
- U2 pad 2: Net-(C23-Pad2) -> Net-(U2-Pad2)
- U2 pad 3: Net-(RV2-Pad1) -> GND
- U2 pad 5: Net-(RV3-Pad1) -> GND
- U2 pad 6: Net-(C26-Pad2) -> Net-(RV3-Pad2)
Routing:
- net Net-(C25-Pad2): track 8.39 -> 39.0 mm
- net Net-(D8-Pad4): track 0.00 -> 28.9 mm
- net Net-(D5-Pad4): track 27.5 -> 0.00 mm
- net GND: track 320.3 -> 294.8 mm
- net Net-(C23-Pad1): track 22.9 -> 0.00 mm, vias 2 -> 0
- net Net-(C25-Pad1): track 8.35 -> 29.8 mm
- net Net-(D10-Pad2): track 26.0 -> 6.33 mm
- net Net-(RV3-Pad2): track 0.00 -> 19.6 mm
- net Net-(C24-Pad2): track 18.6 -> 0.00 mm, vias 1 -> 0
- net Net-(U2-Pad2): track 0.00 -> 17.5 mm
- net Net-(C26-Pad2): track 16.2 -> 0.00 mm
- net Net-(C22-Pad2): track 8.39 -> 24.6 mm
- net Net-(C23-Pad2): track 15.2 -> 0.00 mm
- net Net-(RV3-Pad1): track 12.6 -> 0.00 mm
- net /L: track 45.8 -> 57.0 mm
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Other:
- board text removed: "D6,7,9,10 Germanium"
