File: _Modular/dz_HeadPhones_Amp/dz_HeadPhones_Amp.kicad_sch (KiCad schematic)
At the start: 83 parts, among them J1 In, J2 Through, J3 Power, J4 ModPower, J5 Phones, J6 100uA meter, J7 100uA meter, Q1 BC547, Q2 BC557, Q3 BC547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

Commit message: upd
Parts:
- J6: value 100uA meter -> Meter R
- J7: value 100uA meter -> Meter L
- Q1, Q3: value BC547 -> КТ503
- Q2, Q4: value BC557 -> КТ502
Changed lines of the file:
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@@
       (effects (font (size 1.27 1.27)) (justify left))
     )
-    (property "Value" "BC547" (id 1) (at 225.8314 76.6322 0)
+    (property "Value" "КТ503" (id 1) (at 225.8314 76.6322 0)
       (effects (font (size 1.27 1.27)) (justify left))
     )
@@
       (effects (font (size 1.27 1.27)) (justify right))
     )
-    (property "Value" "100uA meter" (id 1) (at 123.19 53.34 0)
+    (property "Value" "Meter L" (id 1) (at 123.19 53.34 0)
       (effects (font (size 1.27 1.27)) (justify right))
     )
@@
       (effects (font (size 1.27 1.27)) (justify right))
     )
-    (property "Value" "100uA meter" (id 1) (at 123.19 105.41 0)
+    (property "Value" "Meter R" (id 1) (at 123.19 105.41 0)
       (effects (font (size 1.27 1.27)) (justify right))
     )
@@
       (effects (font (size 1.27 1.27)) (justify left))
     )
-    (property "Value" "BC557" (id 1) (at 225.8314 51.2322 0)
+    (property "Value" "КТ502" (id 1) (at 225.8314 51.2322 0)
       (effects (font (size 1.27 1.27)) (justify left))
     )
@@
       (effects (font (size 1.27 1.27)) (justify left))
     )
-    (property "Value" "BC547" (id 1) (at 225.8314 25.8322 0)
+    (property "Value" "КТ503" (id 1) (at 225.8314 25.8322 0)
       (effects (font (size 1.27 1.27)) (justify left))
     )
@@
       (effects (font (size 1.27 1.27)) (justify left))
     )
-    (property "Value" "BC557" (id 1) (at 225.8314 102.0322 0)
+    (property "Value" "КТ502" (id 1) (at 225.8314 102.0322 0)
       (effects (font (size 1.27 1.27)) (justify left))
     )
@@
     )
     (path "/909cb313-5c46-4fc6-acd4-77011131de34"
-      (reference "J6") (unit 1) (value "100uA meter") (footprint "Connector_PinHeader_2.54mm:PinHeader_1x02_P2.54mm_Vertical")
+      (reference "J6") (unit 1) (value "Meter R") (footprint "Connector_PinHeader_2.54mm:PinHeader_1x02_P2.54mm_Vertical")
     )
     (path "/61980665-96ae-4299-9e50-ffc20749fb2a"
-      (reference "J7") (unit 1) (value "100uA meter") (footprint "Connector_PinHeader_2.54mm:PinHeader_1x02_P2.54mm_Vertical")
+      (reference "J7") (unit 1) (value "Meter L") (footprint "Connector_PinHeader_2.54mm:PinHeader_1x02_P2.54mm_Vertical")
     )
     (path "/0c6dbee1-fe20-4327-873a-16cdbcda8145"
@@
     )
     (path "/9c10fe75-cfaa-439f-8c35-ab30d69f7a3a"
-      (reference "Q1") (unit 1) (value "BC547") (footprint "Package_TO_SOT_THT:TO-92_Inline")
+      (reference "Q1") (unit 1) (value "КТ503") (footprint "Package_TO_SOT_THT:TO-92_Inline")
     )
     (path "/96cca99a-11fb-48b4-9ca2-a901b390f633"
-      (reference "Q2") (unit 1) (value "BC557") (footprint "Package_TO_SOT_THT:TO-92_Inline")
+      (reference "Q2") (unit 1) (value "КТ502") (footprint "Package_TO_SOT_THT:TO-92_Inline")
     )
     (path "/5e69ed39-872a-4431-84bd-c0c4fb0d80c7"
-      (reference "Q3") (unit 1) (value "BC547") (footprint "Package_TO_SOT_THT:TO-92_Inline")
+      (reference "Q3") (unit 1) (value "КТ503") (footprint "Package_TO_SOT_THT:TO-92_Inline")
     )
     (path "/f5856ec5-7727-4aef-9fe9-bfb103bee8bb"
-      (reference "Q4") (unit 1) (value "BC557") (footprint "Package_TO_SOT_THT:TO-92_Inline")
+      (reference "Q4") (unit 1) (value "КТ502") (footprint "Package_TO_SOT_THT:TO-92_Inline")
     )
     (path "/21148db9-a300-4e23-8fc4-552b3bdf5e43"

Commit message: meter
Parts:
- removed C23, C26: 1,0, Capacitor_SMD:C_0805_2012Metric_Pad1.18x1.45mm_HandSolder, symbol Device:C
- removed D6, D9: 1N4148, Diode_THT:D_DO-35_SOD27_P2.54mm_Vertical_KathodeUp, symbol Diode:1N4148
- added C14, C19: 56, Capacitor_THT:C_Disc_D5.0mm_W2.5mm_P2.50mm, symbol Device:C
- added R25: 560, Resistor_THT:R_Axial_DIN0207_L6.3mm_D2.5mm_P2.54mm_Vertical, symbol Device:R
- added R26: 9.1k, Resistor_THT:R_Axial_DIN0207_L6.3mm_D2.5mm_P2.54mm_Vertical, symbol Device:R
- R19: value 120k -> 560
- R22: value 120k -> 9.1k
Connections:
- net GND: now also U2.3 (+), U2.5 (+); no longer RV2.3, RV3.3
- net at C22.1, D5.1 (+): now also R25.2, R26.2; no longer J6.1 (Pin_1)
- net at C22.2, D5.2 (-), J6.2 (Pin_2): now also D7.1 (K)
- net at D5.3, U2.1: now also C19.1
- net at D5.4, R21.2: now also RV2.1, C19.2; no longer D7.2 (A)
- net at U2.2 (-): now also RV2.2; no longer D7.1 (K)
- net at RV3.1: now also D8.4, R24.2, C14.2; no longer U2.5 (+)
- net at RV3.2: now also U2.6 (-); no longer R22.1
- net at R19.1: now also D10.2 (A); no longer RV2.2
- net at C25.1, D8.1 (+): now also R19.2, R22.2; no longer J7.1 (Pin_1)
- net at C25.2, D8.2 (-), J7.2 (Pin_2): now also D10.1 (K)
- net at D8.3, U2.7: now also C14.1
- net at C24.2: now also RV3.3; no longer R22.2
- net at C21.2: now also RV2.3; no longer R19.2
- new net: D7.2 (A), R25.1
- new net: J7.1 (Pin_1), R22.1
- new net: J6.1 (Pin_1), R26.1
Other:
- note removed: "Возможно, понадобятся германиевые диоды"
- moved on the sheet: C22, C24, C25, C3, D10, D5, D7, D8, J6, J7, JP2, R20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

Commit message: up
Other:
- note added: "КТ503 синяя точка сверху КТ502 белая точка сверху"
Changed lines of the file:
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@@
     (stroke (width 0) (type default) (color 0 0 0 0))
+  )
+  (text "КТ503 синяя точка сверху\nКТ502 белая точка сверху\n"
+    (at 252.73 33.02 0)
+    (effects (font (size 1.27 1.27)) (justify left bottom))
   )
   (label "In L" (at 156.21 168.91 0)
