File: _Modular/dz_ChorusDelSol_modules/DelSol_Voice.kicad_sch (KiCad schematic)
At the start: 73 parts, among them J1 BBD In, J2 Mod, J3 Phase Out, J4 Power, Q1 3107, Q2 3107, U1 4011, U2 MN3007, U3 L78L05

Commit message: up
Other:
- note added: "For MN3207 (positive power) version: Put all jumpers to other (open) position Q1, Q2 are NPN (КТ3102 or similar) Don't mount R20, D8, R21 and caps around Mount D4, R19, U3 and caps around"
Changed lines of the file:
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@@
     (stroke (width 0) (type default) (color 0 0 0 0))
+  )
+  (text "For MN3207 (positive power) version:\nPut all jumpers to other (open) position\nQ1, Q2 are NPN (КТ3102 or similar)\nDon't mount R20, D8, R21 and caps around\nMount D4, R19, U3 and caps around"
+    (at 195.58 152.4 0)
+    (effects (font (size 1.27 1.27)) (justify left bottom))
   )
   (label "Vdd" (at 137.16 166.37 0)
