File: _Modular/dz_ChorusDelSol_modules/DelSol_Preamp.kicad_sch (KiCad schematic)
At the start: 79 parts, among them J1 Filter Switch, J2 BBD Drive, J3 Dry LMR In, J4 Eq Pot 10k, J5 Eq Pot 10k, J6 Eq Pot 10k, J7 Power, U1 LM2904, U2 MCP601-xP, U3 LM2902

Commit message: up
Parts:
- C17: value 47n -> 47p
Other:
- note added: "C17 was 47n originally Seems to be an error"
Changed lines of the file:
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@@
     (stroke (width 0) (type default) (color 0 0 0 0))
+  )
+  (text "C17 was 47n originally\nSeems to be an error" (at 129.54 88.9 0)
+    (effects (font (size 1.27 1.27)) (justify left bottom))
   )
   (label "1{slash}2" (at 54.61 90.17 180)
@@
   )
   (symbol (lib_id "Device:C") (at 130.81 72.39 0) (unit 1)
-    (in_bom yes) (on_board yes) (fields_autoplaced)
-    (property "Reference" "C15" (id 0) (at 133.731 71.5553 0)
-      (effects (font (size 1.27 1.27)) (justify left))
-    )
-    (property "Value" "22n" (id 1) (at 133.731 74.0922 0)
+    (in_bom yes) (on_board yes)
+    (property "Reference" "C15" (id 0) (at 133.35 73.66 0)
+      (effects (font (size 1.27 1.27)) (justify left))
+    )
+    (property "Value" "22n" (id 1) (at 133.35 76.2 0)
       (effects (font (size 1.27 1.27)) (justify left))
     )
@@
   (symbol (lib_id "Device:R_Potentiometer_Trim") (at 142.24 72.39 0) (unit 1)
     (in_bom yes) (on_board yes)
-    (property "Reference" "RV4" (id 0) (at 140.462 71.5553 0)
+    (property "Reference" "RV4" (id 0) (at 149.86 73.66 0)
       (effects (font (size 1.27 1.27)) (justify right))
     )
@@
   )
   (symbol (lib_id "Device:C") (at 119.38 83.82 90) (unit 1)
-    (in_bom yes) (on_board yes) (fields_autoplaced)
-    (property "Reference" "C17" (id 0) (at 119.38 77.9612 90))
-    (property "Value" "47n" (id 1) (at 119.38 80.4981 90))
+    (in_bom yes) (on_board yes)
+    (property "Reference" "C17" (id 0) (at 125.73 81.28 90))
+    (property "Value" "47p" (id 1) (at 125.73 83.82 90))
     (property "Footprint" "Capacitor_SMD:C_0805_2012Metric_Pad1.18x1.45mm_HandSolder" (id 2) (at 123.19 82.8548 0)
       (effects (font (size 1.27 1.27)) hide)
@@
     )
     (path "/eb1d03a2-bad2-42ad-b450-084ba256afa9"
-      (reference "C17") (unit 1) (value "47n") (footprint "Capacitor_SMD:C_0805_2012Metric_Pad1.18x1.45mm_HandSolder")
+      (reference "C17") (unit 1) (value "47p") (footprint "Capacitor_SMD:C_0805_2012Metric_Pad1.18x1.45mm_HandSolder")
     )
     (path "/1c6d7b9a-9b0c-4066-8a48-2d8e779d4635"
