File: _Modular/TapeDelay_1.1/ControlAtmega32/cpu.kicad_sch (KiCad schematic)
At the start: 56 parts, among them J13 Transport ctl/leds, J14 OLED, J15 Pinch, J16 Encoder/Enter/ESC, J17 ~Mute, J18 AVR-ISP-10, J19 Sensors, J2 Motor1, J7 Motor2, Q4 MMBT3906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

Commit message: up
Parts:
- gave numbers to parts that had none: 1
Changed lines of the file:
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@@
   (symbol (lib_id "power:GND") (at 168.91 66.04 270) (unit 1)
     (in_bom yes) (on_board yes)
-    (property "Reference" "#PWR?" (id 0) (at 162.56 66.04 0)
+    (property "Reference" "#PWR0107" (id 0) (at 162.56 66.04 0)
       (effects (font (size 1.27 1.27)) hide)
     )
@@
   (symbol (lib_id "Device:C") (at 172.72 66.04 270) (unit 1)
     (in_bom yes) (on_board yes)
-    (property "Reference" "C?" (id 0) (at 172.72 69.85 90))
+    (property "Reference" "C35" (id 0) (at 172.72 69.85 90))
     (property "Value" "0,1" (id 1) (at 172.72 62.23 90))
     (property "Footprint" "Capacitor_SMD:C_1206_3216Metric_Pad1.33x1.80mm_HandSolder" (id 2) (at 168.91 67.0052 0)
