File: _Modular/TapeDelay_1.2/TapeDelay_Controls/TapeDelay_Controls.kicad_pcb (KiCad board)
At the start: 2 copper layers, 127 x 35.6 mm, 33 parts, among them J1 Interrupt, J2 Sensors, J3 Encoder/Enter/ESC, J4 OLED, J5 CPU I2C, SW1 Stop, SW2 Run/Pause, SW3 RotaryEncoder_Switch, SW4 Escape, U1 PCF8574

Commit message: up
Parts:
- removed C2: 0,1, Capacitor_SMD:C_1206_3216Metric_Pad1.33x1.80mm_HandSolder
- removed J2: Sensors, Connector_PinHeader_2.54mm:PinHeader_1x08_P2.54mm_Vertical
- removed J3: Encoder/Enter/ESC, Connector_PinHeader_2.54mm:PinHeader_1x05_P2.54mm_Vertical
- removed R6, R8: 4,7k, Resistor_SMD:R_1206_3216Metric_Pad1.30x1.75mm_HandSolder
- removed R7, R9: 47k, Resistor_SMD:R_1206_3216Metric_Pad1.30x1.75mm_HandSolder
- D1: value Run -> Power/Load
- D3: value Power/Error -> Run
- J1: value Interrupt -> Encoder/Interrupt; footprint Connector_PinHeader_2.54mm:PinHeader_1x01_P2.54mm_Vertical -> Connector_PinHeader_2.54mm:PinHeader_1x04_P2.54mm_Vertical; moved to F.Cu
- SW1: value Stop -> Run/Pause
- SW2: value Run/Pause -> Unload
- moved R3 13.4 mm to (75.8, 55.2)
- moved D3 13.3 mm to (74.2, 50.8)
- moved D2 13.3 mm to (61.0, 50.8)
- moved R2 13.1 mm to (62.5, 55.2)
- moved J1 12.7 mm to (159.4, 45.7), turned to 0 degrees
Connections:
- J1 pad 1: Net-(J1-Pad1) -> GND
- R1 pad 2: Net-(J1-Pad1) -> /Int
- R2 pad 1: Net-(U1-Pad6) -> Net-(R2-Pad1)
- R3 pad 1: Net-(U1-Pad7) -> Net-(R3-Pad1)
- R4 pad 1: Net-(U1-Pad4) -> Net-(R4-Pad1)
- R5 pad 1: Net-(U1-Pad5) -> Net-(R5-Pad1)
- U1 pad 10: /S2 -> Net-(R5-Pad1)
- U1 pad 11: Net-(SW2-Pad2) -> Net-(R2-Pad1)
- U1 pad 12: Net-(SW1-Pad2) -> Net-(R3-Pad1)
- U1 pad 13: Net-(J1-Pad1) -> /Int
- U1 pad 4: Net-(U1-Pad4) -> /Enter
- U1 pad 5: Net-(U1-Pad5) -> /Escape
- U1 pad 6: Net-(U1-Pad6) -> Net-(SW2-Pad2)
- U1 pad 7: Net-(U1-Pad7) -> Net-(SW1-Pad2)
- U1 pad 9: /S1 -> Net-(R4-Pad1)
Routing:
- net Net-(R2-Pad1): track 0.00 -> 69.0 mm, vias 0 -> 1
- net /Escape: track 27.3 -> 89.3 mm, vias 0 -> 2
- net Net-(J1-Pad1): track 61.4 -> 0.00 mm, vias 1 -> 0
- net /Int: track 0.00 -> 58.6 mm, vias 0 -> 1
- net /Enter: track 29.1 -> 82.6 mm
- net Net-(R4-Pad1): track 0.00 -> 41.8 mm
- net Net-(U1-Pad7): track 36.8 -> 0.00 mm
- net Net-(R3-Pad1): track 0.00 -> 36.7 mm
- net +5V: track 132.5 -> 98.2 mm
- net Net-(U1-Pad6): track 23.5 -> 0.00 mm
- net GND: track 230.1 -> 209.9 mm
- net Net-(R5-Pad1): track 0.00 -> 19.2 mm
- net /S2: track 15.2 -> 0.00 mm
- net /S1: track 12.6 -> 0.00 mm
- net Net-(U1-Pad5): track 11.4 -> 0.00 mm
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