File: Mixer/Stereo_Channel/Stereo_Channel.kicad_sch (KiCad schematic)
At the start: 81 parts

Commit message: up
Parts:
- removed D?: LED_Dual_AKA, symbol Device:LED_Dual_AKA
- removed R? (x4): 47k, Resistor_SMD:R_1206_3216Metric_Pad1.30x1.75mm_HandSolder, symbol Device:R
- removed SW?: Rec1-2, symbol Switch:SW_DPST
- removed SW?: Rec5-6/7-8, symbol Switch:SW_DPST
- removed SW?: Rec3-4, symbol Switch:SW_DPST
- removed SW?: Ch On, symbol Switch:SW_DPST
- added C15: 0,1, Capacitor_SMD:C_1206_3216Metric_Pad1.33x1.80mm_HandSolder, symbol Device:C
- added C19: 10,0, Capacitor_SMD:C_0805_2012Metric_Pad1.18x1.45mm_HandSolder, symbol Device:C
- added D2, D3, D4, D5: LED, LED_THT:LED_Rectangular_W5.0mm_H2.0mm, symbol Device:LED
- added R10, R35, R36, R37, R38, R8: 47k, Resistor_SMD:R_1206_3216Metric_Pad1.30x1.75mm_HandSolder, symbol Device:R
- added R27: 91, Resistor_SMD:R_1206_3216Metric_Pad1.30x1.75mm_HandSolder, symbol Device:R
- added R30, R34: 10k, Resistor_SMD:R_1206_3216Metric_Pad1.30x1.75mm_HandSolder, symbol Device:R
- added SW1: Rec 3-4, dz_lib:Switch 2P2T 5.5x4.5mm Latched, symbol Switch:SW_DPDT_x2
- added SW3: Ch On, dz_lib:Switch 2P2T 5.5x4.5mm Latched, symbol Switch:SW_DPDT_x2
- added SW4: Rec 5-8, dz_lib:Switch 2P2T 5.5x4.5mm Latched, symbol Switch:SW_DPDT_x2
- added SW5: Rec On, dz_lib:Switch 2P2T 5.5x4.5mm Latched, symbol Switch:SW_DPDT_x2
- added SW6: Rec Select, dz_lib:SR16 Rotary Switch, symbol Switch:SW_Rotary2x6
- added SW7: Rec 1-2, dz_lib:Switch 2P2T 5.5x4.5mm Latched, symbol Switch:SW_DPDT_x2
- added U3: KA2284, Package_SIP:SIP-9_22.3x3mm_P2.54mm, symbol ussr_ic:KA2284
- C10, C12, C14, C3, C5, C7: renamed from C?; footprint Capacitor_THT:C_Disc_D5.0mm_W2.5mm_P2.50mm -> Capacitor_SMD:C_0805_2012Metric_Pad1.18x1.45mm_HandSolder
- C22, C25: renamed from C?; footprint Capacitor_THT:CP_Radial_D6.3mm_P2.50mm -> Capacitor_SMD:C_0805_2012Metric_Pad1.18x1.45mm_HandSolder
- D1: renamed from D?; footprint (none) -> LED_THT:LED_Rectangular_W5.0mm_H2.0mm
- FB1, FB2: renamed from FB?; footprint (none) -> Inductor_THT:L_Axial_L6.6mm_D2.7mm_P10.16mm_Horizontal_Vishay_IM-2
- J3, J4: renamed from J?; footprint (none) -> Connector_PinHeader_2.54mm:PinHeader_1x03_P2.54mm_Vertical
- J5: renamed from J?; footprint (none) -> Connector_PinHeader_2.54mm:PinHeader_2x10_P2.54mm_Vertical
- JP1, JP2: renamed from JP?; footprint (none) -> Jumper:SolderJumper-3_P1.3mm_Bridged12_RoundedPad1.0x1.5mm_NumberLabels
- RV1: renamed from RV?; footprint (none) -> dz_lib:Slider Pot 60mm
- RV2, RV3, RV4: renamed from RV?; footprint (none) -> dz_lib:RK12 Duplex
- gave numbers to parts that had none: 48
Connections:
- net +15V: now also C15.2, R27.2, U3.9 (Vcc)
- net GND: now also C15.1, C19.1, R34.1, SW1.1 (A), SW1.4 (A), SW3.1 (A), SW3.4 (A), SW4.1 (A), SW4.4 (A), SW5.1 (A), SW5.4 (A), SW7.1 (A), SW7.4 (A), U3.5 (GND)
- net L: now also C1.2, R19.2, SW1.3 (C), SW3.3 (C), SW4.3 (C), SW5.3 (C), SW7.3 (C); no longer RV1.4, RV2.4
- net R: now also C8.2, R26.2, SW1.6 (C), SW3.6 (C), SW4.6 (C), SW5.6 (C), SW7.6 (C); no longer RV1.1, RV2.1
- net Rec1: now also SW6.1
- net Rec2: now also SW6.7
- net Rec3: now also R37.1, SW6.2
- net Rec4: now also R38.1, SW6.8
- net Rec5: now also SW6.3
- net Rec6: now also SW6.9
- net Rec7: now also SW6.4
- net Rec8: now also SW6.10
- net at C16.2, D6.3, R31.2: now also R30.2
- net at JP1.2 (C): now also R8.1
- net at R3.2: now also SW7.5 (B)
- net at R1.2: now also SW7.2 (B)
- net at D1.1 (K): now also U3.1 (D1)
- net at D1.2 (A): now also D2.2 (A), D3.2 (A), D4.2 (A), D5.2 (A), R27.1
- new net: R38.2, SW1.5 (B)
- new net: RV1.1, RV2.1, SW3.5 (B)
- new net: RV1.4, RV2.4, SW3.2 (B)
- new net: R35.1, SW5.2 (B)
- new net: R35.2, SW6.13
- new net: D2.1 (K), U3.2 (D2)
- new net: D3.1 (K), U3.3 (D3)
- new net: D4.1 (K), U3.4 (D4)
- new net: D5.1 (K), U3.6 (D5)
- new net: C19.2, R34.2, U3.7 (Out)
- new net: R30.1, U3.8 (In)
- new net: R37.2, SW1.2 (B)
- new net: R36.1, SW5.5 (B)
- new net: R36.2, SW6.14
- new net: R10.2, SW4.5 (B)
- new net: R8.2, SW4.2 (B)
- no-connect marks 0 -> 4
Other:
- moved on the sheet: C13, C14, C16, C17, C18, C2, C20, C21, C22, C23, C24, C25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
